File: hw/Mainboard/IEEE.kicad_sch (KiCad schematic)
At the start: 33 parts, among them J3 IEEE, U2 SN74LS07, U3 SN74LS07, U4 SN74LS07, U5 74LS245, U6 74LS245

Commit message: wip: pre-routing
Connections:
- net +5V: now also RN5.5 (R4.2); no longer RN5.6 (R3.2)
- net ATN: now also U4.12 (6Y); no longer U4.2 (1Y)
- net ATN_OUT: now also U4.13 (6A); no longer U4.1 (1A)
- net DIO1: now also U2.8 (4Y); no longer U2.2 (1Y)
- net DIO2: now also U2.6 (3Y); no longer U2.4 (2Y)
- net DIO3: now also U2.10 (5Y); no longer U2.6 (3Y)
- net DIO4: now also U2.4 (2Y); no longer U2.8 (4Y)
- net DIO6: now also U3.6 (3Y); no longer U3.10 (5Y)
- net DIO7: now also U3.10 (5Y); no longer U3.12 (6Y)
- net DIO_OUT1: now also U2.9 (4A); no longer U2.1 (1A)
- net DIO_OUT2: now also U2.5 (3A); no longer U2.3 (2A)
- net DIO_OUT3: now also U2.11 (5A); no longer U2.5 (3A)
- net DIO_OUT4: now also U2.3 (2A); no longer U2.9 (4A)
- net DIO_OUT6: now also U3.5 (3A); no longer U3.11 (5A)
- net DIO_OUT7: now also U3.11 (5A); no longer U3.13 (6A)
- net EOI: now also U4.2 (1Y); no longer U4.8 (4Y)
- net EOI_OUT: now also U4.1 (1A); no longer U4.9 (4A)
- net GND: no longer U2.11 (5A), U2.13 (6A), U3.3 (2A), U3.5 (3A)
- net IFC: now also RN5.4 (R4.1), RN6.5 (R4.2), U4.4 (2Y); no longer RN5.2 (R2.1), RN6.7 (R2.2), U4.12 (6Y)
- net IFC_OUT: now also U4.3 (2A); no longer U4.13 (6A)
- net NDAC: now also U4.8 (4Y); no longer U4.4 (2Y)
- net NDAC_OUT: now also U4.9 (4A); no longer U4.3 (2A)
- net SRQ: now also RN5.2 (R2.1), RN6.7 (R2.2); no longer RN5.4 (R4.1), RN6.5 (R4.2)
- no-connect marks 8 -> 4

Commit message: wip: decent routing, remove run btn
Connections:
- net GND: now also U2.1 (1A), U2.13 (6A), U3.13 (6A), U3.3 (2A)
- no-connect marks 4 -> 8
Changed lines of the file:
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@@
   (junction (at 206.375 63.5) (diameter 0) (color 0 0 0 0)
   )
+  (junction (at 52.07 92.71) (diameter 0) (color 0 0 0 0)
+  )
   (junction (at 182.88 137.16) (diameter 0) (color 0 0 0 0)
   )
@@
   (junction (at 218.44 63.5) (diameter 0) (color 0 0 0 0)
   )
+  (junction (at 52.07 46.99) (diameter 0) (color 0 0 0 0)
+  )
   (junction (at 66.04 102.87) (diameter 0) (color 0 0 0 0)
   )
@@
   (junction (at 232.41 33.02) (diameter 0) (color 0 0 0 0)
   )
+  (no_connect (at 78.74 82.55))
+  (no_connect (at 78.74 92.71))
+  (no_connect (at 78.74 46.99))
+  (no_connect (at 78.74 34.29))
   (no_connect (at 199.39 64.77))
   (no_connect (at 199.39 74.93))
@@
     (stroke (width 0) (type default) (color 0 0 0 0))
   )
+  (wire (pts (xy 52.07 34.29) (xy 52.07 46.99))
+    (stroke (width 0) (type default) (color 0 0 0 0))
+  )
   (wire (pts (xy 218.44 74.93) (xy 218.44 102.87))
     (stroke (width 0) (type default) (color 0 0 0 0))
@@
     (stroke (width 0) (type default) (color 0 0 0 0))
   )
+  (wire (pts (xy 52.07 46.99) (xy 52.07 57.15))
+    (stroke (width 0) (type default) (color 0 0 0 0))
+  )
   (bus (pts (xy 38.1 36.83) (xy 38.1 39.37))
     (stroke (width 0) (type default) (color 0 0 0 0))
@@
     (stroke (width 0) (type default) (color 0 0 0 0))
   )
-  (wire (pts (xy 53.34 57.15) (xy 66.04 57.15))
+  (wire (pts (xy 52.07 57.15) (xy 66.04 57.15))
     (stroke (width 0) (type default) (color 0 0 0 0))
   )
@@
     (stroke (width 0) (type default) (color 0 0 0 0))
   )
+  (wire (pts (xy 52.07 82.55) (xy 52.07 92.71))
+    (stroke (width 0) (type default) (color 0 0 0 0))
+  )
   (wire (pts (xy 210.82 137.16) (xy 213.36 137.16))
     (stroke (width 0) (type default) (color 0 0 0 0))
@@
     (stroke (width 0) (type default) (color 0 0 0 0))
   )
+  (wire (pts (xy 53.34 34.29) (xy 52.07 34.29))
+    (stroke (width 0) (type default) (color 0 0 0 0))
+  )
   (wire (pts (xy 48.26 168.91) (xy 53.34 168.91))
     (stroke (width 0) (type default) (color 0 0 0 0))
@@
     (stroke (width 0) (type default) (color 0 0 0 0))
   )
+  (wire (pts (xy 53.34 82.55) (xy 52.07 82.55))
+    (stroke (width 0) (type default) (color 0 0 0 0))
+  )
   (wire (pts (xy 227.33 63.5) (xy 229.87 63.5))
     (stroke (width 0) (type default) (color 0 0 0 0))
@@
     (stroke (width 0) (type default) (color 0 0 0 0))
   )
-  (bus (pts (xy 87.63 36.83) (xy 87.63 39.37))
-    (stroke (width 0) (type default) (color 0 0 0 0))
-  )
   (wire (pts (xy 85.09 173.99) (xy 78.74 173.99))
     (stroke (width 0) (type default) (color 0 0 0 0))
@@
     (stroke (width 0) (type default) (color 0 0 0 0))
   )
+  (wire (pts (xy 52.07 46.99) (xy 53.34 46.99))
+    (stroke (width 0) (type default) (color 0 0 0 0))
+  )
+  (wire (pts (xy 52.07 92.71) (xy 52.07 102.87))
+    (stroke (width 0) (type default) (color 0 0 0 0))
+  )
   (wire (pts (xy 148.59 36.83) (xy 165.1 36.83))
     (stroke (width 0) (type default) (color 0 0 0 0))
   )
+  (wire (pts (xy 52.07 92.71) (xy 53.34 92.71))
+    (stroke (width 0) (type default) (color 0 0 0 0))
+  )
   (wire (pts (xy 177.8 107.95) (xy 177.8 125.73))
     (stroke (width 0) (type default) (color 0 0 0 0))
@@
     (stroke (width 0) (type default) (color 0 0 0 0))
   )
-  (bus (pts (xy 87.63 87.63) (xy 87.63 90.17))
-    (stroke (width 0) (type default) (color 0 0 0 0))
-  )

Commit message: gnd/+5v on unused resistors to improve routing
Connections:
- net +5V: now also RN5.6 (R3.2)
- net GND: now also RN6.3 (R3.1)
- no-connect marks 8 -> 6
Changed lines of the file:
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@@
   (junction (at 242.57 43.18) (diameter 0) (color 0 0 0 0)
   )
+  (junction (at 199.39 63.5) (diameter 0) (color 0 0 0 0)
+  )
   (junction (at 229.87 137.16) (diameter 0) (color 0 0 0 0)
   )
   (junction (at 201.93 63.5) (diameter 0) (color 0 0 0 0)
+  )
+  (junction (at 199.39 137.16) (diameter 0) (color 0 0 0 0)
   )
   (junction (at 229.87 87.63) (diameter 0) (color 0 0 0 0)
@@
   (no_connect (at 78.74 46.99))
   (no_connect (at 78.74 34.29))
-  (no_connect (at 199.39 64.77))
   (no_connect (at 199.39 74.93))
-  (no_connect (at 199.39 135.89))
   (no_connect (at 199.39 125.73))
   (bus_entry (at 167.64 102.87) (size 2.54 2.54)
@@
     (stroke (width 0) (type default) (color 0 0 0 0))
   )
+  (wire (pts (xy 199.39 63.5) (xy 201.93 63.5))
+    (stroke (width 0) (type default) (color 0 0 0 0))
+  )
   (bus (pts (xy 167.64 46.99) (xy 167.64 49.53))
     (stroke (width 0) (type default) (color 0 0 0 0))
@@
     (stroke (width 0) (type default) (color 0 0 0 0))
   )
+  (wire (pts (xy 199.39 63.5) (xy 199.39 64.77))
+    (stroke (width 0) (type default) (color 0 0 0 0))
+  )
   (wire (pts (xy 78.74 161.29) (xy 85.09 161.29))
     (stroke (width 0) (type default) (color 0 0 0 0))
@@
     (stroke (width 0) (type default) (color 0 0 0 0))
   )
-  (wire (pts (xy 196.85 137.16) (xy 201.93 137.16))
+  (wire (pts (xy 196.85 137.16) (xy 199.39 137.16))
     (stroke (width 0) (type default) (color 0 0 0 0))
   )
@@
     (stroke (width 0) (type default) (color 0 0 0 0))
   )
-  (wire (pts (xy 196.85 63.5) (xy 201.93 63.5))
+  (wire (pts (xy 196.85 63.5) (xy 199.39 63.5))
+    (stroke (width 0) (type default) (color 0 0 0 0))
+  )
+  (wire (pts (xy 199.39 137.16) (xy 201.93 137.16))
     (stroke (width 0) (type default) (color 0 0 0 0))
   )
@@
     (stroke (width 0) (type default) (color 0 0 0 0))
   )
+  (wire (pts (xy 199.39 135.89) (xy 199.39 137.16))
+    (stroke (width 0) (type default) (color 0 0 0 0))
+  )

Commit message: hw: small layout adjustments
Connections:
- net DAV: now also RN3.1 (R1.1), RN4.8 (R1.2); no longer RN3.2 (R2.1), RN4.7 (R2.2)
- net EOI: now also RN3.2 (R2.1), RN4.7 (R2.2); no longer RN3.1 (R1.1), RN4.8 (R1.2)
Other:
- note added: "'07 drivers can sink 40ma '245 trancievers provide: • TTL → CMOS level conversion • Hysterises • Hi-Z inputs to avoid loading driver"
- note removed: "'245 trancievers provide TTL->CMOS level conversion, hysterises, and avoid loading drivers due to high impedence inputs."
Changed lines of the file:
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@@
   (junction (at 220.98 33.02) (diameter 0) (color 0 0 0 0)
   )
-  (junction (at 177.8 107.95) (diameter 0) (color 0 0 0 0)
-  )
   (junction (at 213.36 63.5) (diameter 0) (color 0 0 0 0)
   )
@@
   (junction (at 218.44 102.87) (diameter 0) (color 0 0 0 0)
   )
+  (junction (at 180.34 107.95) (diameter 0) (color 0 0 0 0)
+  )
   (junction (at 135.89 62.23) (diameter 0) (color 0 0 0 0)
   )
@@
   (junction (at 260.35 125.73) (diameter 0) (color 0 0 0 0)
   )
-  (junction (at 180.34 110.49) (diameter 0) (color 0 0 0 0)
-  )
   (junction (at 135.89 173.99) (diameter 0) (color 0 0 0 0)
   )
@@
   )
   (junction (at 194.31 137.16) (diameter 0) (color 0 0 0 0)
+  )
+  (junction (at 177.8 110.49) (diameter 0) (color 0 0 0 0)
   )
   (junction (at 194.31 63.5) (diameter 0) (color 0 0 0 0)
@@
     (stroke (width 0) (type default) (color 0 0 0 0))
   )
+  (wire (pts (xy 180.34 107.95) (xy 180.34 125.73))
+    (stroke (width 0) (type default) (color 0 0 0 0))
+  )
   (wire (pts (xy 242.57 40.64) (xy 242.57 43.18))
     (stroke (width 0) (type default) (color 0 0 0 0))
@@
     (stroke (width 0) (type default) (color 0 0 0 0))
   )
-  (wire (pts (xy 170.18 110.49) (xy 180.34 110.49))
+  (wire (pts (xy 170.18 110.49) (xy 177.8 110.49))
     (stroke (width 0) (type default) (color 0 0 0 0))
   )
@@
     (stroke (width 0) (type default) (color 0 0 0 0))
   )
+  (wire (pts (xy 180.34 107.95) (xy 246.38 107.95))
+    (stroke (width 0) (type default) (color 0 0 0 0))
+  )
   (wire (pts (xy 149.86 166.37) (xy 149.86 173.99))
     (stroke (width 0) (type default) (color 0 0 0 0))
@@
     (stroke (width 0) (type default) (color 0 0 0 0))
   )
-  (wire (pts (xy 180.34 110.49) (xy 246.38 110.49))
-    (stroke (width 0) (type default) (color 0 0 0 0))
-  )
   (bus (pts (xy 167.64 77.47) (xy 167.64 80.01))
     (stroke (width 0) (type default) (color 0 0 0 0))
   )
-  (wire (pts (xy 170.18 107.95) (xy 177.8 107.95))
+  (wire (pts (xy 170.18 107.95) (xy 180.34 107.95))
     (stroke (width 0) (type default) (color 0 0 0 0))
   )
@@
     (stroke (width 0) (type default) (color 0 0 0 0))
   )
+  (wire (pts (xy 177.8 110.49) (xy 177.8 125.73))
+    (stroke (width 0) (type default) (color 0 0 0 0))
+  )
   (wire (pts (xy 148.59 46.99) (xy 165.1 46.99))
     (stroke (width 0) (type default) (color 0 0 0 0))
@@
     (stroke (width 0) (type default) (color 0 0 0 0))
   )
+  (wire (pts (xy 177.8 110.49) (xy 246.38 110.49))
+    (stroke (width 0) (type default) (color 0 0 0 0))
+  )
   (wire (pts (xy 170.18 113.03) (xy 182.88 113.03))
     (stroke (width 0) (type default) (color 0 0 0 0))
@@
     (stroke (width 0) (type default) (color 0 0 0 0))
   )
+  (wire (pts (xy 180.34 74.93) (xy 180.34 107.95))
+    (stroke (width 0) (type default) (color 0 0 0 0))
+  )
   (wire (pts (xy 149.86 166.37) (xy 148.59 166.37))
     (stroke (width 0) (type default) (color 0 0 0 0))
@@
     (stroke (width 0) (type default) (color 0 0 0 0))
   )
-  (wire (pts (xy 177.8 107.95) (xy 246.38 107.95))
-    (stroke (width 0) (type default) (color 0 0 0 0))
-  )
   (wire (pts (xy 201.93 63.5) (xy 201.93 64.77))
     (stroke (width 0) (type default) (color 0 0 0 0))
   )
-  (wire (pts (xy 177.8 74.93) (xy 177.8 107.95))
-    (stroke (width 0) (type default) (color 0 0 0 0))
-  )
   (wire (pts (xy 269.24 85.09) (xy 269.24 100.33))
     (stroke (width 0) (type default) (color 0 0 0 0))
   )
+  (wire (pts (xy 177.8 74.93) (xy 177.8 110.49))
+    (stroke (width 0) (type default) (color 0 0 0 0))
+  )
   (wire (pts (xy 78.74 171.45) (xy 85.09 171.45))
     (stroke (width 0) (type default) (color 0 0 0 0))
@@
     (stroke (width 0) (type default) (color 0 0 0 0))
   )
-  (wire (pts (xy 180.34 110.49) (xy 180.34 125.73))
-    (stroke (width 0) (type default) (color 0 0 0 0))
-  )
   (wire (pts (xy 232.41 63.5) (xy 232.41 64.77))
     (stroke (width 0) (type default) (color 0 0 0 0))
@@
     (stroke (width 0) (type default) (color 0 0 0 0))
   )
-  (wire (pts (xy 180.34 74.93) (xy 180.34 110.49))
-    (stroke (width 0) (type default) (color 0 0 0 0))
-  )
   (wire (pts (xy 48.26 171.45) (xy 53.34 171.45))
     (stroke (width 0) (type default) (color 0 0 0 0))
@@
     (stroke (width 0) (type default) (color 0 0 0 0))
   )
-  (wire (pts (xy 177.8 107.95) (xy 177.8 125.73))
-    (stroke (width 0) (type default) (color 0 0 0 0))
-  )
   (wire (pts (xy 210.82 35.56) (xy 210.82 33.02))
     (stroke (width 0) (type default) (color 0 0 0 0))
@@
     (stroke (width 0) (type default) (color 0 0 0 0))
   )
-  (text "'245 trancievers provide TTL->CMOS\nlevel conversion, hysterises, and\navoid loading drivers due to high\nimpedence inputs.\n\n"
-    (at 107.95 87.63 0)
+  (text "'07 drivers can sink 40ma\n\n'245 trancievers provide:\n• TTL → CMOS level conversion\n• Hysterises\n• Hi-Z inputs to avoid loading driver\n\n"
+    (at 116.84 106.68 0)
     (effects (font (size 1.27 1.27)) (justify left bottom))
   )

Commit message: Document schematics
Other:
- note added: "Cheap/decent approximation of MC3446 '07 drivers can sink 40ma '245 recievers provide: • TTL → CMOS level conversion • Hysterises • Hi-Z inputs to avoid loading driver"
- note removed: "'07 drivers can sink 40ma '245 trancievers provide: • TTL → CMOS level conversion • Hysterises • Hi-Z inputs to avoid loading driver"
Changed lines of the file:
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@@
-    (stroke (width 0) (type default) (color 0 0 0 0))
-  )
-  (bus (pts (xy 38.1 87.63) (xy 38.1 90.17))
     (stroke (width 0) (type default) (color 0 0 0 0))
   )
@@
     (stroke (width 0) (type default) (color 0 0 0 0))
   )
-  (text "'07 drivers can sink 40ma\n\n'245 trancievers provide:\n• TTL → CMOS level conversion\n• Hysterises\n• Hi-Z inputs to avoid loading driver\n\n"
-    (at 116.84 106.68 0)
+  (text "Cheap/decent approximation of MC3446\n\n'07 drivers can sink 40ma\n\n'245 recievers provide:\n• TTL → CMOS level conversion\n• Hysterises\n• Hi-Z inputs to avoid loading driver\n"
+    (at 106.68 111.76 0)
     (effects (font (size 1.27 1.27)) (justify left bottom))
   )

Commit message: hw: more schematic comments / cleanup
Other:
- note added: "Cheap/decent approximation of MC3446 '07 drivers can sink 40ma '245 recievers provide: • TTL → CMOS level conversion • Hysterises • Hi-Z inputs to avoid loading driver 1K resistors protect PIA2 in case it is accidentally configured to drive DIO_IN[0..7]"
- note removed: "Cheap/decent approximation of MC3446 '07 drivers can sink 40ma '245 recievers provide: • TTL → CMOS level conversion • Hysterises • Hi-Z inputs to avoid loading driver"
Changed lines of the file:
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@@
     (stroke (width 0) (type default) (color 0 0 0 0))
   )
-  (text "Cheap/decent approximation of MC3446\n\n'07 drivers can sink 40ma\n\n'245 recievers provide:\n• TTL → CMOS level conversion\n• Hysterises\n• Hi-Z inputs to avoid loading driver\n"
+  (text "Cheap/decent approximation of MC3446\n\n'07 drivers can sink 40ma\n\n'245 recievers provide:\n• TTL → CMOS level conversion\n• Hysterises\n• Hi-Z inputs to avoid loading driver\n\n1K resistors protect PIA2 in case it is\naccidentally configured to drive DIO_IN[0..7]"
     (at 106.68 111.76 0)
     (effects (font (size 1.27 1.27)) (justify left bottom))

Commit message: hw: wip add MCU, 2 layer board
Parts:
- removed R10, R11, R12, R15, R16, R17, R18, R19, R20, R21, R22, R9: 1k, Resistor_SMD:R_0402_1005Metric, symbol Device:R_Small
- added RN11, RN12, RN13: 470, Resistor_SMD:R_Array_Convex_4x0603, symbol Device:R_Pack04
- J3: footprint PET:EDGE_CON_24P_IEEE -> Retrocomputing:CBM_PET_IEEE_EDGE_CON_24P; symbol Mainboard-rescue:Conn_02x12_Card_Edge-PET -> Retrocomputing:CBM_PET_IEEE_Conn_02x12_Card_Edge
- R13, R14: value 1k -> 470; LCSC C11702 -> C25117
Connections:
- net ATN_IN: now also RN13.8 (R1.2)
- net DIO_IN1: now also RN11.8 (R1.2)
- net DIO_IN2: now also RN11.7 (R2.2)
- net DIO_IN3: now also RN11.6 (R3.2)
- net DIO_IN4: now also RN11.5 (R4.2)
- net DIO_IN5: now also RN12.8 (R1.2)
- net DIO_IN6: now also RN12.7 (R2.2)
- net DIO_IN7: now also RN12.6 (R3.2)
- net DIO_IN8: now also RN12.5 (R4.2)
- net EOI_IN: now also RN13.7 (R2.2)
- net NDAC_IN: now also RN13.6 (R3.2)
- net SRQ_IN: now also RN13.5 (R4.2)
- net at U5.11 (B7): now also RN12.4 (R4.1)
- net at U5.12 (B6): now also RN12.3 (R3.1)
- net at U5.13 (B5): now also RN12.2 (R2.1)
- net at U5.14 (B4): now also RN12.1 (R1.1)
- net at U5.15 (B3): now also RN11.4 (R4.1)
- net at U5.16 (B2): now also RN11.3 (R3.1)
- net at U5.17 (B1): now also RN11.2 (R2.1)
- net at U5.18 (B0): now also RN11.1 (R1.1)
- net at U6.15 (B3): now also RN13.4 (R4.1)
- net at U6.16 (B2): now also RN13.3 (R3.1)
- net at U6.17 (B1): now also RN13.2 (R2.1)
- net at U6.18 (B0): now also RN13.1 (R1.1)
Other:
- moved on the sheet: R13, R14

Commit message: hw: routable (wip)
Connections:
- net GND: no longer J3.12 (GND)
- net GNDPWR renamed CHASSIS_GND
- new net PD_GND: J3.12 (GND)
Changed lines of the file:
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@@
   (bus_alias "IEEE_IN" (members "DAV_IN" "NRFD_IN" "NDAC_IN" "ATN_IN" "EOI_IN" "SRQ_IN"))
   (bus_alias "IEEE" (members "ATN" "EOI" "NDAC" "SRQ" "NRFD" "DAV" "IFC"))
-  (junction (at 234.95 137.16) (diameter 0) (color 0 0 0 0)
-  )
   (junction (at 260.35 123.19) (diameter 0) (color 0 0 0 0)
   )
@@
     (stroke (width 0) (type default) (color 0 0 0 0))
   )
-  (wire (pts (xy 246.38 125.73) (xy 245.11 125.73))
+  (wire (pts (xy 245.11 125.73) (xy 245.11 127))
     (stroke (width 0) (type default) (color 0 0 0 0))
   )
@@
     (stroke (width 0) (type default) (color 0 0 0 0))
   )
-  (wire (pts (xy 234.95 137.16) (xy 245.11 137.16))
-    (stroke (width 0) (type default) (color 0 0 0 0))
-  )
   (bus (pts (xy 87.63 173.99) (xy 87.63 176.53))
     (stroke (width 0) (type default) (color 0 0 0 0))
@@
     (stroke (width 0) (type default) (color 0 0 0 0))
   )
+  (wire (pts (xy 245.11 125.73) (xy 246.38 125.73))
+    (stroke (width 0) (type default) (color 0 0 0 0))
+  )
   (wire (pts (xy 218.44 135.89) (xy 218.44 137.16))
     (stroke (width 0) (type default) (color 0 0 0 0))
@@
   )
   (wire (pts (xy 199.39 137.16) (xy 201.93 137.16))
-    (stroke (width 0) (type default) (color 0 0 0 0))
-  )
-  (wire (pts (xy 245.11 125.73) (xy 245.11 137.16))
     (stroke (width 0) (type default) (color 0 0 0 0))
   )
@@
     (pin "1")
   )
+  (symbol (lib_id "PET:PD_GND") (at 245.11 127 0) (unit 1)
+    (in_bom yes) (on_board yes)
+    (property "Reference" "#PWR0183" (id 0) (at 245.11 133.35 0)
+      (effects (font (size 1.27 1.27)) hide)
+    )
+    (property "Value" "PD_GND" (id 1) (at 245.11 130.81 0))
+    (property "Footprint" "" (id 2) (at 245.11 127 0)
+      (effects (font (size 1.27 1.27)) hide)
+    )
+    (property "Datasheet" "" (id 3) (at 245.11 127 0)
+      (effects (font (size 1.27 1.27)) hide)
+    )
+    (pin "1")
+  )
   (symbol (lib_id "Device:R_Pack04") (at 116.84 44.45 90) (mirror x) (unit 1)
     (in_bom yes) (on_board yes)
@@
     (pin "1")
   )
-  (symbol (lib_id "power:GNDPWR") (at 260.35 127 0) (unit 1)
-    (in_bom yes) (on_board yes)
-    (property "Reference" "#PWR0145" (id 0) (at 260.35 132.08 0)
-      (effects (font (size 1.27 1.27)) hide)
-    )
-    (property "Value" "GNDPWR" (id 1) (at 260.4516 130.9116 0))
-    (property "Footprint" "" (id 2) (at 260.35 128.27 0)
-      (effects (font (size 1.27 1.27)) hide)
-    )
-    (property "Datasheet" "" (id 3) (at 260.35 128.27 0)
-      (effects (font (size 1.27 1.27)) hide)
-    )
-    (pin "1")
-  )
   (symbol (lib_id "Device:R_Pack04") (at 232.41 69.85 0) (unit 1)
     (in_bom yes) (on_board yes)
@@
     (pin "8")
   )
+  (symbol (lib_id "PET:CHASSIS_GND") (at 260.35 127 0) (unit 1)
+    (in_bom yes) (on_board yes)
+    (property "Reference" "#PWR0184" (id 0) (at 260.35 132.08 0)
+      (effects (font (size 1.27 1.27)) hide)
+    )
+    (property "Value" "CHASSIS_GND" (id 1) (at 260.35 130.81 0))
+    (property "Footprint" "" (id 2) (at 260.35 128.27 0)
+      (effects (font (size 1.27 1.27)) hide)
+    )
+    (property "Datasheet" "" (id 3) (at 260.35 128.27 0)
+      (effects (font (size 1.27 1.27)) hide)
+    )
+    (pin "1")
+  )
 )
