File: hw/Mainboard/CPLD.kicad_sch (KiCad schematic)
At the start: 4 parts, among them J21 FPGA-P4, J22 FPGA_P1, J23 FPGA_P2, J24 FPGA_P3

Commit message: wip: pre-routing
Connections:
- net P21 is gone; now on net ~{PI_PENDING}: J21.14 (Pin_14)
- net P23 is gone; now on net ~{PI_DONE}: J21.23 (Pin_23)
- net P88 is gone; now on net SYNC: J23.12 (Pin_12)
- net AUDIO: now also J21.21 (Pin_21); no longer J23.4 (Pin_4)
- net RAM_A10: now also J23.4 (Pin_4); no longer J23.9 (Pin_9)
- net RAM_A11: now also J23.5 (Pin_5); no longer J23.8 (Pin_8)
- net R~{W}: now also J23.25 (Pin_25); no longer J24.23 (Pin_23)
- net SYNC: no longer J23.25 (Pin_25)
- net ~{IRQ}: now also J24.23 (Pin_23); no longer J23.10 (Pin_10)
- net ~{PI_DONE}: no longer J21.21 (Pin_21)
- net ~{PI_PENDING}: no longer J21.13 (Pin_13)
- net ~{RD_STROBE}: now also J23.10 (Pin_10); no longer J23.5 (Pin_5)
- new net P22: J21.13 (Pin_13)
- new net P80_GND: J23.8 (Pin_8)
- new net P81_1V2: J23.9 (Pin_9)
Changed lines of the file:
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@@
     (stroke (width 0) (type default) (color 0 0 0 0))
   )
-  (wire (pts (xy 146.05 58.42) (xy 146.05 64.77))
+  (wire (pts (xy 146.05 58.42) (xy 146.05 69.85))
     (stroke (width 0) (type default) (color 0 0 0 0))
   )
@@
     (stroke (width 0) (type default) (color 0 0 0 0))
   )
-  (wire (pts (xy 153.67 58.42) (xy 153.67 67.31))
+  (wire (pts (xy 153.67 58.42) (xy 153.67 69.85))
     (stroke (width 0) (type default) (color 0 0 0 0))
   )
@@
     (stroke (width 0) (type default) (color 0 0 0 0))
   )
-  (wire (pts (xy 95.25 109.22) (xy 88.9 109.22))
+  (wire (pts (xy 95.25 109.22) (xy 90.17 109.22))
     (stroke (width 0) (type default) (color 0 0 0 0))
   )
@@
     (effects (font (size 1.27 1.27)) (justify left bottom))
   )
-  (label "~{IRQ}" (at 146.05 64.77 90)
+  (label "~{IRQ}" (at 90.17 106.68 0)
     (effects (font (size 1.27 1.27)) (justify left bottom))
   )
@@
     (effects (font (size 1.27 1.27)) (justify right bottom))
   )
-  (label "~{PI_DONE}" (at 152.4 156.21 90)
-    (effects (font (size 1.27 1.27)) (justify left bottom))
+  (label "~{PI_DONE}" (at 154.94 156.21 90)
+    (effects (font (size 1.27 1.27) (thickness 0.254) bold) (justify left bottom))
   )
   (label "VIA_CB2" (at 208.28 129.54 180)
@@
     (effects (font (size 1.27 1.27)) (justify right bottom))
   )
-  (label "P88" (at 143.51 64.77 90)
-    (effects (font (size 1.27 1.27)) (justify left bottom))
-  )
   (label "~{LED_D2}" (at 129.54 158.75 90)
     (effects (font (size 1.27 1.27)) (justify left bottom))
@@
     (effects (font (size 1.27 1.27)) (justify right bottom))
   )
-  (label "~{RES}" (at 88.9 109.22 0)
+  (label "~{RES}" (at 90.17 109.22 0)
     (effects (font (size 1.27 1.27)) (justify left bottom))
   )
@@
     (effects (font (size 1.27 1.27)) (justify left bottom))
   )
-  (label "SYNC" (at 125.73 38.1 270)
+  (label "SYNC" (at 143.51 64.77 90)
+    (effects (font (size 1.27 1.27) italic) (justify left bottom))
+  )
+  (label "P81_1V2" (at 146.05 34.29 270)
     (effects (font (size 1.27 1.27)) (justify right bottom))
   )
@@
   )
   (label "D4" (at 128.27 64.77 90)
-    (effects (font (size 1.27 1.27)) (justify left bottom))
+    (effects (font (size 1.27 1.27) (thickness 0.254) bold) (justify left bottom))
   )
   (label "PI_A10" (at 241.3 57.15 180)
     (effects (font (size 1.27 1.27)) (justify right bottom))
   )
-  (label "P21" (at 142.24 111.76 270)
-    (effects (font (size 1.27 1.27)) (justify right bottom))
+  (label "P22" (at 142.24 158.75 90)
+    (effects (font (size 1.27 1.27) italic) (justify left bottom))
   )
   (label "PI_A14" (at 185.42 99.06 180)
@@
   )
   (label "ϕ2" (at 154.94 111.76 270)
-    (effects (font (size 1.27 1.27)) (justify right bottom))
-  )
-  (label "AUDIO" (at 153.67 67.31 90)
+    (effects (font (size 1.27 1.27) (thickness 0.254) bold) (justify right bottom))
+  )
+  (label "AUDIO" (at 152.4 156.21 90)
     (effects (font (size 1.27 1.27)) (justify left bottom))
   )
   (label "CLK_50" (at 139.7 158.75 90)
-    (effects (font (size 1.27 1.27)) (justify left bottom))
+    (effects (font (size 1.27 1.27) italic) (justify left bottom))
   )
   (label "A12" (at 213.36 62.23 180)
@@
   )
   (label "PI_CLK" (at 139.7 111.76 270)
-    (effects (font (size 1.27 1.27)) (justify right bottom))
+    (effects (font (size 1.27 1.27) italic) (justify right bottom))
   )
   (label "PI_D4" (at 241.3 88.9 180)
@@
     (effects (font (size 1.27 1.27)) (justify left bottom))
   )
-  (label "~{PI_PENDING}" (at 142.24 158.75 90)
-    (effects (font (size 1.27 1.27)) (justify left bottom))
+  (label "~{PI_PENDING}" (at 142.24 111.76 270)
+    (effects (font (size 1.27 1.27) italic) (justify right bottom))
   )
   (label "BE" (at 241.3 148.59 180)
@@
     (effects (font (size 1.27 1.27)) (justify right bottom))
   )
-  (label "R~{W}" (at 90.17 106.68 0)
-    (effects (font (size 1.27 1.27)) (justify left bottom))
+  (label "R~{W}" (at 125.73 38.1 270)
+    (effects (font (size 1.27 1.27) (thickness 0.254) bold) (justify right bottom))
   )
   (label "RAM_A11" (at 234.95 21.59 0)
@@
     (effects (font (size 1.27 1.27)) (justify right bottom))
   )
-  (label "RAM_A10" (at 146.05 34.29 270)
-    (effects (font (size 1.27 1.27)) (justify right bottom))
+  (label "RAM_A10" (at 153.67 69.85 90)
+    (effects (font (size 1.27 1.27)) (justify left bottom))
   )
   (label "PI_A6" (at 241.3 46.99 180)
@@
   )
   (label "GRAPHICS" (at 138.43 34.29 270)
-    (effects (font (size 1.27 1.27)) (justify right bottom))
+    (effects (font (size 1.27 1.27) italic) (justify right bottom))
   )
   (label "PI_A0" (at 241.3 31.75 180)
@@
     (effects (font (size 1.27 1.27)) (justify right bottom))
   )
-  (label "~{RD_STROBE}" (at 151.13 31.75 270)
-    (effects (font (size 1.27 1.27)) (justify right bottom))
+  (label "~{RD_STROBE}" (at 146.05 69.85 90)
+    (effects (font (size 1.27 1.27)) (justify left bottom))
   )
   (label "~{LED_D4}" (at 132.08 158.75 90)
@@
   )
   (label "DIAG" (at 140.97 34.29 270)
-    (effects (font (size 1.27 1.27)) (justify right bottom))
+    (effects (font (size 1.27 1.27) italic) (justify right bottom))
   )
   (label "RAM_A10" (at 234.95 19.05 0)
@@
     (effects (font (size 1.27 1.27)) (justify left bottom))
   )
-  (label "RAM_A11" (at 148.59 69.85 90)
-    (effects (font (size 1.27 1.27)) (justify left bottom))
+  (label "RAM_A11" (at 151.13 31.75 270)
+    (effects (font (size 1.27 1.27)) (justify right bottom))
   )
   (label "A2" (at 90.17 86.36 0)
@@
   )
   (label "VIA_CB2" (at 140.97 69.85 90)
-    (effects (font (size 1.27 1.27)) (justify left bottom))
+    (effects (font (size 1.27 1.27) italic) (justify left bottom))
   )
   (label "PI_A12" (at 241.3 62.23 180)
@@
     (effects (font (size 1.27 1.27)) (justify right bottom))
   )
+  (label "P80_GND" (at 148.59 69.85 90)
+    (effects (font (size 1.27 1.27)) (justify left bottom))
+  )
   (label "A7" (at 213.36 49.53 180)
     (effects (font (size 1.27 1.27)) (justify right bottom))
@@
     (effects (font (size 1.27 1.27)) (justify right bottom))
   )
-  (label "P23" (at 154.94 156.21 90)
-    (effects (font (size 1.27 1.27)) (justify left bottom))
-  )
   (label "A1" (at 213.36 34.29 180)

Commit message: Document schematics
Other:
- moved on the sheet: J21, J22, J23, J24

Commit message: hw: T8 (wip)
Parts:
- removed J22: FPGA_P1, Connector_PinSocket_2.54mm:PinSocket_2x14_P2.54mm_Vertical, symbol Connector_Generic:Conn_02x14_Odd_Even
- added C59: 10n, Capacitor_SMD:C_0402_1005Metric, symbol Device:C_Small
- added D8: GRN_DONE, LED_SMD:LED_0603_1608Metric, symbol Device:LED
- added D9: RED_STATUS, LED_SMD:LED_0603_1608Metric, symbol Device:LED
- added J22: Conn_02x15_Odd_Even, Connector_PinHeader_2.54mm:PinHeader_2x15_P2.54mm_Vertical, symbol Connector_Generic:Conn_02x15_Odd_Even
- added JP10: TRI, Jumper:SolderJumper-2_P1.3mm_Open_RoundedPad1.0x1.5mm, symbol Jumper:SolderJumper_2_Open
- added Q4: MMBT3904, Package_TO_SOT_SMD:SOT-23, symbol Transistor_BJT:MMBT3904
- added R27, R32, R33: 10k, Resistor_SMD:R_0402_1005Metric, symbol Device:R_Small
- added R28: 33, Resistor_SMD:R_0402_1005Metric, symbol Device:R_Small
- added R29, R31: 1k, Resistor_SMD:R_0402_1005Metric, symbol Device:R_Small
- added R30: 100k, Resistor_SMD:R_0402_1005Metric, symbol Device:R_Small
- added RN14: 10k, Resistor_SMD:R_Array_Convex_4x0603, symbol Device:R_Pack04
- added U21: T8Q144C3, SnapEDA:QFP50P2200X2200X160-144N, symbol SnapEDA:T8Q144C3
- added X1: 50MHZ, T8Dev:Oscillator_SMD3225_4P, symbol Oscillator:ASCO
- J21, J23, J24: footprint Connector_PinSocket_2.54mm:PinSocket_2x14_P2.54mm_Vertical -> Connector_PinHeader_2.54mm:PinHeader_2x14_P2.54mm_Vertical
Connections:
- net P73_LP is gone; now on net AUDIO: J23.3 (Pin_3)
- net ~{LED_D2} is gone; now on net ϕ2: J21.3 (Pin_3)
- net ~{LED_D4} is gone; now on net ~{PIA1_CS}: J21.5 (Pin_5)
- net ~{LED_D5} is gone; now on net ~{VIA_CS}: J21.7 (Pin_7)
- net +3V3: now also C59.1, R27.2, R29.2, R32.2, RN14.5 (R4.2), RN14.6 (R3.2), RN14.7 (R2.2), RN14.8 (R1.2), X1.4 (VDD); no longer J21.27 (Pin_27), J21.28 (Pin_28), J23.28 (Pin_28), J24.28 (Pin_28)
- net A0: now also J24.1 (Pin_1); no longer J24.3 (Pin_3)
- net A1: now also J24.3 (Pin_3); no longer J24.5 (Pin_5)
- net A10: now also J24.21 (Pin_21); no longer J24.8 (Pin_8)
- net A11: now also J24.25 (Pin_25); no longer J24.10 (Pin_10)
- net A12: now also J24.2 (Pin_2); no longer J24.12 (Pin_12)
- net A13: now also J24.4 (Pin_4); no longer J24.14 (Pin_14)
- net A14: now also J24.6 (Pin_6); no longer J24.16 (Pin_16)
- net A15: now also J24.8 (Pin_8); no longer J24.18 (Pin_18)
- net A16: now also J24.10 (Pin_10); no longer J24.20 (Pin_20)
- net A2: now also J24.5 (Pin_5); no longer J24.7 (Pin_7)
- net A3: now also J24.7 (Pin_7); no longer J24.9 (Pin_9)
- net A4: now also J24.9 (Pin_9); no longer J24.11 (Pin_11)
- net A5: now also J24.11 (Pin_11); no longer J24.13 (Pin_13)
- net A6: now also J24.13 (Pin_13); no longer J24.15 (Pin_15)
- net A7: now also J24.15 (Pin_15); no longer J24.17 (Pin_17)
- net A8: now also J24.17 (Pin_17); no longer J24.4 (Pin_4)
- net A9: now also J24.19 (Pin_19); no longer J24.6 (Pin_6)
- net AUDIO: no longer J21.21 (Pin_21)
- net BE: now also J23.24 (Pin_24); no longer J23.11 (Pin_11)
- net CLK_50: now also J21.10 (Pin_10), R28.1; no longer J21.11 (Pin_11)
- net D0: now also J24.12 (Pin_12); no longer J23.23 (Pin_23)
- net D1: now also J24.14 (Pin_14); no longer J23.21 (Pin_21)
- net D2: now also J24.16 (Pin_16); no longer J23.19 (Pin_19)
- net D3: now also J24.18 (Pin_18); no longer J23.17 (Pin_17)
- net D4: now also J24.20 (Pin_20); no longer J23.24 (Pin_24)
- net D5: now also J24.22 (Pin_22); no longer J23.22 (Pin_22)
- net D6: now also J24.24 (Pin_24); no longer J23.20 (Pin_20)
- net D7: now also J24.26 (Pin_26); no longer J23.18 (Pin_18)
- net DIAG: now also J23.11 (Pin_11); no longer J23.13 (Pin_13)
- net GND: now also J21.27 (Pin_27), J21.28 (Pin_28), J23.28 (Pin_28), C59.2, D9.1 (K), J22.1 (Pin_1), J22.2 (Pin_2), J22.29 (Pin_29), JP10.1 (A), Q4.2 (E), R33.1, X1.2 (GND); no longer J21.10 (Pin_10), J21.25 (Pin_25), J21.26 (Pin_26), J21.8 (Pin_8), J21.9 (Pin_9), J23.26 (Pin_26), J24.1 (Pin_1), J24.2 (Pin_2), J24.26 (Pin_26), J24.27 (Pin_27)
- net GRAPHICS: now also J23.13 (Pin_13); no longer J23.15 (Pin_15)
- net HORIZ: now also J21.8 (Pin_8); no longer J21.16 (Pin_16)
- net RAM_A10: now also J24.23 (Pin_23); no longer J23.4 (Pin_4)
- net RAM_A11: now also J24.27 (Pin_27); no longer J23.5 (Pin_5)
- net RDY: now also J23.19 (Pin_19); no longer J21.15 (Pin_15)
- net R~{W}: now also J24.28 (Pin_28); no longer J23.25 (Pin_25)
- net SYNC: now also J23.26 (Pin_26); no longer J23.12 (Pin_12)
- net ~{IO_OE}: now also J21.11 (Pin_11); no longer J24.24 (Pin_24)
- net ~{IRQ}: now also J23.22 (Pin_22); no longer J24.23 (Pin_23)
- net ~{NMI}: now also J23.25 (Pin_25); no longer J23.16 (Pin_16)
- net ~{PIA1_CS}: no longer J24.21 (Pin_21)
- net ~{PIA2_CS}: now also J21.9 (Pin_9); no longer J24.22 (Pin_22)
- net ~{RAM_CE}: now also J23.16 (Pin_16); no longer J23.7 (Pin_7)
- net ~{RD_STROBE}: now also J23.15 (Pin_15); no longer J23.10 (Pin_10)
- net ~{RES}: now also J23.20 (Pin_20); no longer J24.25 (Pin_25)
- net ~{VIA_CS}: no longer J24.19 (Pin_19)
- net ~{WR_STROBE}: now also J23.17 (Pin_17); no longer J23.6 (Pin_6)
- net ϕ2: no longer J21.24 (Pin_24)
- net +1V2: no longer names the net of J21.19 (Pin_19)
- net +1V2: no longer J21.20 (Pin_20)
- net P22: no longer names the net of J21.13 (Pin_13)
- net P26_1V2: no longer names the net of J21.18 (Pin_18)
- net P27_GND: no longer names the net of J21.17 (Pin_17)
- net P80_GND: no longer names the net of J23.8 (Pin_8)
- net P81_1V2: no longer names the net of J23.9 (Pin_9)
- net PI_CLK: no longer names the net of J21.12 (Pin_12)
- net PI_R~{W}: no longer names the net of J21.22 (Pin_22)
- net ~{PI_DONE}: no longer names the net of J21.23 (Pin_23)
- net ~{PI_PENDING}: no longer names the net of J21.14 (Pin_14)
- new net: Q4.1 (B), R30.1
- new net: D8.1 (K), Q4.3 (C)
- new net: D8.2 (A), R29.1
- new net: JP10.2 (B), X1.1 (Tri-State)
- new net: R28.2, X1.3 (OUT)
- new net: R27.1, U21.74 (GPIOR_158_TEST_N)
- new net: D9.2 (A), R31.1
- new net CBUS0: U21.78 (GPIOR_151_CBUS0)
- new net CBUS1: U21.79 (GPIOR_150_CBUS1)
- new net CBUS2: U21.80 (GPIOR_149_CBUS2)
- new net CCK: J22.8 (Pin_8), U21.30 (GPIOL_01_CCK)
- new net CDI0: J22.10 (Pin_10), U21.29 (GPIOL_08_CDI0)
- new net CDI1: J22.12 (Pin_12), U21.28 (GPIOL_09_CDI1)
- new net CDONE: J22.18 (Pin_18), R30.2, R32.1, U21.34 (CDONE)
- new net CSI: U21.32 (GPIOL_04_CSI)
- new net NSTATUS: R31.2, U21.136 (GPIOL_71_NSTATUS)
- new net TCK: J22.24 (Pin_24), RN14.1 (R1.1), U21.26 (TCK)
- new net TDI: J22.26 (Pin_26), RN14.2 (R2.1), U21.27 (TDI)
- new net TDO: J22.28 (Pin_28), RN14.3 (R3.1), U21.24 (TDO)
- new net TMS: J22.30 (Pin_30), RN14.4 (R4.1), U21.25 (TMS)
- new net ~{CRESET}: J22.16 (Pin_16), R33.2, U21.35 (~{CRESET})
- new net ~{ML}: J23.23 (Pin_23)
- new net ~{SO}: J23.21 (Pin_21)
- new net ~{SS}: J22.14 (Pin_14), U21.31 (GPIOL_00_SS_N)
- new net ~{VP}: J23.18 (Pin_18)
- no-connect marks 0 -> 5
Other:
- note added: "AD0"
- note added: "AD1"
- note added: "AD2"
- note added: "AD3"
- note added: "AD4"
- note added: "AD5"
- note added: "BD0"
- note added: "BD1"
- note added: "BD2"
- note added: "BD3"
- note added: "CDONE is an open drain"
- note added: "CDONE is an open drain output with 10k pullup. Driving LED requires a current amplifier."
- note added: "NSTATUS driven low on error"
- note added: "Pull ~{CRESET} low to remain in reset until MCU drives pin high."
- moved on the sheet: J21, J23, J24

Commit message: hw: routing (excluding MCU)
Parts:
- added C60, C69, C70: 1u, Capacitor_SMD:C_0402_1005Metric, symbol Device:C_Small
- added C61, C62, C63, C64, C71, C72, C73, C74, C75, C76: 100n, Capacitor_SMD:C_0402_1005Metric, symbol Device:C_Small
- added C65, C66, C67, C68, C77, C78, C79, C80: 10n, Capacitor_SMD:C_0402_1005Metric, symbol Device:C_Small
- added R34: 12k 1%, Resistor_SMD:R_0402_1005Metric, symbol Device:R_Small
- X1: footprint T8Dev:Oscillator_SMD3225_4P -> Crystal:Crystal_SMD_3225-4Pin_3.2x2.5mm
Connections:
- net CBUS0 is gone; now on net I2C1_SDA: U21.78 (GPIOR_151_CBUS0)
- net CBUS1 is gone; now on net I2C1_SCL: U21.79 (GPIOR_150_CBUS1)
- net CBUS2 is gone; now on net SPI1_~{READY}: U21.80 (GPIOR_149_CBUS2)
- net CSI is gone; now on net GP25: U21.32 (GPIOL_04_CSI)
- net +3V3: now also C69.1, C70.1, C71.1, C72.1, C73.1, C74.1, C75.1, C76.1, C77.1, C78.1, C79.1, C80.1
- net A0: now also U21.65 (GPIOB_RXN07)
- net A1: now also U21.67 (GPIOB_RXP10)
- net A10: now also U21.105 (GPIOR_95_CDI26)
- net A11: now also U21.111 (GPIOR_85)
- net A12: now also U21.66 (GPIOB_RXP07)
- net A13: now also U21.68 (GPIOB_RXN10)
- net A14: now also U21.70 (GPIOB_RXP12_EXTFB0)
- net A15: now also U21.72 (GPIOB_CLKN0)
- net A16: now also U21.77 (GPIOR_154)
- net A2: now also U21.69 (GPIOB_RXN12_EXTFB0)
- net A3: now also U21.71 (GPIOB_CLKP0)
- net A4: now also U21.76 (GPIOR_155)
- net A5: now also U21.81 (GPIOR_139)
- net A6: now also U21.83 (GPIOR_136_CDI16)
- net A7: now also U21.86 (GPIOR_133_CDI18)
- net A8: now also U21.100 (GPIOR_113_CDI22)
- net A9: now also U21.102 (GPIOR_105_CDI24)
- net AUDIO: now also J23.4 (Pin_4), U21.38 (GPIOB_TXP00); no longer J23.3 (Pin_3)
- net BE: now also U21.59 (GPIOB_RXN02)
- net CLK_50: now also J21.16 (Pin_16), U21.131 (GPIOL_75_PLLIN1); no longer J21.10 (Pin_10)
- net D0: now also U21.82 (GPIOR_138)
- net D1: now also U21.84 (GPIOR_135_CDI17)
- net D2: now also U21.87 (GPIOR_132_CDI19)
- net D3: now also U21.101 (GPIOR_112_CDI23)
- net D4: now also U21.103 (GPIOR_104_CDI25)
- net D5: now also U21.106 (GPIOR_94_CDI27)
- net D6: now also U21.110 (GPIOR_87_CDI29)
- net D7: now also U21.112 (GPIOR_86)
- net DIAG: now also J23.12 (Pin_12), U21.42 (GPIOB_TXP04); no longer J23.11 (Pin_11)
- net GND: now also C60.2, C61.2, C62.2, C63.2, C64.2, C65.2, C66.2, C67.2, C68.2, C69.2, C70.2, C71.2, C72.2, C73.2, C74.2, C75.2, C76.2, C77.2, C78.2, C79.2, C80.2, R34.1; no longer J22.1 (Pin_1)
- net GRAPHICS: now also U21.43 (GPIOB_TXN04)
- net HORIZ: now also U21.118 (GPIOR_79_EXTFB1_CDI30)
- net RAM_A10: now also U21.109 (GPIOR_88_CDI28)
- net RAM_A11: now also U21.113 (GPIOR_84)
- net RDY: now also U21.54 (GPIOB_TXN11)
- net R~{W}: now also U21.99 (GPIOR_116_CTRL15)
- net SYNC: now also U21.61 (GPIOB_RXP03)
- net VERT: now also U21.116 (GPIOR_81_MREFCLK)
- net VIA_CB2: now also U21.45 (GPIOB_TXP06)
- net VIDEO: now also U21.114 (GPIOR_83)
- net ~{IO_OE}: now also J21.10 (Pin_10), U21.123 (GPIOR_77_PLLIN1); no longer J21.11 (Pin_11)
- net ~{IRQ}: now also U21.56 (GPIOB_RXN00)
- net ~{ML}: now also U21.58 (GPIOB_RXP02)
- net ~{NMI}: now also U21.60 (GPIOB_RXN03)
- net ~{PIA1_CS}: now also U21.115 (GPIOR_82)
- net ~{PIA2_CS}: now also U21.119 (GPIOR_78_EXTFB0_CDI31)
- net ~{RAM_CE}: now also U21.47 (GPIOB_TXP09)
- net ~{RD_STROBE}: now also U21.46 (GPIOB_TXN06)
- net ~{RES}: now also U21.98 (GPIOR_117_CTRL14)
- net ~{SO}: now also U21.55 (GPIOB_RXP00)
- net ~{VIA_CS}: now also U21.117 (GPIOR_80)
- net ~{VP}: now also U21.53 (GPIOB_TXP11)
- net ~{WR_STROBE}: now also U21.48 (GPIOB_TXN09)
- net ϕ2: now also U21.97 (GPIOR_122_CLK13_CDI21)
- net MCU_CLK: now reaches J21.15 (Pin_15)
- net MCU_CLK: now also U21.132 (GPIOL_74_PLLIN0)
- net S1: now reaches J23.10 (Pin_10)
- net S1: now also U21.41 (GPIOB_TXN02)
- net S3: now reaches J23.6 (Pin_6)
- net S3: now also U21.39 (GPIOB_TXN00)
- net S2: now reaches J23.8 (Pin_8)
- net S2: now also U21.40 (GPIOB_TXP02)
- net at U21.36 (REF_RES): now also R34.2
- net SPI1_~{CS}: now reaches U21.10 (GPIOL_32_CTRL4_CDI7)
- net SPI1_~{CS}: now also J22.5 (Pin_5)
- net SPI1_SCK: now reaches U21.11 (GPIOL_31_CLK7_CDI6)
- net SPI1_SCK: now also J22.7 (Pin_7)
- net SPI1_TX: now reaches U21.7 (GPIOL_41_CDI9)
- net SPI1_TX: now also J22.1 (Pin_1)
- net SPI1_RX: now reaches U21.8 (GPIOL_40_CDI8)
- net SPI1_RX: now also J22.3 (Pin_3)
- net I2C1_SCL: now reaches J22.15 (Pin_15)
- net I2C1_SDA: now reaches J22.17 (Pin_17)
- net MCU_CEC: now reaches J22.19 (Pin_19)
- net GP25: now reaches J22.21 (Pin_21)
- net GP27: now reaches J22.23 (Pin_23)
- net I2C0_SCL: now reaches J22.25 (Pin_25)
- net I2C0_SDA: now reaches J22.27 (Pin_27)
- net SPI1_~{READY}: now reaches J22.9 (Pin_9)
- net CCK renamed SPI0_SCK
- net CDI0 renamed SPI0_TX
- net CDI1 renamed SPI0_RX
- net ~{SS} renamed SPI0_~{CS}
- new net VCORE: C60.1, C61.1, C62.1, C63.1, C64.1, C65.1, C66.1, C67.1, C68.1
- no-connect marks 5 -> 20
Other:
- note added: "CSO is to daisy chain multiple devices"
- note added: "Pull ~{CRESET} low to suspend FPGA until MCU drives pin."
- note removed: "Pull ~{CRESET} low to remain in reset until MCU drives pin high."
- moved on the sheet: D8, D9, J21, J22, J23, J24, Q4, R27, R29, R30, R31, R32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

Commit message: hw: routed, but trace sizes need to be reviewed/fixed
Parts:
- added R48, R51, R63: 10k, Resistor_SMD:R_0402_1005Metric, symbol Device:R_Small
- added SW5: CONFIG, Button_Switch_THT:SW_DIP_SPSTx04_Slide_6.7x11.72mm_W7.62mm_P2.54mm_LowProfile, symbol Switch:SW_DIP_x04
Connections:
- net MCU_CEC is gone; now on net I2C1_SDA: J22.19 (Pin_19)
- net +3V3: now also R48.2, R51.2, R63.2
- net GND: now also SW5.1, SW5.2, SW5.3, SW5.4
- net I2C1_SCL: now also J22.17 (Pin_17); no longer J22.15 (Pin_15), U21.79 (GPIOR_150_CBUS1)
- net I2C1_SDA: no longer J22.17 (Pin_17)
- net NSTATUS: now also J21.20 (Pin_20)
- net S1: now also J21.18 (Pin_18), U21.134 (GPIOL_73_EXTFB1_CDI15), SW5.8; no longer J23.10 (Pin_10), U21.41 (GPIOB_TXN02)
- net S2: now also J21.17 (Pin_17), U21.135 (GPIOL_72_EXTFB0_CDI14), SW5.7; no longer J23.8 (Pin_8), U21.40 (GPIOB_TXP02)
- net S3: now also J21.19 (Pin_19), U21.139 (GPIOL_68), SW5.6; no longer J23.6 (Pin_6), U21.39 (GPIOB_TXN00)
- net SPI1_~{READY}: no longer U21.80 (GPIOR_149_CBUS2)
- net S5: now reaches J21.21 (Pin_21)
- net S5: now also U21.141 (GPIOL_65)
- net S4: now reaches J21.22 (Pin_22)
- net S4: now also U21.140 (GPIOL_67_CDI13), SW5.5
- net S6: now reaches J21.24 (Pin_24)
- net S6: now also U21.142 (GPIOL_66_CDI12)
- net ~{TEST}: now reaches R27.1, U21.74 (GPIOR_158_TEST_N)
- net GP25: no longer names the net of J22.21 (Pin_21)
- net GP25: no longer U21.32 (GPIOL_04_CSI)
- net GP27: no longer names the net of J22.23 (Pin_23)
- net I2C0_SCL: no longer names the net of J22.25 (Pin_25)
- net I2C0_SDA: no longer names the net of J22.27 (Pin_27)
- new net CBUS1: R51.1, U21.79 (GPIOR_150_CBUS1)
- new net CBUS2: R63.1, U21.80 (GPIOR_149_CBUS2)
- new net CSI: R48.1, U21.32 (GPIOL_04_CSI)
- new net X1: J23.10 (Pin_10), U21.41 (GPIOB_TXN02)
- new net X2: J23.8 (Pin_8), U21.40 (GPIOB_TXP02)
- new net X3: J23.6 (Pin_6), U21.39 (GPIOB_TXN00)
- no-connect marks 20 -> 27
Other:
- note added: "Pull CSI high to enable FPGA configuration Pull TEST_N high to deactivate test mode Pull CBUS[2:1] high as we don't support more than 2x Leave CBSEL[1:0] floating CRESET_N pulled low to reset FPGA until MCU is ready Config sequence: MCU drives CBUS[0] high for 1x or low for 2x MCU drives SS_N low to select passive SPI MCU transitions CRESET_N low -> high to begin (320 ns) MCU sends bitsteam via C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"
- note removed: "CSO is to daisy chain multiple devices"
- moved on the sheet: R27

Commit message: hw: routable (wip)
Parts:
- added NT7, NT8: +3V3, PET:NetTie-2_SMD_Pad_0.4_to_0.2mm, symbol Device:NetTie_2
- added unit 13 of U21
Connections:
- net +3V3: now also NT7.2; no longer C69.1, C70.1, C71.1, C72.1, C73.1, C74.1, C75.1, C76.1, C77.1, C78.1, C79.1, C80.1
- net GND: now also NT8.1
- net REF_RES: now reaches R34.2, U21.36 (REF_RES)
- net VCORE renamed FPGA_VCC
- net FPGA_VCC: now also U21.125 (VCC), U21.128 (VCC), U21.13 (VCC), U21.130 (VCC), U21.22 (VCC), U21.49 (VCC), U21.57 (VCC), U21.85 (VCC), U21.96 (VCC)
- new net FPGA_GND: NT8.2, U21.1 (GND), U21.104 (GND), U21.108 (GND), U21.120 (GND), U21.121 (GND), U21.126 (GND), U21.127 (GND), U21.129 (GND), U21.133 (GND), U21.37 (GND), U21.44 (GND), U21.5 (GND), U21.50 (GND), U21.64 (GND), U21.9 (GND), U21.94 (GND)
- new net FPGA_VCCA: U21.107 (VCCA_TR), U21.2 (VCCA_TL), U21.73 (VCCA_BR)
- new net FPGA_VCCIO: C69.1, C70.1, C71.1, C72.1, C73.1, C74.1, C75.1, C76.1, C77.1, C78.1, C79.1, C80.1, NT7.1, U21.12 (VCCIO1C_1D), U21.122 (VCCIO3A), U21.143 (VCCIO1E), U21.21 (VCCIO1B), U21.23 (VCCIO1A), U21.51 (VCCIO4B), U21.52 (VCCIO4B), U21.62 (VCCIO4A), U21.63 (VCCIO4A), U21.88 (VCCIO3E), U21.91 (VCCIO3D), U21.95 (VCCIO3B_3C)
- no-connect marks 27 -> 31
