File: hw/Mainboard/Mainboard.kicad_pcb (KiCad board)
At the start: 2 copper layers, 262.9 x 107.9 mm, 181 parts, among them J1 Audio, J10 5V PWR, J12 NOT_HDMI_A, J13 Micro_SD, J14 USB, J15 DEBUG, J18 PET_Power_01x09_Male, J2 KEYBOARD, J21 FPGA-P4, J22 FPGA_P1, J23 FPGA_P2, J24 FPGA_P3, J3 IEEE, J4 USER, J5 CASS A, J6 CASS B, J7 9V POWER, J8 SPEAKER, J9 PET_Video, Q1 AO3401A, Q2 MMBT3904, Q3 AO3401A, SW1 NMI, SW3 RUN, SW4 RESET, SW5 BOOTSEL, U1 74LS145, U10 XL1509-5.0E1, U11 W65C02S, U12 AS6C1008, U13 AMS1117-3.3, U14 RP2040, U15 LM317AG-TN3-R, U16 W25Q128JVS, U18 SN74LVC4245APWR, U19 SN74LVC4245APWR, U2 SN74LS07, U20 SN74LVC4245APWR, U3 SN74LS07, U4 SN74LS07, U5 74LS245, U6 74LS245, U7 W65C21N, U8 W65C21N, U9 W65C22N, Y1 12 MHz

Commit message: hw: T8 (wip)
Parts:
- added C52: 22u 25V, Capacitor_SMD:C_0805_2012Metric, F.Cu at (-233.1, 73.4)
- added C53: 22u 25V, Capacitor_SMD:C_0805_2012Metric, F.Cu at (-240.4, 12.4)
- added C54: 10u, Capacitor_Tantalum_SMD:CP_EIA-3216-18_Kemet-A, F.Cu at (-33.7, 11.7)
- added C55: 10u, Capacitor_Tantalum_SMD:CP_EIA-3216-18_Kemet-A, F.Cu at (-37.3, 5.85)
- added C56: 100n, Capacitor_SMD:C_0402_1005Metric, F.Cu at (-35.9, 26.8)
- added C57: 100n, Capacitor_SMD:C_0402_1005Metric, F.Cu at (-33.5, 26.8)
- added C58: 4.7u, Capacitor_SMD:C_0402_1005Metric, F.Cu at (-24.9, 26.6)
- added C59: 10n, Capacitor_SMD:C_0402_1005Metric, F.Cu at (-27.8, 26.7)
- added D8: GRN_DONE, LED_SMD:LED_0603_1608Metric, F.Cu at (-38.5, 32.6)
- added D9: RED_STATUS, LED_SMD:LED_0603_1608Metric, F.Cu at (-36.4, 42.1)
- added FB1: 600, Inductor_SMD:L_0603_1608Metric, F.Cu at (-30.8, 26.7)
- added JP10: TRI, Jumper:SolderJumper-2_P1.3mm_Open_RoundedPad1.0x1.5mm, F.Cu at (-40.5, 60.1)
- added Q4: MMBT3904, Package_TO_SOT_SMD:SOT-23, F.Cu at (-35.8, 37.5)
- added R24: 10k, Resistor_SMD:R_0402_1005Metric, F.Cu at (-118.9, 12.8)
- added R27: 10k, Resistor_SMD:R_0402_1005Metric, F.Cu at (-27.8, 24.7)
- added R28: 33, Resistor_SMD:R_0402_1005Metric, F.Cu at (-39.8, 63.7)
- added R29: 1k, Resistor_SMD:R_0402_1005Metric, F.Cu at (-35.9, 32.6)
- added R30: 100k, Resistor_SMD:R_0402_1005Metric, F.Cu at (-39.1, 36.5)
- added R31: 1k, Resistor_SMD:R_0402_1005Metric, F.Cu at (-39.0, 42.0)
- added R32: 10k, Resistor_SMD:R_0402_1005Metric, F.Cu at (-55.3, 34.4)
- added R33: 10k, Resistor_SMD:R_0402_1005Metric, F.Cu at (-55.3, 35.6)
- added RN14: 10k, Resistor_SMD:R_Array_Convex_4x0603, F.Cu at (-32.3, 19.1)
- added U17: LM1117-1.2, Package_TO_SOT_SMD:SOT-223, F.Cu at (-31.7, 6.90)
- added U21: T8Q144C3, SnapEDA:QFP50P2200X2200X160-144N, F.Cu at (-68.7, 36.6)
- J1: value Audio -> SJ-43504-SMT-TR; footprint PET:STX31205B -> SnapEDA:CUI_SJ-43504-SMT-TR
- J18: value PET_Power_01x09_Male -> PET POWER
- J21, J23, J24: footprint Connector_PinSocket_2.54mm:PinSocket_2x14_P2.54mm_Vertical -> Connector_PinHeader_2.54mm:PinHeader_2x14_P2.54mm_Vertical; moved to F.Cu
- J22: value FPGA_P1 -> Conn_02x15_Odd_Even; footprint Connector_PinSocket_2.54mm:PinSocket_2x14_P2.54mm_Vertical -> Connector_PinHeader_2.54mm:PinHeader_2x15_P2.54mm_Vertical; moved to F.Cu
- moved U13 56.0 mm to (-54.0, 4.00), turned to 180 degrees
- moved C21 53.9 mm to (-51.3, -0.70), turned to 180 degrees
- moved J10 45.4 mm to (-47.7, 1.70), turned to 90 degrees
- moved C36 44.7 mm to (-48.5, 5.35), turned to -90 degrees
- moved C13 37.8 mm to (-217.2, 69.6), turned to 180 degrees
- moved C35 25.6 mm to (-242.0, 62.2), turned to 90 degrees
- moved J9 18.8 mm to (-97.7, 84.0), turned to 90 degrees
- moved J22 17.4 mm to (-44.6, 52.8), turned to 180 degrees
- moved J23 17.4 mm to (-52.3, 12.1), turned to -90 degrees
- moved J24 17.4 mm to (-93.0, 19.8), turned to 0 degrees
- moved J21 17.4 mm to (-85.3, 60.5), turned to 90 degrees
- moved C17 16.6 mm to (-241.3, 31.4), turned to 0 degrees
- moved J8 16.5 mm to (-7.30, 33.6), turned to 0 degrees
- moved C33 15.4 mm to (-220.7, 70.3), turned to 180 degrees
- moved R52 15.1 mm to (-68.0, 7.59)
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Connections:
- C13 pad 1: +9V_Unreg -> Net-(C12-Pad2)
- J21 pad 10: GND -> /MAGIC/CPLD/CLK_50
- J21 pad 11: /MAGIC/CPLD/CLK_50 -> /MAGIC/~{IO_OE}
- J21 pad 12: /MAGIC/PI_CLK -> unconnected-(J21-Pad12)
- J21 pad 13: /MAGIC/CPLD/P22 -> unconnected-(J21-Pad13)
- J21 pad 14: /MAGIC/~{PI_PENDING} -> unconnected-(J21-Pad14)
- J21 pad 15: /MAGIC/CPLD/RDY -> unconnected-(J21-Pad15)
- J21 pad 16: /MAGIC/HORIZ -> unconnected-(J21-Pad16)
- J21 pad 17: /MAGIC/CPLD/P27_GND -> unconnected-(J21-Pad17)
- J21 pad 18: /MAGIC/CPLD/P26_1V2 -> unconnected-(J21-Pad18)
- J21 pad 19: +1V2 -> unconnected-(J21-Pad19)
- J21 pad 20: +1V2 -> unconnected-(J21-Pad20)
- J21 pad 21: /MAGIC/CPLD/AUDIO -> unconnected-(J21-Pad21)
- J21 pad 22: /MAGIC/PI_R~{W} -> unconnected-(J21-Pad22)
- J21 pad 23: /MAGIC/~{PI_DONE} -> unconnected-(J21-Pad23)
- J21 pad 24: /MAGIC/ϕ2 -> unconnected-(J21-Pad24)
- J21 pad 25: GND -> unconnected-(J21-Pad25)
- J21 pad 26: GND -> unconnected-(J21-Pad26)
- J21 pad 27: +3V3 -> GND
- J21 pad 28: +3V3 -> GND
- J21 pad 3: /MAGIC/CPLD/~{LED_D2} -> /MAGIC/ϕ2
- J21 pad 5: /MAGIC/CPLD/~{LED_D4} -> /MAGIC/~{PIA1_CS}
- J21 pad 7: /MAGIC/CPLD/~{LED_D5} -> /MAGIC/~{VIA_CS}
- J21 pad 8: GND -> /MAGIC/HORIZ
- J21 pad 9: GND -> /MAGIC/~{PIA2_CS}
- J22 pad 1: /MAGIC/PI_D7 -> GND
- J22 pad 10: /MAGIC/PI_A7 -> /MAGIC/CPLD/CDI0
- J22 pad 11: /MAGIC/PI_A14 -> unconnected-(J22-Pad11)
- J22 pad 12: /MAGIC/PI_A6 -> /MAGIC/CPLD/CDI1
- J22 pad 13: /MAGIC/PI_A13 -> unconnected-(J22-Pad13)
- J22 pad 14: /MAGIC/PI_A5 -> /MAGIC/CPLD/~{SS}
- J22 pad 15: /MAGIC/PI_A12 -> unconnected-(J22-Pad15)
- J22 pad 16: /MAGIC/PI_A4 -> /MAGIC/CPLD/~{CRESET}
- J22 pad 17: /MAGIC/PI_A11 -> unconnected-(J22-Pad17)
- J22 pad 18: /MAGIC/PI_A3 -> /MAGIC/CPLD/CDONE
- J22 pad 19: /MAGIC/PI_A10 -> unconnected-(J22-Pad19)
- J22 pad 2: /MAGIC/PI_D3 -> GND
- J22 pad 20: /MAGIC/PI_A2 -> unconnected-(J22-Pad20)
- J22 pad 21: /MAGIC/PI_A9 -> unconnected-(J22-Pad21)
- J22 pad 22: /MAGIC/PI_A1 -> unconnected-(J22-Pad22)
- J22 pad 23: /MAGIC/PI_A8 -> unconnected-(J22-Pad23)
- J22 pad 24: /MAGIC/PI_A0 -> /MAGIC/CPLD/TCK
- J22 pad 25: GND -> unconnected-(J22-Pad25)
- J22 pad 26: GND -> /MAGIC/CPLD/TDI
- J22 pad 27: +3V3 -> unconnected-(J22-Pad27)
- J22 pad 28: +3V3 -> /MAGIC/CPLD/TDO
- J22 pad 3: /MAGIC/PI_D6 -> unconnected-(J22-Pad3)
- J22 pad 4: /MAGIC/PI_D2 -> unconnected-(J22-Pad4)
- J22 pad 5: /MAGIC/PI_D5 -> unconnected-(J22-Pad5)
- J22 pad 6: /MAGIC/PI_D1 -> unconnected-(J22-Pad6)
- J22 pad 7: /MAGIC/PI_D4 -> unconnected-(J22-Pad7)
- J22 pad 8: /MAGIC/PI_D0 -> /MAGIC/CPLD/CCK
- J22 pad 9: /MAGIC/PI_A15 -> unconnected-(J22-Pad9)
- J23 pad 10: /MAGIC/CPLD/~{RD_STROBE} -> unconnected-(J23-Pad10)
- J23 pad 11: /MAGIC/CPLD/BE -> /MAGIC/CPLD/DIAG
- J23 pad 12: /MAGIC/CPLD/SYNC -> unconnected-(J23-Pad12)
- J23 pad 13: /MAGIC/CPLD/DIAG -> /MAGIC/CPLD/GRAPHICS
- J23 pad 15: /MAGIC/CPLD/GRAPHICS -> /MAGIC/CPLD/~{RD_STROBE}
- J23 pad 16: /MAGIC/CPLD/~{NMI} -> /MAGIC/CPLD/~{RAM_CE}
- J23 pad 17: /CPU \ RAM/D3 -> /MAGIC/CPLD/~{WR_STROBE}
- J23 pad 18: /CPU \ RAM/D7 -> /MAGIC/CPLD/~{VP}
- J23 pad 19: /CPU \ RAM/D2 -> /MAGIC/CPLD/RDY
- J23 pad 20: /CPU \ RAM/D6 -> /MAGIC/~{RES}
- J23 pad 21: /CPU \ RAM/D1 -> /MAGIC/CPLD/~{SO}
- J23 pad 22: /CPU \ RAM/D5 -> /MAGIC/CPLD/~{IRQ}
- J23 pad 23: /CPU \ RAM/D0 -> /MAGIC/CPLD/~{ML}
- J23 pad 24: /CPU \ RAM/D4 -> /MAGIC/CPLD/BE
- J23 pad 25: /MAGIC/R~{W} -> /MAGIC/CPLD/~{NMI}
- J23 pad 26: GND -> /MAGIC/CPLD/SYNC
- J23 pad 28: +3V3 -> GND
- J23 pad 3: /MAGIC/CPLD/P73_LP -> /MAGIC/CPLD/AUDIO
- J23 pad 4: /CPU \ RAM/RAM_A10 -> unconnected-(J23-Pad4)
- J23 pad 5: /CPU \ RAM/RAM_A11 -> unconnected-(J23-Pad5)
- J23 pad 6: /MAGIC/CPLD/~{WR_STROBE} -> unconnected-(J23-Pad6)
- J23 pad 7: /MAGIC/CPLD/~{RAM_CE} -> unconnected-(J23-Pad7)
- J23 pad 8: /MAGIC/CPLD/P80_GND -> unconnected-(J23-Pad8)
- J23 pad 9: /MAGIC/CPLD/P81_1V2 -> unconnected-(J23-Pad9)
- J24 pad 1: GND -> /MAGIC/CPLD/A0
- J24 pad 10: /CPU \ RAM/A11 -> /MAGIC/CPLD/A16
- J24 pad 11: /CPU \ RAM/A4 -> /MAGIC/CPLD/A5
- J24 pad 12: /CPU \ RAM/A12 -> /MAGIC/CPLD/D0
- J24 pad 13: /CPU \ RAM/A5 -> /MAGIC/CPLD/A6
- J24 pad 14: /CPU \ RAM/A13 -> /MAGIC/CPLD/D1
- J24 pad 15: /CPU \ RAM/A6 -> /MAGIC/CPLD/A7
- J24 pad 16: /CPU \ RAM/A14 -> /MAGIC/CPLD/D2
- J24 pad 17: /CPU \ RAM/A7 -> /MAGIC/CPLD/A8
- J24 pad 18: /CPU \ RAM/A15 -> /MAGIC/CPLD/D3
- J24 pad 19: /MAGIC/~{VIA_CS} -> /MAGIC/CPLD/A9
- J24 pad 2: GND -> /MAGIC/CPLD/A12
- J24 pad 20: /CPU \ RAM/A16 -> /MAGIC/CPLD/D4
- J24 pad 21: /MAGIC/~{PIA1_CS} -> /MAGIC/CPLD/A10
- J24 pad 22: /MAGIC/~{PIA2_CS} -> /MAGIC/CPLD/D5
- J24 pad 23: /MAGIC/CPLD/~{IRQ} -> /MAGIC/CPLD/RAM_A10
- J24 pad 24: /MAGIC/~{IO_OE} -> /MAGIC/CPLD/D6
- J24 pad 25: /MAGIC/~{RES} -> /MAGIC/CPLD/A11
- J24 pad 26: GND -> /MAGIC/CPLD/D7
- J24 pad 27: GND -> /MAGIC/CPLD/RAM_A11
- J24 pad 28: +3V3 -> /MAGIC/R~{W}
- J24 pad 3: /CPU \ RAM/A0 -> /MAGIC/CPLD/A1
- J24 pad 4: /CPU \ RAM/A8 -> /MAGIC/CPLD/A13
- J24 pad 5: /CPU \ RAM/A1 -> /MAGIC/CPLD/A2
- J24 pad 6: /CPU \ RAM/A9 -> /MAGIC/CPLD/A14
- J24 pad 7: /CPU \ RAM/A2 -> /MAGIC/CPLD/A3
- J24 pad 8: /CPU \ RAM/A10 -> /MAGIC/CPLD/A15
- J24 pad 9: /CPU \ RAM/A3 -> /MAGIC/CPLD/A4
- RV1 pad 2: Net-(J1-PadRN) -> Net-(RV1-Pad2)
- U11 pad 1: unconnected-(U11-Pad1) -> /CPU \ RAM/~{VP}
- U11 pad 38: +3V3 -> /CPU \ RAM/~{SO}
- U11 pad 5: unconnected-(U11-Pad5) -> /CPU \ RAM/~{ML}
- U12 pad 12: /CPU \ RAM/A12 -> /CPU \ RAM/RAM_A10
- U12 pad 13: /CPU \ RAM/D5 -> /CPU \ RAM/D1
- U12 pad 14: /CPU \ RAM/D6 -> /CPU \ RAM/D3
- U12 pad 15: /CPU \ RAM/D7 -> /CPU \ RAM/D5
- U12 pad 17: /CPU \ RAM/D4 -> /CPU \ RAM/D7
- U12 pad 18: /CPU \ RAM/D3 -> /CPU \ RAM/D6
- U12 pad 19: /CPU \ RAM/D2 -> /CPU \ RAM/D4
- U12 pad 20: /CPU \ RAM/D1 -> /CPU \ RAM/D2
- U12 pad 23: /CPU \ RAM/A13 -> /CPU \ RAM/RAM_A11
- U12 pad 27: /CPU \ RAM/A16 -> /CPU \ RAM/A12
- U12 pad 28: /CPU \ RAM/RAM_A11 -> /CPU \ RAM/A13
- U12 pad 31: /CPU \ RAM/RAM_A10 -> /CPU \ RAM/A16
- U20 pad 19: /MAGIC/~{VIDEO} -> /MAGIC/HORIZ
- U20 pad 21: /MAGIC/HORIZ -> /MAGIC/~{VIDEO}
- U20 pad 3: /MAGIC/BHORIZ -> /MAGIC/~{BVIDEO}
- U20 pad 5: /MAGIC/~{BVIDEO} -> /MAGIC/BHORIZ
Routing:
- net GND: track 285.4 -> 2061.8 mm, vias 9 -> 24
- net +5V: track 22.3 -> 708.0 mm, vias 5 -> 10
- net /CASS/CASS_WRITE: track 0.00 -> 324.1 mm, vias 1 -> 5
- net +6V: track 0.00 -> 270.7 mm
- net +3V3: track 35.5 -> 288.7 mm, vias 3 -> 5
- net /CPU \ RAM/D0: track 0.00 -> 234.7 mm, vias 0 -> 2
- net /IEEE/SRQ: track 0.00 -> 227.7 mm, vias 0 -> 5
- net /IO/BVERT: track 0.00 -> 227.5 mm, vias 0 -> 4
- net /CPU \ RAM/D4: track 0.00 -> 221.4 mm, vias 0 -> 5
- net /IEEE/EOI: track 0.00 -> 221.3 mm, vias 0 -> 6
- net /IO/VIA_CB2: track 0.00 -> 191.2 mm, vias 0 -> 3
- net /MAGIC/CPLD/~{IRQ}: track 0.00 -> 187.8 mm, vias 0 -> 4
- net /MAGIC/BHORIZ: track 0.00 -> 185.7 mm, vias 0 -> 3
- net /MAGIC/~{RES}: track 0.00 -> 171.9 mm, vias 0 -> 1
- net /MAGIC/~{BVIDEO}: track 0.00 -> 168.6 mm, vias 0 -> 1
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- added copper zone on F.Cu, net Net-(D5-Pad1)
Other:
- board size 262.9 x 107.9 mm -> 262.9 x 95.2 mm
- board text added: "CCK"
- board text added: "CDI0"
- board text added: "CDI1"
- board text added: "CDONE"
- board text added: "TCK"
- board text added: "TDI"
- board text added: "TDO"
- board text added: "TMS"
- board text added: "~{CRESET}"
- board text added: "~{ML}"
- board text added: "~{RDY}"
- board text added: "~{SO}"
- board text added: "~{SS}"
- board text added: "~{VP}"
- board text removed: "22"
- board text removed: "26"
- board text removed: "27"
- board text removed: "5V"
- board text removed: "73"
- board text removed: "80"
- board text removed: "81"
- board text removed: "VIDEO"
- board text removed: "~{DON}"
- board text removed: "~{L2}"
- board text removed: "~{L4}"
- board text removed: "~{L5}"
- board text removed: "~{PEN}"

Commit message: hw: routing (excluding MCU)
Parts:
- added C60: 1u, Capacitor_SMD:C_0402_1005Metric, F.Cu at (-68.7, 51.6)
- added C61: 100n, Capacitor_SMD:C_0402_1005Metric, F.Cu at (-67.7, 51.6)
- added C62: 100n, Capacitor_SMD:C_0402_1005Metric, F.Cu at (-54.0, 34.6)
- added C63: 100n, Capacitor_SMD:C_0402_1005Metric, F.Cu at (-70.5, 21.0)
- added C64: 100n, Capacitor_SMD:C_0402_1005Metric, F.Cu at (-84.5, 39.3)
- added C65: 10n, Capacitor_SMD:C_0402_1005Metric, F.Cu at (-70.0, 51.6)
- added C66: 10n, Capacitor_SMD:C_0402_1005Metric, F.Cu at (-54.0, 38.8)
- added C67: 10n, Capacitor_SMD:C_0402_1005Metric, F.Cu at (-84.5, 33.4)
- added C68: 10n, Capacitor_SMD:C_0402_1005Metric, F.Cu at (-66.3, 21.0)
- added C69: 1u, Capacitor_SMD:C_0402_1005Metric, F.Cu at (-54.0, 33.5)
- added C70: 1u, Capacitor_SMD:C_0402_1005Metric, F.Cu at (-84.5, 36.6)
- added C71: 100n, Capacitor_SMD:C_0402_1005Metric, F.Cu at (-67.3, 21.0)
- added C72: 100n, Capacitor_SMD:C_0402_1005Metric, F.Cu at (-54.0, 35.6)
- added C73: 100n, Capacitor_SMD:C_0402_1005Metric, F.Cu at (-73.8, 21.0)
- added C74: 100n, Capacitor_SMD:C_0402_1005Metric, F.Cu at (-68.4, 21.0)
- added C75: 100n, Capacitor_SMD:C_0402_1005Metric, F.Cu at (-61.0, 51.6)
- added C76: 100n, Capacitor_SMD:C_0402_1005Metric, F.Cu at (-84.5, 38.2)
- added C77: 10n, Capacitor_SMD:C_0402_1005Metric, F.Cu at (-84.5, 35.2)
- added C78: 10n, Capacitor_SMD:C_0402_1005Metric, F.Cu at (-72.8, 21.0)
- added C79: 10n, Capacitor_SMD:C_0402_1005Metric, F.Cu at (-71.5, 51.6)
- added C80: 10n, Capacitor_SMD:C_0402_1005Metric, F.Cu at (-54.0, 39.9)
- added J11: 9V POWER, Connector_PinHeader_2.54mm:PinHeader_1x02_P2.54mm_Vertical, F.Cu at (-233.4, 21.0)
- added R34: 12k 1%, Resistor_SMD:R_0402_1005Metric, F.Cu at (-54.0, 27.6)
- added R35: 5k1, Resistor_SMD:R_0402_1005Metric, F.Cu at (5.35, 73.5)
- added R36: 5k1, Resistor_SMD:R_0402_1005Metric, F.Cu at (4.55, 66.8)
- added X1: 50MHZ, Crystal:Crystal_SMD_3225-4Pin_3.2x2.5mm, F.Cu at (-70.7, 54.4)
- C36: value 22u -> 22u 25V
- C54, C55: value 10u -> 10u 16V
- D1: value RED LED -> RED_9V
- J14: value USB -> USB_C_Receptacle_USB2.0; footprint JLCPCB:MICRO-USB_MICRO-USB-17 -> JLCPCB:USB-C_SMD-TYPE-C-31-M-12
- JP10: moved to B.Cu
- SW3: footprint SamacSys_Parts:TL4115AF160Q -> JLCPCB:KEY-TH_SKHLLBA010
- SW5: footprint Button_Switch_THT:SW_PUSH_6mm -> JLCPCB:SW-TH_L6.0-W3.5-P6.50
- moved C58 62.2 mm to (-84.5, 44.6), turned to 180 degrees
- moved R27 56.9 mm to (-84.5, 28.5), turned to 180 degrees
- moved FB1 53.5 mm to (-84.2, 27.2), turned to 180 degrees
- moved C59 52.7 mm to (-73.3, 53.3), turned to 90 degrees
- moved C56 48.6 mm to (-84.5, 25.9)
- moved R33 42.1 mm to (-49.9, 77.4), turned to -90 degrees
- moved D8 41.4 mm to (-43.8, 73.7)
- moved R32 41.4 mm to (-49.9, 75.4), turned to -90 degrees
- moved R29 40.4 mm to (-43.8, 72.3), turned to 180 degrees
- moved R30 38.5 mm to (-49.9, 73.4), turned to -90 degrees
- moved Q4 38.2 mm to (-47.4, 73.8)
- moved R31 35.5 mm to (-46.4, 76.8)
- moved D9 35.5 mm to (-43.8, 76.8)
- moved JP10 30.7 mm to (-70.7, 54.4), turned to 180 degrees
- moved R28 29.7 mm to (-67.5, 53.2), turned to 180 degrees
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Connections:
- net /MAGIC/CPLD/CDONE renamed /MAGIC/FPGA/CDONE
- net /MAGIC/CPLD/NSTATUS renamed /MAGIC/FPGA/NSTATUS
- net /MAGIC/CPLD/TCK renamed /MAGIC/FPGA/TCK
- net /MAGIC/CPLD/TDI renamed /MAGIC/FPGA/TDI
- net /MAGIC/CPLD/TDO renamed /MAGIC/FPGA/TDO
- net /MAGIC/CPLD/TMS renamed /MAGIC/FPGA/TMS
- C24 pad 1: /MAGIC/CPLD/~{NMI} -> /MAGIC/FPGA/~{NMI}
- C31 pad 1: /MAGIC/CPLD/AUDIO -> /MAGIC/FPGA/AUDIO
- J13 pad 3: /MAGIC/MCU/SPI1_TX -> /MAGIC/FPGA/SPI1_TX
- J13 pad 7: /MAGIC/MCU/SPI1_RX -> /MAGIC/FPGA/SPI1_RX
- J21 pad 10: /MAGIC/CPLD/CLK_50 -> /MAGIC/~{IO_OE}
- J21 pad 11: /MAGIC/~{IO_OE} -> unconnected-(J21-Pad11)
- J21 pad 15: unconnected-(J21-Pad15) -> /MAGIC/FPGA/MCU_CLK
- J21 pad 16: unconnected-(J21-Pad16) -> /MAGIC/FPGA/CLK_50
- J22 pad 1: GND -> /MAGIC/FPGA/SPI1_TX
- J22 pad 10: /MAGIC/CPLD/CDI0 -> /MAGIC/FPGA/CDI0
- J22 pad 12: /MAGIC/CPLD/CDI1 -> /MAGIC/FPGA/CDI1
- J22 pad 14: /MAGIC/CPLD/~{SS} -> /MAGIC/FPGA/~{SS}
- J22 pad 15: unconnected-(J22-Pad15) -> /MAGIC/FPGA/CBUS1
- J22 pad 16: /MAGIC/CPLD/~{CRESET} -> /MAGIC/FPGA/~{CRESET}
- J22 pad 17: unconnected-(J22-Pad17) -> /MAGIC/FPGA/CBUS0
- J22 pad 19: unconnected-(J22-Pad19) -> /MAGIC/FPGA/MCU_CEC
- J22 pad 21: unconnected-(J22-Pad21) -> /MAGIC/FPGA/CSI
- J22 pad 23: unconnected-(J22-Pad23) -> /MAGIC/FPGA/GP27
- J22 pad 25: unconnected-(J22-Pad25) -> /MAGIC/FPGA/I2C0_SCL
- J22 pad 27: unconnected-(J22-Pad27) -> /MAGIC/FPGA/I2C0_SDA
- J22 pad 3: unconnected-(J22-Pad3) -> /MAGIC/FPGA/SPI1_RX
- J22 pad 5: unconnected-(J22-Pad5) -> /MAGIC/FPGA/SPI1_~{CS}
- J22 pad 7: unconnected-(J22-Pad7) -> /MAGIC/FPGA/SPI1_SCK
- J22 pad 8: /MAGIC/CPLD/CCK -> /MAGIC/FPGA/CCK
- J22 pad 9: unconnected-(J22-Pad9) -> /MAGIC/FPGA/CBUS2
- J23 pad 10: unconnected-(J23-Pad10) -> /MAGIC/FPGA/S1
- J23 pad 11: /MAGIC/CPLD/DIAG -> unconnected-(J23-Pad11)
- J23 pad 12: unconnected-(J23-Pad12) -> /MAGIC/FPGA/DIAG
- J23 pad 13: /MAGIC/CPLD/GRAPHICS -> /MAGIC/FPGA/GRAPHICS
- J23 pad 14: /MAGIC/CPLD/VIA_CB2 -> /MAGIC/FPGA/VIA_CB2
- J23 pad 15: /MAGIC/CPLD/~{RD_STROBE} -> /MAGIC/FPGA/~{RD_STROBE}
- J23 pad 16: /MAGIC/CPLD/~{RAM_CE} -> /MAGIC/FPGA/~{RAM_CE}
- J23 pad 17: /MAGIC/CPLD/~{WR_STROBE} -> /MAGIC/FPGA/~{WR_STROBE}
- J23 pad 18: /MAGIC/CPLD/~{VP} -> /MAGIC/FPGA/~{VP}
- J23 pad 19: /MAGIC/CPLD/RDY -> /MAGIC/FPGA/RDY
- J23 pad 21: /MAGIC/CPLD/~{SO} -> /MAGIC/FPGA/~{SO}
- J23 pad 22: /MAGIC/CPLD/~{IRQ} -> /MAGIC/FPGA/~{IRQ}
- J23 pad 23: /MAGIC/CPLD/~{ML} -> /MAGIC/FPGA/~{ML}
- J23 pad 24: /MAGIC/CPLD/BE -> /MAGIC/FPGA/BE
- J23 pad 25: /MAGIC/CPLD/~{NMI} -> /MAGIC/FPGA/~{NMI}
- J23 pad 26: /MAGIC/CPLD/SYNC -> /MAGIC/FPGA/SYNC
- J23 pad 3: /MAGIC/CPLD/AUDIO -> unconnected-(J23-Pad3)
- J23 pad 4: unconnected-(J23-Pad4) -> /MAGIC/FPGA/AUDIO
- J23 pad 6: unconnected-(J23-Pad6) -> /MAGIC/FPGA/S3
- J23 pad 8: unconnected-(J23-Pad8) -> /MAGIC/FPGA/S2
- J24 pad 1: /MAGIC/CPLD/A0 -> /CPU \ RAM/A0
- J24 pad 10: /MAGIC/CPLD/A16 -> /CPU \ RAM/A16
- J24 pad 11: /MAGIC/CPLD/A5 -> /CPU \ RAM/A5
- J24 pad 12: /MAGIC/CPLD/D0 -> /CPU \ RAM/D0
- J24 pad 13: /MAGIC/CPLD/A6 -> /CPU \ RAM/A6
- J24 pad 14: /MAGIC/CPLD/D1 -> /CPU \ RAM/D1
- J24 pad 15: /MAGIC/CPLD/A7 -> /CPU \ RAM/A7
- J24 pad 16: /MAGIC/CPLD/D2 -> /CPU \ RAM/D2
- J24 pad 17: /MAGIC/CPLD/A8 -> /CPU \ RAM/A8
- J24 pad 18: /MAGIC/CPLD/D3 -> /CPU \ RAM/D3
- J24 pad 19: /MAGIC/CPLD/A9 -> /CPU \ RAM/A9
- J24 pad 2: /MAGIC/CPLD/A12 -> /CPU \ RAM/A12
- J24 pad 20: /MAGIC/CPLD/D4 -> /CPU \ RAM/D4
- J24 pad 21: /MAGIC/CPLD/A10 -> /CPU \ RAM/A10
- J24 pad 22: /MAGIC/CPLD/D5 -> /CPU \ RAM/D5
- J24 pad 23: /MAGIC/CPLD/RAM_A10 -> /CPU \ RAM/RAM_A10
- J24 pad 24: /MAGIC/CPLD/D6 -> /CPU \ RAM/D6
- J24 pad 25: /MAGIC/CPLD/A11 -> /CPU \ RAM/A11
- J24 pad 26: /MAGIC/CPLD/D7 -> /CPU \ RAM/D7
- J24 pad 27: /MAGIC/CPLD/RAM_A11 -> /CPU \ RAM/RAM_A11
- J24 pad 3: /MAGIC/CPLD/A1 -> /CPU \ RAM/A1
- J24 pad 4: /MAGIC/CPLD/A13 -> /CPU \ RAM/A13
- J24 pad 5: /MAGIC/CPLD/A2 -> /CPU \ RAM/A2
- J24 pad 6: /MAGIC/CPLD/A14 -> /CPU \ RAM/A14
- J24 pad 7: /MAGIC/CPLD/A3 -> /CPU \ RAM/A3
- J24 pad 8: /MAGIC/CPLD/A15 -> /CPU \ RAM/A15
- J24 pad 9: /MAGIC/CPLD/A4 -> /CPU \ RAM/A4
- R20 pad 2: /MAGIC/MCU/SPI1_RX -> /MAGIC/FPGA/SPI1_RX
- R28 pad 1: /MAGIC/CPLD/CLK_50 -> /MAGIC/FPGA/CLK_50
- R33 pad 2: /MAGIC/CPLD/~{CRESET} -> /MAGIC/FPGA/~{CRESET}
- R38 pad 2: /MAGIC/CPLD/~{NMI} -> /MAGIC/FPGA/~{NMI}
- R39 pad 2: /MAGIC/CPLD/~{IRQ} -> /MAGIC/FPGA/~{IRQ}
- R40 pad 1: /MAGIC/CPLD/RDY -> /MAGIC/FPGA/RDY
- R52 pad 1: /MAGIC/CPLD/GRAPHICS -> /MAGIC/FPGA/GRAPHICS
- R54 pad 1: /MAGIC/CPLD/GRAPHICS -> /MAGIC/FPGA/GRAPHICS
- R55 pad 1: /MAGIC/CPLD/DIAG -> /MAGIC/FPGA/DIAG
- R57 pad 1: /MAGIC/CPLD/VIA_CB2 -> /MAGIC/FPGA/VIA_CB2
- R58 pad 1: /MAGIC/CPLD/VIA_CB2 -> /MAGIC/FPGA/VIA_CB2
- R60 pad 1: /MAGIC/CPLD/DIAG -> /MAGIC/FPGA/DIAG
- SW1 pad 2: /MAGIC/CPLD/~{NMI} -> /MAGIC/FPGA/~{NMI}
- U11 pad 36: /MAGIC/CPLD/BE -> /MAGIC/FPGA/BE
- U11 pad 4: /MAGIC/CPLD/~{IRQ} -> /MAGIC/FPGA/~{IRQ}
- U11 pad 6: /MAGIC/CPLD/~{NMI} -> /MAGIC/FPGA/~{NMI}
- U11 pad 7: /MAGIC/CPLD/SYNC -> /MAGIC/FPGA/SYNC
- U12 pad 22: /MAGIC/CPLD/~{RAM_CE} -> /MAGIC/FPGA/~{RAM_CE}
- U12 pad 24: /MAGIC/CPLD/~{RD_STROBE} -> /MAGIC/FPGA/~{RD_STROBE}
- U12 pad 25: /CPU \ RAM/A14 -> /CPU \ RAM/A16
- U12 pad 27: /CPU \ RAM/A12 -> /CPU \ RAM/A14
- U12 pad 29: /MAGIC/CPLD/~{WR_STROBE} -> /MAGIC/FPGA/~{WR_STROBE}
- U12 pad 31: /CPU \ RAM/A16 -> /CPU \ RAM/A12
- U14 pad 13: /MAGIC/MCU/MCU_CEC -> /MAGIC/FPGA/CBUS2
- U14 pad 14: /MAGIC/MCU/SPI1_~{READY} -> /MAGIC/FPGA/MCU_CLK
- U14 pad 15: /MAGIC/MCU/SPI1_RX -> /MAGIC/FPGA/SPI1_RX
- U14 pad 16: /MAGIC/MCU/SPI1_~{CS} -> /MAGIC/FPGA/SPI1_~{CS}
- U14 pad 17: /MAGIC/MCU/SPI1_SCLK -> /MAGIC/FPGA/SPI1_SCK
- U14 pad 18: /MAGIC/MCU/SPI1_TX -> /MAGIC/FPGA/SPI1_TX
- U14 pad 36: /MAGIC/MCU/GP24 -> /MAGIC/MCU/MCU_CEC
- U14 pad 38: /MAGIC/MCU/GP26 -> /MAGIC/FPGA/~{CRESET}
- U14 pad 6: /MAGIC/MCU/SPI0_RX -> /MAGIC/FPGA/CDI1
- U14 pad 7: /MAGIC/MCU/SPI0_~{CS} -> /MAGIC/FPGA/~{SS}
- U14 pad 8: /MAGIC/MCU/SPI0_SCLK -> /MAGIC/FPGA/CCK
- U14 pad 9: /MAGIC/MCU/SPI0_TX -> /MAGIC/FPGA/CDI0
- U21 pad 10: unconnected-(U21-Pad10) -> /MAGIC/FPGA/SPI1_~{CS}
- U21 pad 100: unconnected-(U21-Pad100) -> /CPU \ RAM/A8
- U21 pad 101: unconnected-(U21-Pad101) -> /CPU \ RAM/D3
- U21 pad 102: unconnected-(U21-Pad102) -> /CPU \ RAM/A9
- U21 pad 103: unconnected-(U21-Pad103) -> /CPU \ RAM/D4
- U21 pad 105: unconnected-(U21-Pad105) -> /CPU \ RAM/A10
- U21 pad 106: unconnected-(U21-Pad106) -> /CPU \ RAM/D5
- U21 pad 109: unconnected-(U21-Pad109) -> /CPU \ RAM/RAM_A10
- U21 pad 11: unconnected-(U21-Pad11) -> /MAGIC/FPGA/SPI1_SCK
- U21 pad 110: unconnected-(U21-Pad110) -> /CPU \ RAM/D6
- U21 pad 111: unconnected-(U21-Pad111) -> /CPU \ RAM/A11
- U21 pad 112: unconnected-(U21-Pad112) -> /CPU \ RAM/D7
- U21 pad 113: unconnected-(U21-Pad113) -> /CPU \ RAM/RAM_A11
- U21 pad 114: unconnected-(U21-Pad114) -> /MAGIC/~{VIDEO}
- U21 pad 115: unconnected-(U21-Pad115) -> /MAGIC/~{PIA1_CS}
- U21 pad 116: unconnected-(U21-Pad116) -> /MAGIC/VERT
- U21 pad 117: unconnected-(U21-Pad117) -> /MAGIC/~{VIA_CS}
- U21 pad 118: unconnected-(U21-Pad118) -> /MAGIC/HORIZ
- U21 pad 119: unconnected-(U21-Pad119) -> /MAGIC/~{PIA2_CS}
- U21 pad 123: unconnected-(U21-Pad123) -> /MAGIC/~{IO_OE}
- U21 pad 131: unconnected-(U21-Pad131) -> /MAGIC/FPGA/CLK_50
- U21 pad 132: unconnected-(U21-Pad132) -> /MAGIC/FPGA/MCU_CLK
- U21 pad 28: /MAGIC/CPLD/CDI1 -> /MAGIC/FPGA/CDI1
- U21 pad 29: /MAGIC/CPLD/CDI0 -> /MAGIC/FPGA/CDI0
- U21 pad 30: /MAGIC/CPLD/CCK -> /MAGIC/FPGA/CCK
- U21 pad 31: /MAGIC/CPLD/~{SS} -> /MAGIC/FPGA/~{SS}
- U21 pad 32: /MAGIC/CPLD/CSI -> /MAGIC/FPGA/CSI
- U21 pad 35: /MAGIC/CPLD/~{CRESET} -> /MAGIC/FPGA/~{CRESET}
- U21 pad 36: unconnected-(U21-Pad36) -> Net-(R34-Pad2)
- U21 pad 38: unconnected-(U21-Pad38) -> /MAGIC/FPGA/AUDIO
- U21 pad 39: unconnected-(U21-Pad39) -> /MAGIC/FPGA/S3
- U21 pad 40: unconnected-(U21-Pad40) -> /MAGIC/FPGA/S2
- U21 pad 41: unconnected-(U21-Pad41) -> /MAGIC/FPGA/S1
- U21 pad 42: unconnected-(U21-Pad42) -> /MAGIC/FPGA/DIAG
- U21 pad 43: unconnected-(U21-Pad43) -> /MAGIC/FPGA/GRAPHICS
- U21 pad 45: unconnected-(U21-Pad45) -> /MAGIC/FPGA/VIA_CB2
- U21 pad 46: unconnected-(U21-Pad46) -> /MAGIC/FPGA/~{RD_STROBE}
- U21 pad 47: unconnected-(U21-Pad47) -> /MAGIC/FPGA/~{RAM_CE}
- U21 pad 48: unconnected-(U21-Pad48) -> /MAGIC/FPGA/~{WR_STROBE}
- U21 pad 53: unconnected-(U21-Pad53) -> /MAGIC/FPGA/~{VP}
- U21 pad 54: unconnected-(U21-Pad54) -> /MAGIC/FPGA/RDY
- U21 pad 55: unconnected-(U21-Pad55) -> /MAGIC/FPGA/~{SO}
- U21 pad 56: unconnected-(U21-Pad56) -> /MAGIC/FPGA/~{IRQ}
- U21 pad 58: unconnected-(U21-Pad58) -> /MAGIC/FPGA/~{ML}
- U21 pad 59: unconnected-(U21-Pad59) -> /MAGIC/FPGA/BE
- U21 pad 60: unconnected-(U21-Pad60) -> /MAGIC/FPGA/~{NMI}
- U21 pad 61: unconnected-(U21-Pad61) -> /MAGIC/FPGA/SYNC
- U21 pad 65: unconnected-(U21-Pad65) -> /CPU \ RAM/A0
- U21 pad 66: unconnected-(U21-Pad66) -> /CPU \ RAM/A12
- U21 pad 67: unconnected-(U21-Pad67) -> /CPU \ RAM/A1
- U21 pad 68: unconnected-(U21-Pad68) -> /CPU \ RAM/A13
- U21 pad 69: unconnected-(U21-Pad69) -> /CPU \ RAM/A2
- U21 pad 7: unconnected-(U21-Pad7) -> /MAGIC/FPGA/SPI1_TX
- U21 pad 70: unconnected-(U21-Pad70) -> /CPU \ RAM/A14
- U21 pad 71: unconnected-(U21-Pad71) -> /CPU \ RAM/A3
- U21 pad 72: unconnected-(U21-Pad72) -> /CPU \ RAM/A15
- U21 pad 76: unconnected-(U21-Pad76) -> /CPU \ RAM/A4
- U21 pad 77: unconnected-(U21-Pad77) -> /CPU \ RAM/A16
- U21 pad 78: /MAGIC/CPLD/CBUS0 -> /MAGIC/FPGA/CBUS0
- U21 pad 79: /MAGIC/CPLD/CBUS1 -> /MAGIC/FPGA/CBUS1
- U21 pad 8: unconnected-(U21-Pad8) -> /MAGIC/FPGA/SPI1_RX
- U21 pad 80: /MAGIC/CPLD/CBUS2 -> /MAGIC/FPGA/CBUS2
- U21 pad 81: unconnected-(U21-Pad81) -> /CPU \ RAM/A5
- U21 pad 82: unconnected-(U21-Pad82) -> /CPU \ RAM/D0
- U21 pad 83: unconnected-(U21-Pad83) -> /CPU \ RAM/A6
- U21 pad 84: unconnected-(U21-Pad84) -> /CPU \ RAM/D1
- U21 pad 86: unconnected-(U21-Pad86) -> /CPU \ RAM/A7
- U21 pad 87: unconnected-(U21-Pad87) -> /CPU \ RAM/D2
- U21 pad 97: unconnected-(U21-Pad97) -> /MAGIC/ϕ2
- U21 pad 98: unconnected-(U21-Pad98) -> /MAGIC/~{RES}
- U21 pad 99: unconnected-(U21-Pad99) -> /MAGIC/R~{W}
- U7 pad 37: /MAGIC/CPLD/~{IRQ} -> /MAGIC/FPGA/~{IRQ}
- U7 pad 38: /MAGIC/CPLD/~{IRQ} -> /MAGIC/FPGA/~{IRQ}
- U8 pad 37: /MAGIC/CPLD/~{IRQ} -> /MAGIC/FPGA/~{IRQ}
- U8 pad 38: /MAGIC/CPLD/~{IRQ} -> /MAGIC/FPGA/~{IRQ}
- U9 pad 21: /MAGIC/CPLD/~{IRQ} -> /MAGIC/FPGA/~{IRQ}
Routing:
- net GND: track 2061.8 -> 1784.8 mm, vias 24 -> 39
- net /CASS/CASS_A_READ: track 0.00 -> 215.5 mm, vias 0 -> 2
- net +3V3: track 288.7 -> 503.1 mm, vias 5 -> 9
- net /CASS/CASS_A_~{SWITCH}: track 0.00 -> 210.8 mm, vias 0 -> 2
- net /CASS/CASS_A_~{MOTOR}: track 0.00 -> 204.3 mm, vias 0 -> 1
- net /MAGIC/FPGA/~{IRQ}: track 0.00 -> 201.0 mm, vias 0 -> 3
- net /MAGIC/CPLD/~{IRQ}: track 187.8 -> 0.00 mm, vias 4 -> 0
- net +5V: track 708.0 -> 885.1 mm, vias 10 -> 11
- net VCORE: track 0.00 -> 168.6 mm, vias 0 -> 5
- net /CPU \ RAM/D0: track 234.7 -> 80.0 mm, vias 2 -> 0
- net /CPU \ RAM/D4: track 221.4 -> 72.7 mm, vias 5 -> 0
- net /MAGIC/FPGA/~{NMI}: track 0.00 -> 147.8 mm, vias 0 -> 1
- net /MAGIC/CPLD/~{NMI}: track 147.6 -> 0.00 mm
- net /MAGIC/FPGA/SPI1_RX: track 0.00 -> 131.9 mm, vias 0 -> 2
- net /CPU \ RAM/D1: track 0.00 -> 102.2 mm, vias 0 -> 2
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- removed copper zone on F.Cu, net +5V
- removed copper zone on F.Cu, net GND
Other:
- outline, holes or cut-outs redrawn
- board text added: "9V"
- board text added: "RX"
- board text added: "SCK"
- board text added: "TX"
- board text added: "~{CRST}"
- board text added: "~{CS}"
- board text removed: "CCK"
- board text removed: "CDI0"
- board text removed: "CDI1"
- board text removed: "CLK"
- board text removed: "~{CRESET}"
- board text removed: "~{SS}"

Commit message: hw: routed, but trace sizes need to be reviewed/fixed
Parts:
- added C81: 47u 10V, Capacitor_SMD:C_1206_3216Metric, F.Cu at (-41.0, 5.87)
- added J16: MCU_EXT, Connector_PinHeader_2.54mm:PinHeader_1x05_P2.54mm_Vertical, F.Cu at (-13.8, 75.7)
- added J17: BOOTSEL, Connector_PinHeader_2.54mm:PinHeader_1x02_P2.54mm_Vertical, F.Cu at (-4.75, 42.2)
- added JP11: FPGA PWR, Jumper:SolderJumper-3_P1.3mm_Bridged12_RoundedPad1.0x1.5mm, B.Cu at (-36.0, 5.90)
- added R37: 470, Resistor_SMD:R_0402_1005Metric, F.Cu at (-39.2, 5.87)
- added R48: 10k, Resistor_SMD:R_0402_1005Metric, F.Cu at (-54.6, 23.5)
- added R51: 10k, Resistor_SMD:R_0402_1005Metric, F.Cu at (-58.0, 22.7)
- added R63: 10k, Resistor_SMD:R_0402_1005Metric, F.Cu at (-58.8, 22.0)
- added SW2: MCU_RESET, Button_Switch_THT:SW_PUSH_6mm, F.Cu at (-37.9, 76.0)
- D6: value RED LED -> CASS_A_RED
- D7: value RED LED -> CASS_B_RED
- J14: value USB_C_Receptacle_USB2.0 -> USB2.0_HOST_TYPE_C
- J2: footprint PET:Keyboard_Header_1x20_P2.54mm_Vertical -> Retrocomputing:CBM_PET_KEYBOARD_KEYED_20P
- Q1, Q3: footprint PET:SOT-23-3L -> JLCPCB:SOT-23_L2.9-W1.3-P1.90-LS2.4-BR
- SW1: value NMI -> RESET
- SW3: value RUN -> MENU
- SW4: value RESET -> NMI
- SW5: value BOOTSEL -> CONFIG; footprint JLCPCB:SW-TH_L6.0-W3.5-P6.50 -> Button_Switch_THT:SW_DIP_SPSTx04_Slide_6.7x11.72mm_W7.62mm_P2.54mm_LowProfile
- moved SW5 67.8 mm to (-72.6, 74.0)
- moved R18 39.8 mm to (-30.7, 68.5), turned to -90 degrees
- moved R7 16.2 mm to (-29.6, 69.5), turned to -90 degrees
- moved R16 15.7 mm to (-28.3, 70.8), turned to -90 degrees
- moved JP7 10.9 mm to (-17.4, 68.4), turned to 90 degrees
- moved D9 9.45 mm to (-48.6, 85.0)
- moved D8 9.43 mm to (-48.6, 81.8)
- moved R20 8.38 mm to (-3.55, 54.9), turned to -90 degrees
- moved R29 6.70 mm to (-47.5, 77.9), turned to 90 degrees
- moved R31 5.72 mm to (-52.0, 77.9), turned to 90 degrees
- moved D7 5.21 mm to (-186.0, 72.9)
- moved R19 4.61 mm to (-2.91, 59.9), turned to -45 degrees
- moved Q4 3.89 mm to (-49.8, 76.9), turned to -90 degrees
- moved R32 3.61 mm to (-48.8, 72.0), turned to 90 degrees
- moved R33 3.53 mm to (-50.7, 74.0), turned to 90 degrees
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Connections:
- net Net-(C57-Pad1) renamed /POWER/VCCA
- net Net-(R27-Pad1) renamed /MAGIC/FPGA/~{TEST}
- C24 pad 1: /MAGIC/FPGA/~{NMI} -> /MAGIC/~{RES}
- C25 pad 1: /MAGIC/~{RES} -> /MAGIC/FPGA/~{NMI}
- C55 pad 1: VCORE -> Net-(U17-Pad2)
- J13 pad 5: /MAGIC/MCU/SPI1_SCLK -> /MAGIC/FPGA/SPI1_SCK
- J21 pad 17: unconnected-(J21-Pad17) -> /MAGIC/FPGA/S2
- J21 pad 18: unconnected-(J21-Pad18) -> /MAGIC/FPGA/S1
- J21 pad 19: unconnected-(J21-Pad19) -> /MAGIC/FPGA/S3
- J21 pad 20: unconnected-(J21-Pad20) -> /MAGIC/FPGA/NSTATUS
- J21 pad 21: unconnected-(J21-Pad21) -> /MAGIC/FPGA/S5
- J21 pad 22: unconnected-(J21-Pad22) -> /MAGIC/FPGA/S4
- J21 pad 24: unconnected-(J21-Pad24) -> /MAGIC/FPGA/S6
- J22 pad 15: /MAGIC/FPGA/CBUS1 -> unconnected-(J22-Pad15)
- J22 pad 17: /MAGIC/FPGA/CBUS0 -> /MAGIC/FPGA/I2C1_SCL
- J22 pad 19: /MAGIC/FPGA/MCU_CEC -> /MAGIC/FPGA/CBUS0
- J22 pad 21: /MAGIC/FPGA/CSI -> unconnected-(J22-Pad21)
- J22 pad 23: /MAGIC/FPGA/GP27 -> unconnected-(J22-Pad23)
- J22 pad 25: /MAGIC/FPGA/I2C0_SCL -> unconnected-(J22-Pad25)
- J22 pad 27: /MAGIC/FPGA/I2C0_SDA -> unconnected-(J22-Pad27)
- J22 pad 9: /MAGIC/FPGA/CBUS2 -> /MAGIC/FPGA/SPI1_~{READY}
- J23 pad 10: /MAGIC/FPGA/S1 -> /MAGIC/FPGA/X1
- J23 pad 6: /MAGIC/FPGA/S3 -> /MAGIC/FPGA/X3
- J23 pad 8: /MAGIC/FPGA/S2 -> /MAGIC/FPGA/X2
- SW1 pad 2: /MAGIC/FPGA/~{NMI} -> /MAGIC/~{RES}
- SW3 pad 1: GND -> /MAGIC/MCU/GP27
- SW3 pad 2: /MAGIC/MCU/RUN -> GND
- SW4 pad 2: /MAGIC/~{RES} -> /MAGIC/FPGA/~{NMI}
- SW5 pad 2: /MAGIC/MCU/BOOTSEL -> GND
- U14 pad 13: /MAGIC/FPGA/CBUS2 -> /MAGIC/FPGA/SPI1_~{READY}
- U14 pad 4: /MAGIC/MCU/I2C1_SDA -> /MAGIC/FPGA/CBUS0
- U14 pad 5: /MAGIC/MCU/I2C1_SCL -> /MAGIC/FPGA/I2C1_SCL
- U17 pad 2: VCORE -> Net-(U17-Pad2)
- U21 pad 134: unconnected-(U21-Pad134) -> /MAGIC/FPGA/S1
- U21 pad 135: unconnected-(U21-Pad135) -> /MAGIC/FPGA/S2
- U21 pad 139: unconnected-(U21-Pad139) -> /MAGIC/FPGA/S3
- U21 pad 140: unconnected-(U21-Pad140) -> /MAGIC/FPGA/S4
- U21 pad 141: unconnected-(U21-Pad141) -> /MAGIC/FPGA/S5
- U21 pad 142: unconnected-(U21-Pad142) -> /MAGIC/FPGA/S6
- U21 pad 39: /MAGIC/FPGA/S3 -> /MAGIC/FPGA/X3
- U21 pad 40: /MAGIC/FPGA/S2 -> /MAGIC/FPGA/X2
- U21 pad 41: /MAGIC/FPGA/S1 -> /MAGIC/FPGA/X1
Routing:
- net /MAGIC/FPGA/SPI1_SCK: track 16.1 -> 97.8 mm, vias 0 -> 2
- net +1V1: track 16.6 -> 91.8 mm, vias 0 -> 1
- net /MAGIC/FPGA/MCU_CLK: track 14.3 -> 85.0 mm
- net GND: track 1784.8 -> 1851.0 mm, vias 39 -> 49
- net +3V3: track 503.1 -> 558.4 mm, vias 9 -> 19
- net /MAGIC/FPGA/CBUS0: track 40.2 -> 91.1 mm, vias 0 -> 3
- net /MAGIC/FPGA/I2C1_SCL: track 0.00 -> 47.8 mm, vias 0 -> 2
- net +5V: track 885.1 -> 840.7 mm, vias 11 -> 18
- net /MAGIC/FPGA/CDI0: track 19.6 -> 63.2 mm, vias 1 -> 3
- net /MAGIC/FPGA/~{SS}: track 15.7 -> 58.9 mm, vias 0 -> 2
- net /MAGIC/FPGA/CDI1: track 16.4 -> 58.3 mm, vias 0 -> 2
- net /MAGIC/FPGA/SPI1_RX: track 131.9 -> 92.7 mm, vias 2 -> 3
- net /MAGIC/MCU/GP27: track 0.00 -> 38.8 mm
- net /MAGIC/FPGA/CCK: track 22.4 -> 60.5 mm, vias 1 -> 3
- net /MAGIC/FPGA/~{CRESET}: track 67.8 -> 105.4 mm, vias 1 -> 2
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- added copper zone on F.Cu, net +5V
- removed copper zone on F.Cu, net +3V3
- removed copper zone on B.Cu, net GND
- removed copper zone on F.Cu, net Net-(D5-Pad1)
Other:
- board size 262.9 x 95.2 mm -> 262.5 x 95.2 mm
- board text added: "$E810"
- board text added: "$E820"
- board text added: "$E840"
- board text added: "+"
- board text added: "+9V"
- board text added: "-"
- board text added: "AS6C1008"
- board text added: "CPU"
- board text added: "MCU RESET"
- board text added: "NMI"
- board text added: "NSTATUS"
- board text added: "PIA1"
- board text added: "PIA2"
- board text added: "RAM"
- board text added: "RESET"
- board text added: "SCL"
- board text added: "SDA"
- board text added: "SPEAKER"
- board text added: "VIA"
- board text added: "VIDEO"
- board text added: "W65C02S"
- board text added: "W65C21N"
- board text added: "W65C22N"
- board text added: "↑"
- board text added: "↓"
- board text added: "∿"
- board text removed: "9V↑"
- board text removed: "DC↓"
