File: hw/Mainboard/Mainboard.kicad_pcb (KiCad board)
At the start: 2 copper layers, 262.5 x 95.2 mm, 240 parts, among them J1 SJ-43504-SMT-TR, J10 5V PWR, J11 9V POWER, J12 NOT_HDMI_A, J13 Micro_SD, J14 USB2.0_HOST_TYPE_C, J15 DEBUG, J16 MCU_EXT, J17 BOOTSEL, J18 PET POWER, J2 KEYBOARD, J21 FPGA-P4, J22 Conn_02x15_Odd_Even, J23 FPGA_P2, J24 FPGA_P3, J3 IEEE, J4 USER, J5 CASS A, J6 CASS B, J7 9V POWER, J8 SPEAKER, J9 PET_Video, Q1 AO3401A, Q2 MMBT3904, Q3 AO3401A, Q4 MMBT3904, SW1 RESET, SW2 MCU_RESET, SW3 MENU, SW4 NMI, SW5 CONFIG, U1 74LS145, U10 XL1509-5.0E1, U11 W65C02S, U12 AS6C1008, U13 AMS1117-3.3, U14 RP2040, U15 LM317AG-TN3-R, U16 W25Q128JVS, U17 LM1117-1.2, U18 SN74LVC4245APWR, U19 SN74LVC4245APWR, U2 SN74LS07, U20 SN74LVC4245APWR, U21 T8Q144C3, U3 SN74LS07, U4 SN74LS07, U5 74LS245, U6 74LS245, U7 W65C21N, U8 W65C21N, U9 W65C22N, X1 50MHZ, Y1 12 MHz

Commit message: hw: routable (wip)
Parts:
- removed R24: 10k, Resistor_SMD:R_0402_1005Metric
- added NT1: GND, PET:NetTie-2_SMD_Pad_1.6_to_0.4mm, F.Cu at (-242.5, 21.9)
- added NT10: +5V, PET:NetTie-2_SMD_Pad_1.6_to_0.4mm, F.Cu at (-168.3, 59.1)
- added NT11: +6V, PET:NetTie-2_SMD_Pad_1.6_to_0.4mm, F.Cu at (-192.7, 68.3)
- added NT12: +6V, PET:NetTie-2_SMD_Pad_1.6_to_0.4mm, F.Cu at (-21.2, 4.65)
- added NT13: +5V, PET:NetTie-2_SMD_Pad_1.6_to_0.4mm, F.Cu at (-189.6, 59.1)
- added NT14: +5V, PET:NetTie-2_SMD_Pad_1.6_to_0.4mm, F.Cu at (-210.4, 59.1)
- added NT15: +5V, PET:NetTie-2_SMD_Pad_1.6_to_0.4mm, F.Cu at (-210.4, 10.9)
- added NT16: +9V, PET:NetTie-2_SMD_Pad_1.6_to_0.4mm, F.Cu at (-201.6, 68.8)
- added NT17: GND, PET:NetTie-2_SMD_Pad_1.6_to_0.4mm, F.Cu at (-243.8, 44.7)
- added NT2: +9V, PET:NetTie-2_SMD_Pad_1.6_to_0.4mm, F.Cu at (-235.7, 24.0)
- added NT3: +3V3, PET:NetTie-2_SMD_Pad_0.4_to_0.2mm, F.Cu at (-12.9, 58.4)
- added NT4: GND, PET:NetTie-2_SMD_Pad_0.4_to_0.2mm, F.Cu at (-22.8, 81.0)
- added NT5: +3V3, PET:NetTie-2_SMD_Pad_0.4_to_0.2mm, F.Cu at (-18.9, 60.8)
- added NT6: +5V, PET:NetTie-2_SMD_Pad_0.4_to_0.2mm, F.Cu at (-30.8, 76.2)
- added NT7: +3V3, PET:NetTie-2_SMD_Pad_0.4_to_0.2mm, F.Cu at (-52.1, 8.40)
- added NT8: +3V3, PET:NetTie-2_SMD_Pad_0.4_to_0.2mm, F.Cu at (-53.5, 26.2)
- added NT9: +6V, PET:NetTie-2_SMD_Pad_1.6_to_0.4mm, F.Cu at (-21.2, 8.25)
- added R64: 4k7, Resistor_SMD:R_0402_1005Metric, F.Cu at (-37.9, 29.4)
- added R65: 4k7, Resistor_SMD:R_0402_1005Metric, F.Cu at (-37.9, 32.0)
- C35: footprint Capacitor_THT:CP_Radial_D10.0mm_P5.00mm -> PET:CP_Radial_D16.0mm_P5.00mm_P7.50mm
- JP11: value FPGA PWR -> FPGA VCC
- R20, R38, R39, R40, R59: value 10k -> 4k7
- R41: value 2.7k -> 2k7
- R44, R50: value 1.5k -> 1k5
- moved C34 9.64 mm to (-242.4, 47.0), turned to 180 degrees
- moved C35 8.95 mm to (-234.8, 56.8), turned to 180 degrees
- moved C17 6.37 mm to (-243.7, 24.4)
- moved C26 6.01 mm to (-233.1, 39.6)
- moved L1 6.01 mm to (-240.9, 38.7)
- moved D5 6.01 mm to (-233.6, 32.3)
- moved C14 6.01 mm to (-233.1, 44.2)
- moved C16 6.01 mm to (-233.1, 37.2)
- moved C32 6.01 mm to (-233.1, 42.0)
- moved U10 6.01 mm to (-239.9, 28.9)
- moved C53 4.10 mm to (-236.7, 23.0)
- moved J7 1.22 mm to (-237.5, 17.2)
- moved J11 1.22 mm to (-232.4, 19.4)
- moved C8 1.15 mm to (-191.5, 58.7)
- moved R9 0.84 mm to (-30.3, 75.4)
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Connections:
- net +1V1 renamed MCU_DVDD
- net /POWER/VCCA renamed FPGA_VCCA
- net GNDPWR renamed CHASSIS_GND
- net Net-(J14-PadA5) renamed /MAGIC/MCU/CC1
- net Net-(J14-PadB5) renamed /MAGIC/MCU/CC2
- net Net-(R34-Pad2) renamed /MAGIC/FPGA/REF_RES
- net VCORE renamed FPGA_VCC
- C13 pad 2: GND -> PD_GND
- C14 pad 1: +5V -> PD_5V
- C14 pad 2: GND -> PD_GND
- C16 pad 1: +5V -> PD_5V
- C16 pad 2: GND -> PD_GND
- C17 pad 1: +9V_Unreg -> Net-(C17-Pad1)
- C17 pad 2: GND -> Net-(C17-Pad2)
- C21 pad 1: +5V -> PD_5V
- C26 pad 1: +5V -> PD_5V
- C26 pad 2: GND -> PD_GND
- C29 pad 1: +6V -> Net-(C29-Pad1)
- C32 pad 1: +5V -> PD_5V
- C32 pad 2: GND -> PD_GND
- C33 pad 1: GND -> PD_GND
- C34 pad 1: +5V -> PD_5V
- C34 pad 2: GND -> PD_GND
- C35 pad 2: GND -> PD_GND
- C38 pad 1: +3V3 -> MCU_IOVDD
- C41 pad 1: +3V3 -> MCU_IOVDD
- C42 pad 1: +3V3 -> MCU_IOVDD
- C43 pad 1: +3V3 -> MCU_IOVDD
- C45 pad 1: +3V3 -> MCU_IOVDD
- C46 pad 1: +3V3 -> MCU_IOVDD
- C52 pad 2: GND -> PD_GND
- C53 pad 2: GND -> PD_GND
- C69 pad 1: +3V3 -> FPGA_VCCIO
- C70 pad 1: +3V3 -> FPGA_VCCIO
- C71 pad 1: +3V3 -> FPGA_VCCIO
- C72 pad 1: +3V3 -> FPGA_VCCIO
- C73 pad 1: +3V3 -> FPGA_VCCIO
- C74 pad 1: +3V3 -> FPGA_VCCIO
- C75 pad 1: +3V3 -> FPGA_VCCIO
- C76 pad 1: +3V3 -> FPGA_VCCIO
- C77 pad 1: +3V3 -> FPGA_VCCIO
- C78 pad 1: +3V3 -> FPGA_VCCIO
- C79 pad 1: +3V3 -> FPGA_VCCIO
- C80 pad 1: +3V3 -> FPGA_VCCIO
- D2 pad 2: GND -> PD_GND
- D5 pad 2: GND -> PD_GND
- J10 pad 1: +5V -> PD_5V
- J10 pad 2: +5V -> PD_5V
- J10 pad 3: +5V -> PD_5V
- J11 pad 1: GND -> PD_GND
- J12 pad 11: GND -> DVI_GND
- J12 pad 17: GND -> DVI_GND
- J12 pad 18: +5V -> DVI_VDD
- J12 pad 2: GND -> DVI_GND
- J12 pad 5: GND -> DVI_GND
- J12 pad 8: GND -> DVI_GND
- J18 pad 3: GND -> PD_GND
- J18 pad 6: GND -> PD_GND
- J3 pad 12: GND -> PD_GND
- J4 pad 1: GND -> PD_GND
- J4 pad 12: GND -> PD_GND
- J4 pad A: GND -> PD_GND
- J4 pad N: GND -> PD_GND
- J5 pad 1,A: GND -> PD_GND
- J5 pad 2,B: +5V -> PD_5V
- J6 pad 1,A: GND -> PD_GND
- J6 pad 2,B: +5V -> PD_5V
- J7 pad 2: GND -> PD_GND
- J7 pad 3: GND -> PD_GND
- L1 pad 2: +5V -> PD_5V
- Q1 pad 2: +6V -> PD_6V
- Q3 pad 2: +6V -> PD_6V
- R40 pad 2: Net-(R40-Pad2) -> +3V3
- R42 pad 2: GND -> PD_GND
- R43 pad 1: +6V -> Net-(C29-Pad1)
- R44 pad 1: +6V -> Net-(R44-Pad1)
- R47 pad 1: +6V -> Net-(C29-Pad1)
- R50 pad 1: +6V -> Net-(R50-Pad1)
- U10 pad 1: +9V_Unreg -> Net-(C17-Pad1)
- U10 pad 3: +5V -> Net-(U10-Pad3)
- U10 pad 4: GND -> PD_GND
- U10 pad 5: GND -> PD_GND
- U10 pad 6: GND -> PD_GND
- U10 pad 7: GND -> PD_GND
- U10 pad 8: GND -> PD_GND
- U11 pad 2: Net-(R40-Pad2) -> /MAGIC/FPGA/RDY
- U11 pad 21: GND -> PD_GND
- U12 pad 16: GND -> PD_GND
- U13 pad 3: +5V -> PD_5V
- U14 pad 1: +3V3 -> MCU_IOVDD
- U14 pad 10: +3V3 -> MCU_IOVDD
- U14 pad 19: GND -> /MAGIC/MCU/TESTEN
- U14 pad 22: +3V3 -> MCU_IOVDD
- U14 pad 33: +3V3 -> MCU_IOVDD
- U14 pad 42: +3V3 -> MCU_IOVDD
- U14 pad 43: +3V3 -> MCU_IOVDD
- U14 pad 44: +3V3 -> MCU_IOVDD
- U14 pad 48: +3V3 -> MCU_IOVDD
- U14 pad 49: +3V3 -> MCU_IOVDD
- U15 pad 2: +6V -> PD_6V
- U21 pad 1: GND -> FPGA_GND
- U21 pad 104: GND -> FPGA_GND
- U21 pad 108: GND -> FPGA_GND
- U21 pad 12: +3V3 -> FPGA_VCCIO
- U21 pad 120: GND -> FPGA_GND
- U21 pad 121: GND -> FPGA_GND
- U21 pad 122: +3V3 -> FPGA_VCCIO
- U21 pad 126: GND -> FPGA_GND
- U21 pad 127: GND -> FPGA_GND
- U21 pad 129: GND -> FPGA_GND
- U21 pad 133: GND -> FPGA_GND
- U21 pad 143: +3V3 -> FPGA_VCCIO
- U21 pad 21: +3V3 -> FPGA_VCCIO
- U21 pad 23: +3V3 -> FPGA_VCCIO
- U21 pad 37: GND -> FPGA_GND
- U21 pad 44: GND -> FPGA_GND
- U21 pad 5: GND -> FPGA_GND
- U21 pad 50: GND -> FPGA_GND
- U21 pad 51: +3V3 -> FPGA_VCCIO
- U21 pad 52: +3V3 -> FPGA_VCCIO
- U21 pad 62: +3V3 -> FPGA_VCCIO
- U21 pad 63: +3V3 -> FPGA_VCCIO
- U21 pad 64: GND -> FPGA_GND
- U21 pad 88: +3V3 -> FPGA_VCCIO
- U21 pad 9: GND -> FPGA_GND
- U21 pad 91: +3V3 -> FPGA_VCCIO
- U21 pad 94: GND -> FPGA_GND
- U21 pad 95: +3V3 -> FPGA_VCCIO
- U7 pad 1: GND -> PD_GND
- U7 pad 20: +5V -> PD_5V
- U8 pad 1: GND -> PD_GND
- U8 pad 20: +5V -> PD_5V
- U9 pad 1: GND -> PD_GND
- U9 pad 20: +5V -> PD_5V
Routing:
- net PD_GND: track 0.00 -> 601.3 mm, vias 0 -> 7
- net PD_5V: track 0.00 -> 409.0 mm, vias 0 -> 5
- net GND: track 1851.0 -> 1452.2 mm, vias 49 -> 39
- net PD_6V: track 0.00 -> 257.0 mm, vias 0 -> 2
- net +6V: track 270.8 -> 32.4 mm, vias 2 -> 0
- net +5V: track 840.7 -> 671.4 mm, vias 18 -> 17
- net FPGA_VCCIO: track 0.00 -> 165.6 mm, vias 0 -> 7
- net FPGA_GND: track 0.00 -> 109.5 mm, vias 0 -> 4
- net /IEEE/EOI_OUT: track 79.2 -> 182.6 mm, vias 0 -> 7
- net +3V3: track 558.4 -> 488.7 mm, vias 19 -> 6
- net /MAGIC/BHORIZ: track 177.5 -> 114.8 mm
- net /MAGIC/FPGA/~{NMI}: track 159.6 -> 210.5 mm, vias 2 -> 5
- net /IEEE/NRFD_OUT: track 53.9 -> 103.9 mm
- net /MAGIC/FPGA/SYNC: track 77.3 -> 123.2 mm, vias 2 -> 9
- net FPGA_VCC: track 158.0 -> 203.0 mm, vias 9 -> 10
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- removed copper zone on F.Cu, net +5V
Other:
- board text removed: "1V2"
- board text removed: "3V3"

Commit message: hw: wip
Parts:
- added NT18: +5V, PET:NetTie-2_SMD_Pad_1.6_to_0.4mm, F.Cu at (5.45, 74.5)
- added NT19: GND, PET:NetTie-2_SMD_Pad_1.6_to_0.4mm, F.Cu at (8.88, 76.7)
- added NT20: +5V, PET:NetTie-2_SMD_Pad_1.6_to_0.4mm, F.Cu at (3.92, 67.8)
- added NT21: GND, PET:NetTie-2_SMD_Pad_1.6_to_0.4mm, F.Cu at (7.20, 65.2)
- added R24: 1k, Resistor_SMD:R_0402_1005Metric, F.Cu at (-33.6, 67.5)
- added R66: 1k, Resistor_SMD:R_0402_1005Metric, F.Cu at (-34.8, 68.5)
- R64, R65: value 4k7 -> 2k2
- SW1, SW2, SW4: footprint Button_Switch_THT:SW_PUSH_6mm -> JLCPCB:SW-TH_L6.0-W3.5-P6.50
- moved SW2 20.6 mm to (-58.0, 80.7), turned to 90 degrees
- moved SW4 10.5 mm to (-65.0, 80.7), turned to 90 degrees
- moved SW1 6.17 mm to (-72.0, 80.7), turned to 90 degrees
- moved C24 3.86 mm to (-68.5, 81.0)
- moved C25 2.53 mm to (-61.5, 80.5)
Connections:
- C24 pad 2: GND -> PD_GND
- C25 pad 2: GND -> PD_GND
- J14 pad A12_B1: GND -> Net-(J14-PadA12_B1)
- J14 pad A1_B12: GND -> Net-(J14-PadA12_B1)
- J14 pad A4_B9: +5V -> Net-(J14-PadA4_B9)
- J14 pad A9_B4: +5V -> Net-(J14-PadA4_B9)
- J14 pad S1: GND -> Net-(J14-PadA12_B1)
- J2 pad 1: GND -> PD_GND
- J22 pad 22: unconnected-(J22-Pad22) -> /MAGIC/FPGA/~{FPGA_PROG}
- J9 pad 2: GND -> PD_GND
- J9 pad 4: GND -> PD_GND
- J9 pad 7: GND -> PD_GND
- R35 pad 1: +5V -> Net-(J14-PadA4_B9)
- R36 pad 1: +5V -> Net-(J14-PadA4_B9)
- SW1 pad 1: GND -> PD_GND
- SW2 pad 2: /MAGIC/MCU/RUN -> Net-(SW2-Pad2)
- SW4 pad 1: GND -> PD_GND
Routing:
- net GND: track 1452.2 -> 1247.5 mm, vias 39 -> 32
- net /MAGIC/FPGA/~{NMI}: track 210.5 -> 82.9 mm, vias 5 -> 1
- net /IEEE/EOI_OUT: track 182.6 -> 80.3 mm, vias 7 -> 0
- net PD_GND: track 601.3 -> 697.2 mm, vias 7 -> 8
- net PD_5V: track 409.0 -> 468.0 mm, vias 5 -> 4
- net /IEEE/NRFD_OUT: track 103.9 -> 62.9 mm
- net /IEEE/IFC: track 47.6 -> 83.2 mm
- net /IEEE/ATN_OUT: track 66.0 -> 97.5 mm, vias 2 -> 1
- net /IEEE/NDAC_OUT: track 61.0 -> 32.9 mm, vias 4 -> 0
- net /IEEE/NDAC: track 128.2 -> 100.5 mm
- net /MAGIC/FPGA/NSTATUS: track 39.3 -> 11.8 mm, vias 3 -> 1
- net Net-(J14-PadA12_B1): track 0.00 -> 25.5 mm
- net /IEEE/DAV: track 110.6 -> 135.8 mm, vias 5 -> 6
- net /CPU \ RAM/A9: track 64.3 -> 88.9 mm, vias 0 -> 1
- net Net-(D7-Pad2): track 33.4 -> 9.22 mm, vias 4 -> 0
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Other:
- board text added: "RUN"

Commit message: hw: pull cbus0 high
Parts:
- added NT22: GND, PET:NetTie-2_SMD_Pad_1.6_to_0.4mm, F.Cu at (-61.5, 84.0)
- added NT23: GND, PET:NetTie-2_SMD_Pad_1.6_to_0.4mm, F.Cu at (-68.5, 84.0)
- added R67: 10k, Resistor_SMD:R_0402_1005Metric, F.Cu at (-58.7, 22.2)
- moved R63 2.26 mm to (-57.2, 23.6)
- moved NT5 1.33 mm to (-17.8, 61.5), turned to 180 degrees
- moved C24 0.30 mm to (-68.5, 80.7)
- moved R51 0.22 mm to (-58.0, 22.9)
- moved C25 0.20 mm to (-61.5, 80.7)
- turned NT15 to -90 degrees
Connections:
- C24 pad 2: PD_GND -> Net-(C24-Pad2)
- C25 pad 2: PD_GND -> Net-(C25-Pad2)
- J22 pad 19: /MAGIC/FPGA/CBUS0 -> /MAGIC/FPGA/I2C1_SDA
- R64 pad 2: /MAGIC/FPGA/CBUS0 -> /MAGIC/FPGA/I2C1_SDA
- SW2 pad 1: GND -> PD_GND
- U14 pad 4: /MAGIC/FPGA/CBUS0 -> /MAGIC/FPGA/I2C1_SDA
- U21 pad 14: unconnected-(U21-Pad14) -> /MAGIC/FPGA/I2C1_SCL
- U21 pad 15: unconnected-(U21-Pad15) -> /MAGIC/FPGA/I2C1_SDA
Routing:
- net /MAGIC/R~{W}: track 134.1 -> 0.00 mm, vias 6 -> 0
- net PD_GND: track 697.2 -> 786.7 mm
- net /IO/KEY_ROW2: track 88.5 -> 0.00 mm, vias 1 -> 0
- net /CPU \ RAM/A3: track 82.4 -> 0.00 mm, vias 1 -> 0
- net /CPU \ RAM/A14: track 72.0 -> 0.00 mm, vias 2 -> 0
- net /CPU \ RAM/A7: track 64.9 -> 0.00 mm, vias 1 -> 0
- net /MAGIC/FPGA/~{RAM_CE}: track 77.8 -> 13.2 mm
- net /CASS/~{CASS1_SWITCH}: track 63.2 -> 0.00 mm, vias 2 -> 0
- net /MAGIC/FPGA/~{NMI}: track 82.9 -> 144.7 mm, vias 1 -> 2
- net /MAGIC/FPGA/CBUS0: track 84.2 -> 24.3 mm
- net /MAGIC/FPGA/~{RD_STROBE}: track 68.6 -> 15.9 mm
- net Net-(D5-Pad1): track 16.4 -> 68.4 mm
- net /CPU \ RAM/D6: track 74.7 -> 25.0 mm
- net /MAGIC/FPGA/~{FPGA_PROG}: track 0.00 -> 49.1 mm, vias 0 -> 1
- net /MAGIC/FPGA/I2C1_SDA: track 0.00 -> 45.1 mm, vias 0 -> 2
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Other:
- board text removed: "MCU RESET"

Commit message: hw: wip
Parts:
- removed J22: Conn_02x15_Odd_Even, Connector_PinHeader_2.54mm:PinHeader_2x15_P2.54mm_Vertical
- added C82: 100n, Capacitor_SMD:C_0402_1005Metric, F.Cu at (-5.20, 36.9)
- added J19: PROG, Connector_IDC:IDC-Header_2x08_P2.54mm_Vertical, F.Cu at (-16.0, 12.1)
- added NT24: GND, PET:NetTie-2_SMD_Pad_1.6_to_0.4mm, F.Cu at (-3.95, 20.4)
- J16: value MCU_EXT -> MCU; footprint Connector_PinHeader_2.54mm:PinHeader_1x05_P2.54mm_Vertical -> Connector_PinHeader_2.54mm:PinHeader_2x10_P2.54mm_Vertical
- moved J16 60.8 mm to (-47.1, 24.9), turned to 0 degrees
- moved J10 24.5 mm to (-72.0, 4.53), turned to 180 degrees
- moved C21 17.0 mm to (-68.7, 1.45), turned to -90 degrees
- moved C36 15.9 mm to (-62.6, -1.85), turned to 0 degrees
- moved R60 14.6 mm to (-78.2, 0.80), turned to 180 degrees
- moved R55 14.6 mm to (-76.7, 0.29), turned to 90 degrees
- moved R50 13.8 mm to (-9.00, 0.00), turned to 180 degrees
- moved C54 13.6 mm to (-46.2, 6.80)
- moved C81 13.6 mm to (-53.8, 0.97)
- moved JP11 13.6 mm to (-48.7, 1.00)
- moved R37 13.6 mm to (-52.0, 0.97)
- moved U17 13.6 mm to (-44.4, 2.00)
- moved C55 13.6 mm to (-50.3, 0.95)
- moved NT12 13.1 mm to (-8.49, 1.55), turned to 90 degrees
- moved Q3 12.5 mm to (-8.56, -2.64), turned to -90 degrees
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Connections:
- J16 pad 2: /MAGIC/MCU/MCU_CEC -> +3V3
- J16 pad 3: +3V3 -> /MAGIC/MCU/I2C0_SDA
- J16 pad 4: /MAGIC/MCU/I2C0_SCL -> /MAGIC/FPGA/I2C1_SDA
- J16 pad 5: /MAGIC/MCU/I2C0_SDA -> /MAGIC/MCU/I2C0_SCL
- J8 pad 1: GND -> PD_GND
- J8 pad 3: GND -> PD_GND
- R24 pad 1: /MAGIC/FPGA/~{FPGA_PROG} -> /MAGIC/FPGA/~{SPI_ENA}
- R62 pad 2: GND -> PD_GND
- RN14 pad 1: /MAGIC/FPGA/TCK -> /MAGIC/FPGA/TDO
- RN14 pad 2: /MAGIC/FPGA/TDI -> /MAGIC/FPGA/TMS
- RN14 pad 3: /MAGIC/FPGA/TDO -> /MAGIC/FPGA/TCK
- RN14 pad 4: /MAGIC/FPGA/TMS -> /MAGIC/FPGA/TDI
- U14 pad 13: /MAGIC/FPGA/SPI1_~{READY} -> /MAGIC/MCU/SPI1_~{READY}
Routing:
- net /MAGIC/R~{W}: track 0.00 -> 128.0 mm, vias 0 -> 4
- net /CPU \ RAM/A3: track 0.00 -> 87.9 mm, vias 0 -> 1
- net /IO/KEY_ROW2: track 0.00 -> 82.0 mm, vias 0 -> 1
- net /MAGIC/FPGA/NSTATUS: track 37.8 -> 115.5 mm, vias 2 -> 3
- net /CPU \ RAM/A14: track 0.00 -> 72.7 mm, vias 0 -> 1
- net /MAGIC/FPGA/~{RAM_CE}: track 13.2 -> 82.2 mm, vias 0 -> 1
- net /CPU \ RAM/A7: track 0.00 -> 64.0 mm, vias 0 -> 1
- net /MAGIC/FPGA/~{SPI_ENA}: track 0.00 -> 55.6 mm, vias 0 -> 1
- net /CASS/~{CASS1_SWITCH}: track 0.00 -> 53.4 mm, vias 0 -> 2
- net /MAGIC/FPGA/~{RD_STROBE}: track 15.9 -> 68.8 mm
- net /MAGIC/FPGA/I2C1_SDA: track 45.1 -> 96.4 mm, vias 2 -> 3
- net /CPU \ RAM/D6: track 25.0 -> 74.7 mm
- net PD_GND: track 786.7 -> 836.4 mm, vias 8 -> 5
- net /MAGIC/FPGA/~{FPGA_PROG}: track 49.1 -> 0.00 mm, vias 1 -> 0
- net /IO/DIAG: track 155.7 -> 111.6 mm, vias 5 -> 4
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Other:
- board text added: "+1V2"
- board text added: "+3V3"
- board text added: "CCK"
- board text added: "CDI0"
- board text added: "CDI1"
- board text added: "CEC"
- board text added: "CLK"
- board text added: "ENA"
- board text added: "HOLD"
- board text added: "~{CRESET}"
- board text added: "~{SS}"
- board text removed: "~{CRST}"

Commit message: hw: larger schematic pages, routed w/netties
Parts:
- removed R18, R48, R51, R63, R67: 10k, Resistor_SMD:R_0402_1005Metric
- added NT25: +9V, PET:NetTie-2_SMD_Pad_1.6_to_0.4mm, F.Cu at (-205.3, 70.6)
- added NT26: +9V, PET:NetTie-2_SMD_Pad_1.6_to_0.4mm, F.Cu at (-212.4, 73.0)
- added NT27: +9V, PET:NetTie-2_SMD_Pad_1.6_to_0.4mm, F.Cu at (-227.8, 69.0)
- added NT28: +9V, PET:NetTie-2_SMD_Pad_1.6_to_0.4mm, F.Cu at (-228.0, 73.0)
- added NT29: +9V, PET:NetTie-2_SMD_Pad_1.6_to_0.4mm, F.Cu at (-216.3, 69.0)
- added NT30: +9V, PET:NetTie-2_SMD_Pad_1.6_to_0.4mm, F.Cu at (-218.0, 72.0)
- added NT31: +9V, PET:NetTie-2_SMD_Pad_1.6_to_0.4mm, F.Cu at (-214.4, 69.0)
- added RN15: 10k, Resistor_SMD:R_Array_Convex_4x0603, F.Cu at (-56.5, 21.1)
- J9: value PET_Video -> VIDEO
- R24: value 1k -> 10k
- moved C82 18.6 mm to (-11.2, 19.2), turned to 0 degrees
- moved C52 17.8 mm to (-215.3, 73.5), turned to 180 degrees
- moved C51 8.07 mm to (-3.63, 51.2), turned to 0 degrees
- moved R26 6.74 mm to (-7.60, 44.8), turned to 180 degrees
- moved C21 5.35 mm to (-63.4, 1.45)
- moved U13 5.35 mm to (-58.6, 3.65)
- moved C36 5.15 mm to (-57.5, -1.85)
- moved R66 4.64 mm to (-39.0, 66.5), turned to -90 degrees
- moved C33 4.57 mm to (-216.3, 71.5), turned to 90 degrees
- moved R24 4.03 mm to (-29.6, 67.5), turned to 90 degrees
- moved R54 3.58 mm to (-81.8, 4.79)
- moved R58 3.58 mm to (-81.8, 2.79)
- moved R52 3.58 mm to (-80.2, 4.28)
- moved R55 3.58 mm to (-80.2, 0.29)
- moved R57 3.58 mm to (-80.2, 2.28)
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Connections:
- net +6V renamed Net-(Q2-Pad3)
- net /MAGIC/FPGA/I2C1_SCL renamed /MAGIC/MCU/I2C1_SCL
- net /MAGIC/FPGA/I2C1_SDA renamed /MAGIC/MCU/I2C1_SDA
- net /MAGIC/FPGA/SPI1_RX renamed /MAGIC/MCU/SPI1_RX
- net /MAGIC/FPGA/SPI1_SCK renamed /MAGIC/MCU/SPI1_SCK
- net /MAGIC/FPGA/SPI1_TX renamed /MAGIC/MCU/SPI1_TX
- net /MAGIC/FPGA/SPI1_~{CS} renamed /MAGIC/MCU/SPI1_~{CS}
- C13 pad 1: Net-(C12-Pad2) -> /POWER/+9V_UNFILT
- C15 pad 1: Net-(C12-Pad2) -> Net-(C15-Pad1)
- C22 pad 1: +9V_Unreg -> Net-(C22-Pad1)
- C33 pad 1: PD_GND -> Net-(C33-Pad1)
- C33 pad 2: Net-(C12-Pad2) -> Net-(C33-Pad2)
- D2 pad 1: Net-(C12-Pad2) -> /POWER/+9V_UNFILT
- D3 pad 1: Net-(C12-Pad2) -> /POWER/+9V_UNFILT
- D3 pad 2: Net-(C12-Pad1) -> /POWER/VAC1
- D4 pad 1: Net-(C12-Pad2) -> /POWER/+9V_UNFILT
- D4 pad 2: Net-(C15-Pad2) -> /POWER/VAC2
- J18 pad 1: Net-(C12-Pad1) -> /POWER/VAC1
- J18 pad 2: Net-(C12-Pad2) -> +9V_Unreg
- J18 pad 4: +9V_Unreg -> /POWER/+9V_UNFILT
- J18 pad 5: Net-(C15-Pad2) -> /POWER/VAC2
- J19 pad 1: +3V3 -> unconnected-(J19-Pad1)
- J19 pad 3: unconnected-(J19-Pad3) -> +3V3
- R24 pad 1: /MAGIC/FPGA/~{SPI_ENA} -> +3V3
- R66 pad 1: Net-(R66-Pad1) -> /MAGIC/FPGA/~{SPI_ENA}
- SW2 pad 2: Net-(R66-Pad1) -> /MAGIC/MCU/RUN
- U11 pad 1: /CPU \ RAM/~{VP} -> /MAGIC/FPGA/~{VP}
- U11 pad 38: /CPU \ RAM/~{SO} -> /MAGIC/FPGA/~{SO}
- U11 pad 5: /CPU \ RAM/~{ML} -> /MAGIC/FPGA/~{ML}
- U21 pad 18: unconnected-(U21-Pad18) -> /MAGIC/MCU/SPI1_~{READY}
Routing:
- net PD_GND: track 836.4 -> 918.2 mm
- net /MAGIC/FPGA/~{VP}: track 12.9 -> 82.9 mm
- net /MAGIC/FPGA/~{ML}: track 17.6 -> 81.1 mm
- net /MAGIC/FPGA/~{SO}: track 17.2 -> 65.5 mm, vias 1 -> 2
- net /MAGIC/MCU/SPI1_~{READY}: track 41.5 -> 72.3 mm, vias 0 -> 1
- net Net-(C12-Pad2): track 29.3 -> 0.82 mm
- net /POWER/+9V_UNFILT: track 0.00 -> 27.3 mm
- net /MAGIC/MCU/RUN: track 16.2 -> 43.4 mm
- net Net-(R66-Pad1): track 26.8 -> 0.00 mm
- net /IO/VIA_CB2: track 187.6 -> 162.1 mm
- net /MAGIC/MCU/I2C1_SDA: track 96.4 -> 72.1 mm
- net /MAGIC/FPGA/TDI: track 58.8 -> 37.8 mm, vias 0 -> 2
- net /MAGIC/MCU/SPI1_TX: track 101.2 -> 122.2 mm
- net /MAGIC/FPGA/~{CRESET}: track 120.5 -> 139.9 mm, vias 3 -> 2
- net /MAGIC/~{RES}: track 169.4 -> 150.5 mm, vias 2 -> 3
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Other:
- outline, holes or cut-outs redrawn
- board text added: "SWCLK"
- board text added: "SWD"
- board text removed: "9V"
