File: hw/Mainboard/Mainboard.kicad_pcb (KiCad board)
At the start: 2 copper layers, 262.5 x 95.2 mm, 300 parts, among them J1 SJ-43504-SMT-TR, J10 5V PWR, J11 9V POWER, J12 NOT_HDMI_A, J13 MicroSD, J14 USB2.0_HOST_TYPE_C, J15 KEYBOARD_EX, J16 MCU, J18 PET POWER, J19 PROG, J2 KEYBOARD, J20 5V PWR, J21 FPGA-P4, J22 MENU, J23 FPGA_P2, J24 Conn_02x15_Odd_Even, J25 IEEE_HEADER, J26 USER_HEADER, J27 CASS_A_HEADER, J28 CASS_B_HEADER, J3 IEEE, J4 USER, J5 CASS A, J6 CASS B, J7 9V POWER, J8 FLASH, J9 VIDEO, Q1 AO3401A, Q3 AO3401A, Q4 MMBT3904, SW1 RESET, SW2 RUN, SW3 MENU, SW4 NMI, SW5 CONFIG, U1 74LS145, U10 LM317AG-TN3-R, U11 W65C02S, U12 AS6C1008, U13 AMS1117-3.3, U14 RP2040, U15 LM317AG-TN3-R, U16 W25Q128JVS, U17 LM317AG-TN3-R, U18 SN74LVC4245APWR, U19 SN74LVC4245APWR, U2 SN74LS07, U20 SN74LVC4245APWR, U21 T8Q144C3, U22 LM386, U3 SN74LS07, U4 SN74LS07, U5 74LS245, U6 74LS245, U7 W65C21N, U8 W65C21N, U9 W65C22N, Y1 12 MHz

Commit message: wip
Parts:
- added JP10: VIDEO_OR_5V, Jumper:SolderJumper-3_P1.3mm_Open_RoundedPad1.0x1.5mm, B.Cu at (260.3, 105.5)
- added PT42: PowerTie_2, PET:NetTie-2_SMD_Pad_0.28, F.Cu at (283.3, 134.7)
- added PT43: PowerTie_2, PET:NetTie-2_SMD_Pad_0.28, F.Cu at (272.3, 122.5)
- added PT44: PowerTie_2, PET:NetTie-2_SMD_Pad_0.28, F.Cu at (268.3, 122.8)
- added PT45: PowerTie_2, PET:NetTie-2_SMD_Pad_0.28, F.Cu at (255.6, 133.5)
- added PT46: PowerTie_2, PET:NetTie-2_SMD_Pad_0.28, F.Cu at (255.6, 139.9)
- added PT47: PowerTie_2, PET:NetTie-2_SMD_Pad_0.28, F.Cu at (270.0, 150.3)
- added PT48: PowerTie_2, PET:NetTie-2_SMD_Pad_0.28, F.Cu at (283.1, 133.3)
- added PT49: PowerTie_2, PET:NetTie-2_SMD_Pad_0.28, F.Cu at (271.1, 123.0)
- added PT50: PowerTie_2, PET:NetTie-2_SMD_Pad_0.28, F.Cu at (264.6, 122.5)
- added PT51: PowerTie_2, PET:NetTie-2_SMD_Pad_0.28, F.Cu at (256.4, 135.2)
- added PT52: PowerTie_2, PET:NetTie-2_SMD_Pad_0.28, F.Cu at (256.4, 138.7)
- added PT53: PowerTie_2, PET:NetTie-2_SMD_Pad_0.28, F.Cu at (267.3, 150.3)
- added PT54: PowerTie_2, PET:NetTie-2_SMD_Pad_0.28, F.Cu at (278.9, 150.3)
- added PT55: PowerTie_2, PET:NetTie-2_SMD_Pad_1.6_to_0.4mm, F.Cu at (171.8, 159.3)
- C52: value 10u -> 2.2u 6.3V; footprint Capacitor_SMD:C_0603_1608Metric -> Capacitor_SMD:C_0402_1005Metric
- PT40: footprint PET:NetTie-2_SMD_Pad_1.6_to_0.4mm -> PET:NetTie-2_SMD_Pad_0.28; moved to F.Cu
- PT41: footprint PET:NetTie-2_SMD_Pad_1.6_to_0.4mm -> PET:NetTie-2_SMD_Pad_0.28
- U15: footprint Package_TO_SOT_SMD:TO-252-2 -> PET:TO-252-2_ThermalVias
- moved C74 49.6 mm to (284.8, 125.3), turned to 0 degrees
- moved C70 22.0 mm to (284.3, 177.7)
- moved PT41 22.0 mm to (283.5, 139.3), turned to 180 degrees
- moved PT40 10.1 mm to (283.5, 140.3), turned to 180 degrees
- moved C36 7.32 mm to (303.3, 100.1)
- moved C21 7.31 mm to (294.0, 95.9)
- moved U13 7.29 mm to (298.6, 100.1)
- moved C24 7.01 mm to (270.2, 177.7)
- moved C25 7.00 mm to (277.3, 177.7)
- moved R66 6.65 mm to (305.2, 167.7)
- moved Q1 6.54 mm to (143.9, 171.1)
- moved R44 6.42 mm to (145.2, 168.4)
- moved PT22 6.42 mm to (142.9, 168.4)
- moved C32 5.95 mm to (289.9, 101.2)
- moved R43 5.93 mm to (289.9, 100.2)
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Connections:
- net /IO/Bϕ2 renamed /IO/BPHI2
- net /MAGIC/ϕ2 renamed /MAGIC/PHI2
- C34 pad 1: /MAGIC/FPGA/VCCIO -> +3V3
- C53 pad 1: /MAGIC/FPGA/VCCIO -> +3V3
- C60 pad 1: /MAGIC/FPGA/VCC -> +1V2
- C61 pad 1: /MAGIC/FPGA/VCC -> +1V2
- C62 pad 1: /MAGIC/FPGA/VCC -> +1V2
- C63 pad 1: /MAGIC/FPGA/VCC -> +1V2
- C64 pad 1: /MAGIC/FPGA/VCC -> +1V2
- C65 pad 1: /MAGIC/FPGA/VCC -> +1V2
- C66 pad 1: /MAGIC/FPGA/VCC -> +1V2
- C67 pad 1: /MAGIC/FPGA/VCC -> +1V2
- C68 pad 1: /MAGIC/FPGA/VCC -> +1V2
- C69 pad 1: /MAGIC/FPGA/VCCIO -> +3V3
- C70 pad 1: /MAGIC/FPGA/~{SPI_ENA} -> Net-(SW2-Pad2)
- C71 pad 1: /MAGIC/FPGA/VCCIO -> +3V3
- C72 pad 1: /MAGIC/FPGA/VCCIO -> +3V3
- C73 pad 1: /MAGIC/FPGA/VCCIO -> +3V3
- C75 pad 1: /MAGIC/FPGA/VCCIO -> +3V3
- C76 pad 1: /MAGIC/FPGA/VCCIO -> +3V3
- C77 pad 1: /MAGIC/FPGA/VCCIO -> +3V3
- C78 pad 1: /MAGIC/FPGA/VCCIO -> +3V3
- C79 pad 1: /MAGIC/FPGA/VCCIO -> +3V3
- C80 pad 1: /MAGIC/FPGA/VCCIO -> +3V3
- C83 pad 1: /MAGIC/FPGA/VCC -> +1V2
- C9 pad 1: +5V -> Net-(C9-Pad1)
- J4 pad 2: /MAGIC/BVIDEO -> /USER/VIDEO_OR_5V
- PT40 pad 2: /MAGIC/FPGA/VCCIO -> /MAGIC/FPGA/VCCIO_12
- PT41 pad 2: /MAGIC/FPGA/VCC -> /MAGIC/FPGA/VCC_13
- R66 pad 1: Net-(R66-Pad1) -> Net-(SW2-Pad2)
- SW2 pad 2: Net-(R66-Pad1) -> Net-(SW2-Pad2)
- U19 pad 17: /CPU \ RAM/A3 -> /CPU \ RAM/~{RES}
- U19 pad 18: /CPU \ RAM/~{RES} -> /CPU \ RAM/A3
- U19 pad 6: /IEEE/IFC_OUT -> /IO/BA3
- U19 pad 7: /IO/BA3 -> /IEEE/IFC_OUT
- U21 pad 12: /MAGIC/FPGA/VCCIO -> /MAGIC/FPGA/VCCIO_12
- U21 pad 122: /MAGIC/FPGA/VCCIO -> /MAGIC/FPGA/VCCIO_122
- U21 pad 125: /MAGIC/FPGA/VCC -> /MAGIC/FPGA/VCC_125
- U21 pad 128: /MAGIC/FPGA/VCC -> /MAGIC/FPGA/VCC_125
- U21 pad 13: /MAGIC/FPGA/VCC -> /MAGIC/FPGA/VCC_13
- U21 pad 130: /MAGIC/FPGA/VCC -> /MAGIC/FPGA/VCC_125
- U21 pad 143: /MAGIC/FPGA/VCCIO -> /MAGIC/FPGA/VCCIO_143
- U21 pad 21: /MAGIC/FPGA/VCCIO -> /MAGIC/FPGA/VCCIO_23
- U21 pad 22: /MAGIC/FPGA/VCC -> /MAGIC/FPGA/VCC_22
- U21 pad 23: /MAGIC/FPGA/VCCIO -> /MAGIC/FPGA/VCCIO_23
- U21 pad 49: /MAGIC/FPGA/VCC -> /MAGIC/FPGA/VCC_49
- U21 pad 51: /MAGIC/FPGA/VCCIO -> /MAGIC/FPGA/VCCIO_52
- U21 pad 52: /MAGIC/FPGA/VCCIO -> /MAGIC/FPGA/VCCIO_52
- U21 pad 57: /MAGIC/FPGA/VCC -> /MAGIC/FPGA/VCC_57
- U21 pad 62: /MAGIC/FPGA/VCCIO -> /MAGIC/FPGA/VCCIO_62
- U21 pad 63: /MAGIC/FPGA/VCCIO -> /MAGIC/FPGA/VCCIO_62
- U21 pad 85: /MAGIC/FPGA/VCC -> /MAGIC/FPGA/VCC_85
- U21 pad 88: /MAGIC/FPGA/VCCIO -> /MAGIC/FPGA/VCCIO_88
- U21 pad 91: /MAGIC/FPGA/VCCIO -> /MAGIC/FPGA/VCCIO_88
- U21 pad 95: /MAGIC/FPGA/VCCIO -> /MAGIC/FPGA/VCCIO_95
- U21 pad 96: /MAGIC/FPGA/VCC -> /MAGIC/FPGA/VCC_96
Routing:
- net /MAGIC/FPGA/VCCIO: track 111.1 -> 0.00 mm, vias 6 -> 0
- net /MAGIC/FPGA/VCC: track 100.8 -> 0.00 mm, vias 6 -> 0
- net /CASS/CASS_A_~{SWITCH}: track 220.0 -> 294.6 mm
- net +1V2: track 58.2 -> 129.9 mm
- net /MAGIC/BHORIZ: track 185.4 -> 122.1 mm, vias 4 -> 2
- net +6V: track 271.9 -> 313.6 mm, vias 2 -> 5
- net /MAGIC/FPGA/SPI1_SCK: track 106.6 -> 66.3 mm, vias 1 -> 2
- net /IO/BD6: track 52.5 -> 90.7 mm
- net /MAGIC/MCU/SD_~{CS}: track 35.0 -> 64.8 mm
- net /IO/VIA_PA5: track 131.8 -> 161.4 mm, vias 1 -> 3
- net /IEEE/NRFD_OUT: track 52.0 -> 80.5 mm, vias 1 -> 2
- net /CPU \ RAM/RAM_A15: track 53.7 -> 25.7 mm, vias 3 -> 1
- net Net-(SW2-Pad2): track 0.00 -> 25.2 mm, vias 0 -> 1
- net /MAGIC/MCU/GP25: track 36.8 -> 58.2 mm, vias 2 -> 0
- net /IEEE/DIO1: track 125.2 -> 103.9 mm, vias 3 -> 2
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Other:
- board text added: "PIN 2"

Commit message: hw: wip
Parts:
- moved PT5 5.16 mm to (110.1, 139.5)
- moved D5 3.80 mm to (105.8, 139.6)
- moved J20 1.58 mm to (104.8, 99.4)
- moved C11 0.31 mm to (240.2, 117.4)
- moved C5 0.27 mm to (112.7, 104.3), turned to -90 degrees
Routing:
- net +3V3: track 479.1 -> 483.4 mm
- net /CASS/CASS1_READ: track 161.2 -> 158.0 mm
- net /IEEE/VCC: track 177.2 -> 174.4 mm
- net Net-(D6-Pad1): track 211.8 -> 209.6 mm
- net GND: track 1177.6 -> 1175.8 mm
- net +9V_Unreg: track 105.2 -> 103.5 mm
- net /IO/BVERT: track 218.0 -> 216.8 mm
- net /IO/VIA_PA5: track 161.4 -> 160.1 mm
- net CHASSIS_GND: track 54.4 -> 53.1 mm
- net /MAGIC/BHORIZ: track 122.1 -> 121.1 mm
- net /CASS/CASS_WRITE: track 285.5 -> 284.6 mm
- net PD_GND: track 843.1 -> 842.3 mm
- net +5V: track 659.7 -> 660.4 mm
- net +6V: track 313.6 -> 314.2 mm
- net /MAGIC/FPGA/BE: track 63.1 -> 62.5 mm
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Other:
- board text added: "5V PWR"

Commit message: hw: routing / silk wip
Parts:
- removed D15: SM4007, Diode_SMD:D_SOD-123F
- added C84: 10u, Capacitor_SMD:C_0603_1608Metric, F.Cu at (342.8, 177.0)
- added C85: 10u, Capacitor_SMD:C_0603_1608Metric, F.Cu at (287.6, 105.5)
- added G***: LOGO, LOGO, F.Cu at (101.0, 120.7)
- added PT56: PowerTie_2, PET:NetTie-2_SMD_Pad_1.6_to_0.4mm, F.Cu at (150.1, 159.3)
- added R73: 2k2, Resistor_SMD:R_0402_1005Metric, F.Cu at (299.1, 139.8)
- added R74: 2k2, Resistor_SMD:R_0402_1005Metric, F.Cu at (300.1, 140.8)
- C81: value 47u 10V -> 10u; footprint Capacitor_SMD:C_1206_3216Metric -> Capacitor_SMD:C_0603_1608Metric
- J16: footprint Connector_PinHeader_2.54mm:PinHeader_2x12_P2.54mm_Vertical -> Connector_PinHeader_2.54mm:PinHeader_2x11_P2.54mm_Vertical
- JP8: value DVI_SCL -> DVI_SDA; footprint Jumper:SolderJumper-2_P1.3mm_Open_RoundedPad1.0x1.5mm -> Jumper:SolderJumper-3_P1.3mm_Open_RoundedPad1.0x1.5mm
- JP9: value DVI_SDA -> DVI_SCL; footprint Jumper:SolderJumper-2_P1.3mm_Open_RoundedPad1.0x1.5mm -> Jumper:SolderJumper-3_P1.3mm_Open_RoundedPad1.0x1.5mm
- R43: value 300 -> 120
- moved C81 165.2 mm to (128.0, 171.9)
- moved R33 50.7 mm to (284.8, 124.3), turned to 0 degrees
- moved JP8 18.8 mm to (305.4, 171.9)
- moved JP9 18.5 mm to (308.4, 171.9)
- moved C26 7.57 mm to (292.5, 96.2)
- moved D14 7.33 mm to (288.0, 100.1)
- moved U17 7.30 mm to (292.7, 102.4)
- moved PT13 7.05 mm to (242.1, 187.9)
- moved R43 6.81 mm to (296.7, 100.3), turned to 90 degrees
- moved PT14 6.09 mm to (290.4, 96.2), turned to 0 degrees
- moved C52 4.66 mm to (346.2, 184.1)
- moved C36 3.44 mm to (306.8, 100.1)
- moved U13 3.44 mm to (302.1, 100.1)
- moved C21 3.25 mm to (297.2, 95.9)
- moved C32 2.81 mm to (288.2, 103.4), turned to 180 degrees
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Connections:
- net Net-(J14-PadA4_B9) renamed /MAGIC/MCU/USB/VBUS1
- net Net-(J14-PadA9_B4) renamed /MAGIC/MCU/USB/VBUS2
- net Net-(JP7-Pad2) renamed /MAGIC/MCU/DVI/CEC
- C8 pad 1: +5V -> Net-(C8-Pad1)
- C81 pad 1: +1V2 -> Net-(C22-Pad1)
- J16 pad 10: /MAGIC/FPGA/L20 -> /MAGIC/FPGA/I2C1_SCL
- J16 pad 11: /MAGIC/FPGA/I2C1_SDA -> /MAGIC/FPGA/SPI0_RX
- J16 pad 12: /MAGIC/FPGA/L21 -> /MAGIC/FPGA/SPI1_~{READY}
- J16 pad 13: /MAGIC/FPGA/I2C1_SCL -> /MAGIC/FPGA/I2C0_SDA
- J16 pad 14: /MAGIC/FPGA/SPI1_~{READY} -> /MAGIC/FPGA/SPI1_~{CS}
- J16 pad 15: /MAGIC/FPGA/L46 -> /MAGIC/FPGA/I2C0_SCL
- J16 pad 16: /MAGIC/FPGA/SPI1_~{CS} -> /MAGIC/FPGA/SPI1_SCK
- J16 pad 17: /MAGIC/MCU/I2C0_SDA -> /MAGIC/FPGA/L46
- J16 pad 18: /MAGIC/FPGA/SPI1_SCK -> /MAGIC/FPGA/SPI1_TX
- J16 pad 19: /MAGIC/MCU/I2C0_SCL -> /MAGIC/FPGA/CEC
- J16 pad 20: /MAGIC/FPGA/SPI1_TX -> /MAGIC/FPGA/SPI1_RX
- J16 pad 21: /MAGIC/FPGA/CEC -> +3V3
- J16 pad 22: /MAGIC/FPGA/SPI1_RX -> +3V3
- J16 pad 3: /MAGIC/FPGA/SPI0_~{CS} -> /MAGIC/FPGA/AUDIO
- J16 pad 4: /MAGIC/FPGA/AUDIO -> /MAGIC/FPGA/L12
- J16 pad 5: /MAGIC/FPGA/SPI0_SCK -> /MAGIC/FPGA/SPI0_~{CS}
- J16 pad 6: /MAGIC/FPGA/L12 -> /MAGIC/FPGA/L13
- J16 pad 7: /MAGIC/FPGA/SPI0_TX -> /MAGIC/FPGA/SPI0_SCK
- J16 pad 8: /MAGIC/FPGA/L13 -> /MAGIC/FPGA/I2C1_SDA
- J16 pad 9: /MAGIC/FPGA/SPI0_RX -> /MAGIC/FPGA/SPI0_TX
- JP8 pad 1: /MAGIC/MCU/I2C0_SCL -> /MAGIC/FPGA/I2C0_SDA
- JP8 pad 2: /MAGIC/MCU/DVI/HDMI_SCL -> /MAGIC/MCU/MCU_I2C0_SDA
- JP9 pad 1: /MAGIC/MCU/I2C0_SDA -> /MAGIC/FPGA/I2C0_SCL
- JP9 pad 2: /MAGIC/MCU/DVI/HDMI_SDA -> /MAGIC/MCU/MCU_I2C0_SCL
- U14 pad 40: /MAGIC/MCU/I2C0_SDA -> /MAGIC/MCU/MCU_I2C0_SDA
- U14 pad 41: /MAGIC/MCU/I2C0_SCL -> /MAGIC/MCU/MCU_I2C0_SCL
- U21 pad 14: /MAGIC/FPGA/FPGA_SPI1_~{READY} -> /MAGIC/FPGA/I2C0_SCL
- U21 pad 16: /MAGIC/FPGA/I2C1_SDA -> /MAGIC/FPGA/FPGA_SPI1_~{READY}
- U21 pad 17: /MAGIC/FPGA/L21 -> /MAGIC/FPGA/I2C0_SDA
- U21 pad 18: /MAGIC/FPGA/L20 -> /MAGIC/FPGA/I2C1_SDA
- U6 pad 8: /IEEE/VSS -> GND
- U6 pad 9: /IEEE/VSS -> GND
Routing:
- net /MAGIC/FPGA/I2C0_SDA: track 0.00 -> 59.7 mm, vias 0 -> 1
- net /MAGIC/FPGA/I2C0_SCL: track 0.00 -> 59.3 mm, vias 0 -> 2
- net /MAGIC/MCU/I2C0_SDA: track 53.5 -> 0.00 mm, vias 1 -> 0
- net /MAGIC/MCU/I2C0_SCL: track 47.9 -> 0.00 mm, vias 1 -> 0
- net /IO/BD6: track 90.7 -> 50.7 mm, vias 1 -> 0
- net /CASS/CASS_A_~{SWITCH}: track 294.6 -> 259.9 mm
- net /MAGIC/MCU/SD_~{CS}: track 64.8 -> 33.1 mm
- net /MAGIC/MCU/MCU_I2C0_SDA: track 0.00 -> 29.2 mm, vias 0 -> 1
- net GND: track 1175.8 -> 1152.2 mm, vias 28 -> 29
- net /MAGIC/FPGA/TDI: track 45.0 -> 67.7 mm, vias 2 -> 1
- net /MAGIC/FPGA/~{CRESET}: track 133.7 -> 112.0 mm
- net /MAGIC/MCU/MCU_I2C0_SCL: track 0.00 -> 21.1 mm, vias 0 -> 1
- net /MAGIC/FPGA/L20: track 15.9 -> 0.00 mm, vias 1 -> 0
- net /MAGIC/MCU/DVI/HDMI_SDA: track 23.7 -> 8.25 mm
- net /MAGIC/FPGA/L21: track 15.0 -> 0.00 mm, vias 1 -> 0
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Other:
- board text added: "CASSETTE"
- board text added: "L75"
- board text added: "R11"
- board text added: "Regulators are HOT if excessive current drawn."
- board text added: "WARNING"
- board text removed: "L20"
- board text removed: "L21"
- board text removed: "R75"
- board text removed: "↑"
- board text removed: "↓"

Commit message: hw: minor cleanup
Parts:
- removed R62: 33, Resistor_SMD:R_0402_1005Metric
- moved C80 0.10 mm to (284.8, 140.2)
- moved C66 0.08 mm to (284.8, 139.2)
- moved PT41 0.08 mm to (283.5, 139.2)
Connections:
- U21 pad 33: /MAGIC/FPGA/CSO -> /MAGIC/FPGA/AUDIO
Routing:
- net GND: track 1152.2 -> 1158.3 mm
- net /MAGIC/FPGA/AUDIO: track 44.3 -> 49.6 mm
- net /MAGIC/FPGA/CSO: track 4.35 -> 0.00 mm
Other:
- board text added: "D5"
- board text added: "HORIZ"
- board text added: "Regulators are HOT if high current drawn."
- board text added: "VERT"
- board text removed: "D8"
- board text removed: "Regulators are HOT if excessive current drawn."
