File: hw/Mainboard/CASS.kicad_sch (KiCad schematic)
At the start: 18 parts, among them J5 CASS A, J6 CASS B, Q1 AO3401A, Q3 AO3401A

Commit message: hw: wip
Parts:
- added NT33, NT34: +5V, PET:NetTie-2_SMD_Pad_1.6_to_0.4mm, symbol PET:PowerTie_2
- NT11, NT12: symbol Device:NetTie_2 -> PET:PowerTie_2
Connections:
- net PD_5V: now also NT33.1, NT34.1
- net +5V: no longer names the net of R56.1
- net +5V: now also NT33.2; no longer R49.1
- new net: NT34.2, R49.1
Changed lines of the file:
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@@
   (junction (at 177.8 106.68) (diameter 0) (color 0 0 0 0)
   )
+  (junction (at 113.03 139.7) (diameter 0) (color 0 0 0 0)
+  )
   (junction (at 139.7 125.73) (diameter 0) (color 0 0 0 0)
   )
@@
   (junction (at 129.54 139.7) (diameter 0) (color 0 0 0 0)
   )
-  (junction (at 119.38 139.7) (diameter 0) (color 0 0 0 0)
-  )
   (junction (at 215.9 86.36) (diameter 0) (color 0 0 0 0)
   )
@@
     (stroke (width 0) (type default) (color 0 0 0 0))
   )
+  (wire (pts (xy 113.03 139.7) (xy 115.57 139.7))
+    (stroke (width 0) (type default) (color 0 0 0 0))
+  )
   (wire (pts (xy 129.54 139.7) (xy 312.42 139.7))
     (stroke (width 0) (type default) (color 0 0 0 0))
@@
     (stroke (width 0) (type default) (color 0 0 0 0))
   )
-  (wire (pts (xy 119.38 139.7) (xy 119.38 144.78))
-    (stroke (width 0) (type default) (color 0 0 0 0))
-  )
   (wire (pts (xy 269.24 130.81) (xy 269.24 132.08))
     (stroke (width 0) (type default) (color 0 0 0 0))
   )
-  (wire (pts (xy 119.38 144.78) (xy 121.92 144.78))
+  (wire (pts (xy 120.65 144.78) (xy 121.92 144.78))
     (stroke (width 0) (type default) (color 0 0 0 0))
   )
@@
     (stroke (width 0) (type default) (color 0 0 0 0))
   )
+  (wire (pts (xy 115.57 144.78) (xy 113.03 144.78))
+    (stroke (width 0) (type default) (color 0 0 0 0))
+  )
   (wire (pts (xy 248.92 179.07) (xy 312.42 179.07))
     (stroke (width 0) (type default) (color 0 0 0 0))
@@
     (stroke (width 0) (type default) (color 0 0 0 0))
   )
+  (wire (pts (xy 113.03 138.43) (xy 113.03 139.7))
+    (stroke (width 0) (type default) (color 0 0 0 0))
+  )
   (wire (pts (xy 196.85 86.36) (xy 196.85 73.66))
     (stroke (width 0) (type default) (color 0 0 0 0))
@@
     (stroke (width 0) (type default) (color 0 0 0 0))
   )
-  (wire (pts (xy 119.38 139.7) (xy 121.92 139.7))
+  (wire (pts (xy 120.65 139.7) (xy 121.92 139.7))
     (stroke (width 0) (type default) (color 0 0 0 0))
   )
@@
   )
   (wire (pts (xy 269.24 166.37) (xy 269.24 167.64))
+    (stroke (width 0) (type default) (color 0 0 0 0))
+  )
+  (wire (pts (xy 113.03 144.78) (xy 113.03 139.7))
     (stroke (width 0) (type default) (color 0 0 0 0))
   )
@@
     (pin "2")
   )
-  (symbol (lib_id "power:+5V") (at 119.38 139.7 0) (unit 1)
-    (in_bom yes) (on_board yes)
-    (property "Reference" "#PWR0124" (id 0) (at 119.38 143.51 0)
-      (effects (font (size 1.27 1.27)) hide)
-    )
-    (property "Value" "+5V" (id 1) (at 119.761 135.3058 0))
-    (property "Footprint" "" (id 2) (at 119.38 139.7 0)
-      (effects (font (size 1.27 1.27)) hide)
-    )
-    (property "Datasheet" "" (id 3) (at 119.38 139.7 0)
-      (effects (font (size 1.27 1.27)) hide)
-    )
-    (pin "1")
-  )
   (symbol (lib_id "Transistor_FET:AO3401A") (at 288.29 127 270) (mirror x) (unit 1)
     (in_bom yes) (on_board yes)
@@
     (pin "3")
   )
+  (symbol (lib_id "PET:PD_5V") (at 113.03 138.43 0) (mirror y) (unit 1)
+    (in_bom yes) (on_board yes) (fields_autoplaced)
+    (property "Reference" "#PWR0103" (id 0) (at 113.03 142.24 0)
+      (effects (font (size 1.27 1.27)) hide)
+    )
+    (property "Value" "PD_5V" (id 1) (at 113.03 133.35 0))
+    (property "Footprint" "" (id 2) (at 113.03 138.43 0)
+      (effects (font (size 1.27 1.27)) hide)
+    )
+    (property "Datasheet" "" (id 3) (at 113.03 138.43 0)
+      (effects (font (size 1.27 1.27)) hide)
+    )
+    (pin "1")
+  )
   (symbol (lib_id "Device:LED") (at 257.81 132.08 0) (mirror x) (unit 1)
     (in_bom yes) (on_board yes)
@@
     (pin "2")
   )
+  (symbol (lib_id "PET:PowerTie_2") (at 118.11 144.78 0) (unit 1)
+    (in_bom yes) (on_board yes) (fields_autoplaced)
+    (property "Reference" "NT34" (id 0) (at 118.11 139.7 0)
+      (effects (font (size 1.27 1.27)) hide)
+    )
+    (property "Value" "+5V" (id 1) (at 118.11 142.24 0)
+      (effects (font (size 1.27 1.27)) hide)
+    )
+    (property "Footprint" "PET:NetTie-2_SMD_Pad_1.6_to_0.4mm" (id 2) (at 118.11 144.78 0)
+      (effects (font (size 1.27 1.27)) hide)
+    )
+    (property "Datasheet" "~" (id 3) (at 118.11 144.78 0)
+      (effects (font (size 1.27 1.27)) hide)
+    )
+    (pin "1")
+    (pin "2")
+  )
   (symbol (lib_id "PET:PD_GND") (at 326.39 163.83 0) (unit 1)
     (in_bom yes) (on_board yes)
@@
     (pin "2")
   )
+  (symbol (lib_id "PET:PowerTie_2") (at 118.11 139.7 0) (unit 1)
+    (in_bom yes) (on_board yes) (fields_autoplaced)
+    (property "Reference" "NT33" (id 0) (at 118.11 134.62 0)
+      (effects (font (size 1.27 1.27)) hide)
+    )
+    (property "Value" "+5V" (id 1) (at 118.11 137.16 0)
+      (effects (font (size 1.27 1.27)) hide)
+    )
+    (property "Footprint" "PET:NetTie-2_SMD_Pad_1.6_to_0.4mm" (id 2) (at 118.11 139.7 0)
+      (effects (font (size 1.27 1.27)) hide)
+    )
+    (property "Datasheet" "~" (id 3) (at 118.11 139.7 0)
+      (effects (font (size 1.27 1.27)) hide)
+    )
+    (pin "1")
+    (pin "2")
+  )
   (symbol (lib_id "PET:PD_6V") (at 280.67 119.38 0) (unit 1)
     (in_bom yes) (on_board yes) (fields_autoplaced)
@@
     (pin "1")
   )
-  (symbol (lib_id "Device:NetTie_2") (at 275.59 166.37 0) (mirror y) (unit 1)
+  (symbol (lib_id "PET:PowerTie_2") (at 275.59 166.37 0) (mirror y) (unit 1)
     (in_bom yes) (on_board yes) (fields_autoplaced)
     (property "Reference" "NT11" (id 0) (at 275.59 163.83 0)
@@
     (pin "3")
   )
-  (symbol (lib_id "Device:NetTie_2") (at 275.59 124.46 0) (mirror y) (unit 1)
+  (symbol (lib_id "PET:PowerTie_2") (at 275.59 124.46 0) (mirror y) (unit 1)
     (in_bom yes) (on_board yes)
     (property "Reference" "NT12" (id 0) (at 275.59 121.92 0)
