File: hw/Mainboard/CASS.kicad_sch (KiCad schematic)
At the start: 16 parts, among them J5 CASS A, J6 CASS B, Q1 AO3401A, Q3 AO3401A

Commit message: hw: comments
Other:
- note added: "CASS A"
- note added: "CASS B"
- moved on the sheet: D6
Changed lines of the file:
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@@
   (junction (at 140.97 54.61) (diameter 0) (color 0 0 0 0)
   )
-  (wire (pts (xy 130.81 100.33) (xy 179.07 100.33))
+  (wire (pts (xy 130.81 100.33) (xy 181.61 100.33))
     (stroke (width 0) (type default) (color 0 0 0 0))
   )
@@
     (stroke (width 0) (type default) (color 0 0 0 0))
   )
-  (wire (pts (xy 186.69 100.33) (xy 194.31 100.33))
+  (wire (pts (xy 189.23 100.33) (xy 194.31 100.33))
     (stroke (width 0) (type default) (color 0 0 0 0))
   )
@@
     (effects (font (size 1.27 1.27)) (justify left bottom))
   )
+  (text "CASS B" (at 239.395 129.54 0)
+    (effects (font (size 1.5 1.5) (thickness 0.8) bold) (justify left bottom))
+  )
   (text "Red LEDs provide a ~2V drop.  This accounts for the difference between the\n5V CMOS logic and the +6V input, causing the P-Channel MOSFET to turn off\ncompletely when ~{MOTOR} is high.  It also avoids over-voltaging PIA1 and VIA."
     (at 175.26 78.105 0)
     (effects (font (size 1.27 1.27)) (justify left bottom))
+  )
+  (text "CASS A" (at 239.395 87.63 0)
+    (effects (font (size 1.5 1.5) (thickness 0.8) bold) (justify left bottom))
   )
   (label "CASS_WRITE" (at 237.49 147.32 180)
@@
     (pin "1")
   )
-  (symbol (lib_id "Device:LED") (at 182.88 100.33 0) (mirror x) (unit 1)
-    (in_bom yes) (on_board yes)
-    (property "Reference" "D6" (id 0) (at 182.7022 93.853 0))
-    (property "Value" "LED_RED" (id 1) (at 182.7022 96.1644 0))
-    (property "Footprint" "LED_SMD:LED_0603_1608Metric" (id 2) (at 182.88 100.33 0)
-      (effects (font (size 1.27 1.27)) hide)
-    )
-    (property "Datasheet" "https://datasheet.lcsc.com/lcsc/1810231112_Hubei-KENTO-Elec-KT-0603R_C2286.pdf" (id 3) (at 182.88 100.33 0)
-      (effects (font (size 1.27 1.27)) hide)
-    )
-    (property "LCSC" "C2286" (id 4) (at 182.88 100.33 0)
-      (effects (font (size 1.27 1.27)) hide)
-    )
+  (symbol (lib_id "Device:LED") (at 185.42 100.33 0) (mirror x) (unit 1)
+    (in_bom yes) (on_board yes)
+    (property "Reference" "D6" (id 0) (at 185.2422 93.853 0))
+    (property "Value" "LED_RED" (id 1) (at 185.2422 96.1644 0))
+    (property "Footprint" "LED_SMD:LED_0603_1608Metric" (id 2) (at 185.42 100.33 0)
+      (effects (font (size 1.27 1.27)) hide)
+    )
+    (property "Datasheet" "https://datasheet.lcsc.com/lcsc/1810231112_Hubei-KENTO-Elec-KT-0603R_C2286.pdf" (id 3) (at 185.42 100.33 0)
+      (effects (font (size 1.27 1.27)) hide)
+    )
+    (property "LCSC" "C2286" (id 4) (at 185.42 100.33 0)
+      (effects (font (size 1.27 1.27)) hide)
+    )

Commit message: hw: wip
Parts:
- added PT15, PT16, PT21, PT22: PowerTie_2, PET:NetTie-2_SMD_Pad_1.6_to_0.4mm, symbol PET:PowerTie_2
Connections:
- net +5V: now also PT15.1, PT16.1; no longer R49.1, R56.1
- net +6V: now also PT21.1, PT22.1; no longer R44.1, R50.1
- net GND renamed PD_GND
- new net: PT15.2, R56.1
- new net: PT16.2, R49.1
- new net: PT21.2, R50.1
- new net: PT22.2, R44.1
Other:
- moved on the sheet: R44, R50

Commit message: hw: autoroute
Parts:
- added J27: CASS_A_HEADER, Connector_PinHeader_2.54mm:PinHeader_1x06_P2.54mm_Vertical, symbol Connector:Conn_01x06_Male
- added J28: CASS_B_HEADER, Connector_PinHeader_2.54mm:PinHeader_1x06_P2.54mm_Vertical, symbol Connector:Conn_01x06_Male
Connections:
- net +5V: now also J27.2 (Pin_2), J28.2 (Pin_2)
- net CASS_A_MOTOR: now also J27.3 (Pin_3)
- net CASS_A_READ: now also J27.4 (Pin_4)
- net CASS_A_~{SWITCH}: now also J27.6 (Pin_6)
- net CASS_B_MOTOR: now also J28.3 (Pin_3)
- net CASS_B_READ: now also J28.4 (Pin_4)
- net CASS_B_~{SWITCH}: now also J28.6 (Pin_6)
- net CASS_WRITE: now also J27.5 (Pin_5), J28.5 (Pin_5)
- net PD_GND: now also J27.1 (Pin_1), J28.1 (Pin_1)
Changed lines of the file:
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@@
+    (stroke (width 0) (type default) (color 0 0 0 0))
+  )
+  (wire (pts (xy 189.23 39.37) (xy 189.23 34.29))
     (stroke (width 0) (type default) (color 0 0 0 0))
   )
@@
     (stroke (width 0) (type default) (color 0 0 0 0))
   )
+  (wire (pts (xy 186.69 41.91) (xy 186.69 34.29))
+    (stroke (width 0) (type default) (color 0 0 0 0))
+  )
   (wire (pts (xy 189.23 142.24) (xy 195.58 142.24))
     (stroke (width 0) (type default) (color 0 0 0 0))
@@
     (stroke (width 0) (type default) (color 0 0 0 0))
   )
+  (wire (pts (xy 186.69 41.91) (xy 190.5 41.91))
+    (stroke (width 0) (type default) (color 0 0 0 0))
+  )
   (wire (pts (xy 54.61 97.79) (xy 54.61 107.95))
     (stroke (width 0) (type default) (color 0 0 0 0))
@@
     (stroke (width 0) (type default) (color 0 0 0 0))
   )
+  (wire (pts (xy 234.95 34.29) (xy 250.19 34.29))
+    (stroke (width 0) (type default) (color 0 0 0 0))
+  )
   (wire (pts (xy 236.22 132.08) (xy 251.46 132.08))
     (stroke (width 0) (type default) (color 0 0 0 0))
@@
     (stroke (width 0) (type default) (color 0 0 0 0))
   )
+  (wire (pts (xy 236.22 39.37) (xy 234.95 39.37))
+    (stroke (width 0) (type default) (color 0 0 0 0))
+  )
   (wire (pts (xy 97.79 74.93) (xy 102.87 74.93))
     (stroke (width 0) (type default) (color 0 0 0 0))
@@
     (stroke (width 0) (type default) (color 0 0 0 0))
   )
+  (wire (pts (xy 190.5 39.37) (xy 189.23 39.37))
+    (stroke (width 0) (type default) (color 0 0 0 0))
+  )
+  (wire (pts (xy 232.41 41.91) (xy 236.22 41.91))
+    (stroke (width 0) (type default) (color 0 0 0 0))
+  )
   (wire (pts (xy 74.93 149.86) (xy 237.49 149.86))
     (stroke (width 0) (type default) (color 0 0 0 0))
@@
     (stroke (width 0) (type default) (color 0 0 0 0))
   )
+  (wire (pts (xy 189.23 34.29) (xy 204.47 34.29))
+    (stroke (width 0) (type default) (color 0 0 0 0))
+  )
   (wire (pts (xy 113.03 78.74) (xy 113.03 144.78))
     (stroke (width 0) (type default) (color 0 0 0 0))
@@
     (stroke (width 0) (type default) (color 0 0 0 0))
   )
+  (wire (pts (xy 234.95 39.37) (xy 234.95 34.29))
+    (stroke (width 0) (type default) (color 0 0 0 0))
+  )
   (wire (pts (xy 195.58 134.62) (xy 195.58 135.89))
     (stroke (width 0) (type default) (color 0 0 0 0))
@@
   )
   (wire (pts (xy 236.22 90.17) (xy 251.46 90.17))
+    (stroke (width 0) (type default) (color 0 0 0 0))
+  )
+  (wire (pts (xy 232.41 41.91) (xy 232.41 34.29))
     (stroke (width 0) (type default) (color 0 0 0 0))
   )
@@
     (effects (font (size 1.27 1.27)) (justify right bottom))
   )
+  (label "CASS_WRITE" (at 190.5 49.53 180)
+    (effects (font (size 1.27 1.27)) (justify right bottom))
+  )
   (label "CASS_A_MOTOR" (at 237.49 100.33 180)
     (effects (font (size 1.27 1.27)) (justify right bottom))
   )
+  (label "CASS_B_READ" (at 236.22 46.99 180)
+    (effects (font (size 1.27 1.27)) (justify right bottom))
+  )
+  (label "CASS_B_MOTOR" (at 236.22 44.45 180)
+    (effects (font (size 1.27 1.27)) (justify right bottom))
+  )
   (label "CASS_A_~{SWITCH}" (at 237.49 107.95 180)
     (effects (font (size 1.27 1.27)) (justify right bottom))
   )
+  (label "CASS_A_~{SWITCH}" (at 190.5 52.07 180)
+    (effects (font (size 1.27 1.27)) (justify right bottom))
+  )
   (label "CASS_B_READ" (at 237.49 144.78 180)
     (effects (font (size 1.27 1.27)) (justify right bottom))
   )
+  (label "CASS_A_READ" (at 190.5 46.99 180)
+    (effects (font (size 1.27 1.27)) (justify right bottom))
+  )
   (label "CASS_A_READ" (at 237.49 102.87 180)
     (effects (font (size 1.27 1.27)) (justify right bottom))
@@
     (effects (font (size 1.27 1.27)) (justify right bottom))
   )
+  (label "CASS_A_MOTOR" (at 190.5 44.45 180)
+    (effects (font (size 1.27 1.27)) (justify right bottom))
+  )
   (label "CASS_WRITE" (at 237.49 105.41 180)
+    (effects (font (size 1.27 1.27)) (justify right bottom))
+  )
+  (label "CASS_WRITE" (at 236.22 49.53 180)
+    (effects (font (size 1.27 1.27)) (justify right bottom))
+  )
+  (label "CASS_B_~{SWITCH}" (at 236.22 52.07 180)
     (effects (font (size 1.27 1.27)) (justify right bottom))
   )
@@
     (pin "2")
   )
+  (symbol (lib_id "Connector:Conn_01x06_Male") (at 195.58 44.45 0) (mirror y) (unit 1)
+    (in_bom yes) (on_board yes) (fields_autoplaced)
+    (property "Reference" "J27" (id 0) (at 196.85 44.4499 0)
+      (effects (font (size 1.27 1.27)) (justify right))
+    )
+    (property "Value" "CASS_A_HEADER" (id 1) (at 196.85 46.9899 0)
+      (effects (font (size 1.27 1.27)) (justify right))
+    )
+    (property "Footprint" "Connector_PinHeader_2.54mm:PinHeader_1x06_P2.54mm_Vertical" (id 2) (at 195.58 44.45 0)
+      (effects (font (size 1.27 1.27)) hide)
+    )
+    (property "Datasheet" "~" (id 3) (at 195.58 44.45 0)
+      (effects (font (size 1.27 1.27)) hide)
+    )
+    (pin "1")
+    (pin "2")
+    (pin "3")
+    (pin "4")
+    (pin "5")
+    (pin "6")
+  )
+  (symbol (lib_id "PET:PD_GND") (at 250.19 34.29 0) (unit 1)
+    (in_bom yes) (on_board yes) (fields_autoplaced)
+    (property "Reference" "#PWR0191" (id 0) (at 250.19 40.64 0)
+      (effects (font (size 1.27 1.27)) hide)
+    )
+    (property "Value" "PD_GND" (id 1) (at 250.19 39.37 0))
+    (property "Footprint" "" (id 2) (at 250.19 34.29 0)
+      (effects (font (size 1.27 1.27)) hide)
+    )
+    (property "Datasheet" "" (id 3) (at 250.19 34.29 0)
+      (effects (font (size 1.27 1.27)) hide)
+    )
+    (pin "1")
+  )
   (symbol (lib_name "SolderJumper_3_Open_1") (lib_id "Jumper:SolderJumper_3_Open") (at 130.81 54.61 0) (unit 1)
     (in_bom yes) (on_board yes)
@@
     (pin "3")
   )
+  (symbol (lib_id "power:+5V") (at 186.69 34.29 0) (unit 1)
+    (in_bom yes) (on_board yes) (fields_autoplaced)
+    (property "Reference" "#PWR0189" (id 0) (at 186.69 38.1 0)
+      (effects (font (size 1.27 1.27)) hide)
+    )
+    (property "Value" "+5V" (id 1) (at 186.69 29.21 0))
+    (property "Footprint" "" (id 2) (at 186.69 34.29 0)
+      (effects (font (size 1.27 1.27)) hide)
+    )
+    (property "Datasheet" "" (id 3) (at 186.69 34.29 0)
+      (effects (font (size 1.27 1.27)) hide)
+    )
+    (pin "1")
+  )
   (symbol (lib_id "PET:PD_GND") (at 251.46 132.08 0) (unit 1)
     (in_bom yes) (on_board yes) (fields_autoplaced)
@@
     )
     (property "Datasheet" "" (id 3) (at 233.68 132.08 0)
+      (effects (font (size 1.27 1.27)) hide)
+    )
+    (pin "1")
+  )
+  (symbol (lib_id "power:+5V") (at 232.41 34.29 0) (unit 1)
+    (in_bom yes) (on_board yes) (fields_autoplaced)
+    (property "Reference" "#PWR0194" (id 0) (at 232.41 38.1 0)
+      (effects (font (size 1.27 1.27)) hide)
+    )
+    (property "Value" "+5V" (id 1) (at 232.41 29.21 0))
+    (property "Footprint" "" (id 2) (at 232.41 34.29 0)
+      (effects (font (size 1.27 1.27)) hide)
+    )
+    (property "Datasheet" "" (id 3) (at 232.41 34.29 0)
       (effects (font (size 1.27 1.27)) hide)
     )
@@
     (pin "2")
   )
+  (symbol (lib_id "Connector:Conn_01x06_Male") (at 241.3 44.45 0) (mirror y) (unit 1)
+    (in_bom yes) (on_board yes) (fields_autoplaced)
+    (property "Reference" "J28" (id 0) (at 242.57 44.4499 0)
+      (effects (font (size 1.27 1.27)) (justify right))
+    )
+    (property "Value" "CASS_B_HEADER" (id 1) (at 242.57 46.9899 0)
+      (effects (font (size 1.27 1.27)) (justify right))
+    )
+    (property "Footprint" "Connector_PinHeader_2.54mm:PinHeader_1x06_P2.54mm_Vertical" (id 2) (at 241.3 44.45 0)
+      (effects (font (size 1.27 1.27)) hide)
+    )
+    (property "Datasheet" "~" (id 3) (at 241.3 44.45 0)
+      (effects (font (size 1.27 1.27)) hide)
+    )
+    (pin "1")
+    (pin "2")
+    (pin "3")
+    (pin "4")
+    (pin "5")
+    (pin "6")
+  )
   (symbol (lib_id "Device:R_Small") (at 195.58 138.43 0) (unit 1)
     (in_bom yes) (on_board yes)
@@
       (effects (font (size 1.27 1.27)) hide)
     )
+    (pin "1")
+  )
+  (symbol (lib_id "PET:PD_GND") (at 204.47 34.29 0) (unit 1)
+    (in_bom yes) (on_board yes) (fields_autoplaced)
+    (property "Reference" "#PWR0190" (id 0) (at 204.47 40.64 0)
+      (effects (font (size 1.27 1.27)) hide)
+    )
+    (property "Value" "PD_GND" (id 1) (at 204.47 39.37 0))
+    (property "Footprint" "" (id 2) (at 204.47 34.29 0)
+      (effects (font (size 1.27 1.27)) hide)
+    )
+    (property "Datasheet" "" (id 3) (at 204.47 34.29 0)
+      (effects (font (size 1.27 1.27)) hide)
+    )

Commit message: hw: wip
Parts:
- JP1, JP2, JP3, JP4, JP5, JP6: footprint Jumper:SolderJumper-3_P1.3mm_Bridged12_RoundedPad1.0x1.5mm -> Jumper:SolderJumper-3_P1.3mm_Open_RoundedPad1.0x1.5mm
Changed lines of the file:
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@@
     (property "Reference" "JP5" (id 0) (at 130.81 49.53 0))
     (property "Value" "CASS A ~{MOTOR}" (id 1) (at 130.81 52.07 0))
-    (property "Footprint" "Jumper:SolderJumper-3_P1.3mm_Bridged12_RoundedPad1.0x1.5mm" (id 2) (at 130.81 54.61 0)
+    (property "Footprint" "Jumper:SolderJumper-3_P1.3mm_Open_RoundedPad1.0x1.5mm" (id 2) (at 130.81 54.61 0)
       (effects (font (size 1.27 1.27)) hide)
     )
@@
     (property "Reference" "JP1" (id 0) (at 54.61 88.9 0))
     (property "Value" "CASS A ~{SWITCH}" (id 1) (at 54.61 91.44 0))
-    (property "Footprint" "Jumper:SolderJumper-3_P1.3mm_Bridged12_RoundedPad1.0x1.5mm" (id 2) (at 54.61 93.98 0)
+    (property "Footprint" "Jumper:SolderJumper-3_P1.3mm_Open_RoundedPad1.0x1.5mm" (id 2) (at 54.61 93.98 0)
       (effects (font (size 1.27 1.27)) hide)
     )
@@
     (property "Reference" "JP3" (id 0) (at 92.71 69.85 0))
     (property "Value" "CASS A READ" (id 1) (at 92.71 72.39 0))
-    (property "Footprint" "Jumper:SolderJumper-3_P1.3mm_Bridged12_RoundedPad1.0x1.5mm" (id 2) (at 92.71 74.93 0)
+    (property "Footprint" "Jumper:SolderJumper-3_P1.3mm_Open_RoundedPad1.0x1.5mm" (id 2) (at 92.71 74.93 0)
       (effects (font (size 1.27 1.27)) hide)
     )
@@
     (property "Reference" "JP2" (id 0) (at 74.93 88.9 0))
     (property "Value" "CASS B ~{SWITCH}" (id 1) (at 74.93 91.44 0))
-    (property "Footprint" "Jumper:SolderJumper-3_P1.3mm_Bridged12_RoundedPad1.0x1.5mm" (id 2) (at 74.93 93.98 0)
+    (property "Footprint" "Jumper:SolderJumper-3_P1.3mm_Open_RoundedPad1.0x1.5mm" (id 2) (at 74.93 93.98 0)
       (effects (font (size 1.27 1.27)) hide)
     )
@@
     (property "Reference" "JP6" (id 0) (at 151.13 49.53 0))
     (property "Value" "CASS B ~{MOTOR}" (id 1) (at 151.13 52.07 0))
-    (property "Footprint" "Jumper:SolderJumper-3_P1.3mm_Bridged12_RoundedPad1.0x1.5mm" (id 2) (at 151.13 54.61 0)
+    (property "Footprint" "Jumper:SolderJumper-3_P1.3mm_Open_RoundedPad1.0x1.5mm" (id 2) (at 151.13 54.61 0)
       (effects (font (size 1.27 1.27)) hide)
     )
@@
     (property "Reference" "JP4" (id 0) (at 113.03 69.85 0))
     (property "Value" "CASS B READ" (id 1) (at 113.03 72.39 0))
-    (property "Footprint" "Jumper:SolderJumper-3_P1.3mm_Bridged12_RoundedPad1.0x1.5mm" (id 2) (at 113.03 74.93 0)
-      (effects (font (size 1.27 1.27)) hide)
-    )
+    (property "Footprint" "Jumper:SolderJumper-3_P1.3mm_Open_RoundedPad1.0x1.5mm" (id 2) (at 113.03 74.93 0)
+      (effects (font (size 1.27 1.27)) hide)
+    )
