File: hw/Mainboard/CASS.kicad_sch (KiCad schematic)
At the start: 23 parts, among them J14 CASS_A_HEADER, J15 CASS_B_HEADER, J16 CASS A, J17 CASS B, Q2 AO3401A, Q3 AO3401A

Commit message: hw: caps & logos (wip)
Parts:
- removed C99: 10u, Capacitor_SMD:C_0603_1608Metric, symbol Device:C_Small
- added C98: 10u, Capacitor_SMD:C_0603_1608Metric, symbol Device:C_Small
- JP2, JP3, JP4, JP5, JP6, JP7: footprint Jumper:SolderJumper-3_P1.3mm_Bridged12_RoundedPad1.0x1.5mm -> Jumper:SolderJumper-3_P1.3mm_Open_RoundedPad1.0x1.5mm
Connections:
- net +5V: now also C98.2
- net PD_GND: now also C98.1
Other:
- note added: "Place decoupling cap near CASS_B connector. CASS_A has sufficient decoupling nearby."
- title: CBM PET Mainboard Replacement -> EconoPET 40/8096
Changed lines of the file:
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@@
   (paper "A")
   (title_block
-    (title "CBM PET Mainboard Replacement")
+    (title "EconoPET 40/8096")
+    (date "2023-10-01")
+    (rev "A")
   )
   (junction (at 74.93 113.03) (diameter 0) (color 0 0 0 0)
@@
   (text "CASS A" (at 239.395 87.63 0)
     (effects (font (size 1.5 1.5) (thickness 0.8) bold) (justify left bottom))
+  )
+  (text "Place decoupling cap near CASS_B connector.\nCASS_A has sufficient decoupling nearby. "
+    (at 45.72 176.53 0)
+    (effects (font (size 1.27 1.27)) (justify left bottom))
   )
   (label "CASS_B_~{MOTOR}" (at 151.13 58.42 270)
@@
     (property "Reference" "JP2" (id 0) (at 130.81 49.53 0))
     (property "Value" "CASS A ~{MOTOR}" (id 1) (at 130.81 52.07 0))
-    (property "Footprint" "Jumper:SolderJumper-3_P1.3mm_Bridged12_RoundedPad1.0x1.5mm" (id 2) (at 130.81 54.61 0)
+    (property "Footprint" "Jumper:SolderJumper-3_P1.3mm_Open_RoundedPad1.0x1.5mm" (id 2) (at 130.81 54.61 0)
       (effects (font (size 1.27 1.27)) hide)
     )
@@
     (pin "2")
     (pin "3")
+  )
+  (symbol (lib_id "power:+5V") (at 34.29 172.72 0) (unit 1)
+    (in_bom yes) (on_board yes) (fields_autoplaced)
+    (property "Reference" "#PWR0182" (id 0) (at 34.29 176.53 0)
+      (effects (font (size 1.27 1.27)) hide)
+    )
+    (property "Value" "+5V" (id 1) (at 34.29 167.64 0))
+    (property "Footprint" "" (id 2) (at 34.29 172.72 0)
+      (effects (font (size 1.27 1.27)) hide)
+    )
+    (property "Datasheet" "" (id 3) (at 34.29 172.72 0)
+      (effects (font (size 1.27 1.27)) hide)
+    )
+    (pin "1")
   )
   (symbol (lib_id "Jumper:SolderJumper_3_Open") (at 54.61 93.98 0) (unit 1)
@@
     (property "Reference" "JP6" (id 0) (at 54.61 88.9 0))
     (property "Value" "CASS A ~{SWITCH}" (id 1) (at 54.61 91.44 0))
-    (property "Footprint" "Jumper:SolderJumper-3_P1.3mm_Bridged12_RoundedPad1.0x1.5mm" (id 2) (at 54.61 93.98 0)
+    (property "Footprint" "Jumper:SolderJumper-3_P1.3mm_Open_RoundedPad1.0x1.5mm" (id 2) (at 54.61 93.98 0)
       (effects (font (size 1.27 1.27)) hide)
     )
@@
     (property "Reference" "JP4" (id 0) (at 92.71 69.85 0))
     (property "Value" "CASS A READ" (id 1) (at 92.71 72.39 0))
-    (property "Footprint" "Jumper:SolderJumper-3_P1.3mm_Bridged12_RoundedPad1.0x1.5mm" (id 2) (at 92.71 74.93 0)
+    (property "Footprint" "Jumper:SolderJumper-3_P1.3mm_Open_RoundedPad1.0x1.5mm" (id 2) (at 92.71 74.93 0)
       (effects (font (size 1.27 1.27)) hide)
     )
@@
     (pin "2")
     (pin "3")
+  )
+  (symbol (lib_id "Device:C_Small") (at 34.29 175.26 0) (mirror x) (unit 1)
+    (in_bom yes) (on_board yes)
+    (property "Reference" "C98" (id 0) (at 36.6268 176.4284 0)
+      (effects (font (size 1.27 1.27)) (justify left))
+    )
+    (property "Value" "10u" (id 1) (at 36.6268 174.117 0)
+      (effects (font (size 1.27 1.27)) (justify left))
+    )
+    (property "Footprint" "Capacitor_SMD:C_0603_1608Metric" (id 2) (at 34.29 175.26 0)
+      (effects (font (size 1.27 1.27)) hide)
+    )
+    (property "Datasheet" "https://datasheet.lcsc.com/lcsc/2304140030_Samsung-Electro-Mechanics-CL10A106MA8NRNC_C96446.pdf" (id 3) (at 34.29 175.26 0)
+      (effects (font (size 1.27 1.27)) hide)
+    )
+    (property "LCSC" "C96446" (id 4) (at 34.29 175.26 0)
+      (effects (font (size 1.27 1.27)) hide)
+    )
+    (pin "1")
+    (pin "2")
   )
   (symbol (lib_id "PET:PowerTie_2") (at 39.37 107.95 0) (unit 1)
@@
     (property "Reference" "JP7" (id 0) (at 74.93 88.9 0))
     (property "Value" "CASS B ~{SWITCH}" (id 1) (at 74.93 91.44 0))
-    (property "Footprint" "Jumper:SolderJumper-3_P1.3mm_Bridged12_RoundedPad1.0x1.5mm" (id 2) (at 74.93 93.98 0)
+    (property "Footprint" "Jumper:SolderJumper-3_P1.3mm_Open_RoundedPad1.0x1.5mm" (id 2) (at 74.93 93.98 0)
       (effects (font (size 1.27 1.27)) hide)
     )
@@
     )
     (property "Datasheet" "" (id 3) (at 232.41 34.29 0)
-      (effects (font (size 1.27 1.27)) hide)
-    )
-    (pin "1")
-  )
-  (symbol (lib_id "PET:PD_GND") (at 41.91 180.34 0) (unit 1)
-    (in_bom yes) (on_board yes) (fields_autoplaced)
-    (property "Reference" "#PWR0177" (id 0) (at 41.91 186.69 0)
-      (effects (font (size 1.27 1.27)) hide)
-    )
-    (property "Value" "PD_GND" (id 1) (at 41.91 185.42 0))
-    (property "Footprint" "" (id 2) (at 41.91 180.34 0)
-      (effects (font (size 1.27 1.27)) hide)
-    )
-    (property "Datasheet" "" (id 3) (at 41.91 180.34 0)
       (effects (font (size 1.27 1.27)) hide)
     )
@@
     (pin "6")
   )
-  (symbol (lib_id "power:+5V") (at 41.91 175.26 0) (unit 1)
-    (in_bom yes) (on_board yes) (fields_autoplaced)
-    (property "Reference" "#PWR0176" (id 0) (at 41.91 179.07 0)
-      (effects (font (size 1.27 1.27)) hide)
-    )
-    (property "Value" "+5V" (id 1) (at 41.91 170.18 0))
-    (property "Footprint" "" (id 2) (at 41.91 175.26 0)
-      (effects (font (size 1.27 1.27)) hide)
-    )
-    (property "Datasheet" "" (id 3) (at 41.91 175.26 0)
+  (symbol (lib_id "PET:PD_GND") (at 34.29 177.8 0) (unit 1)
+    (in_bom yes) (on_board yes) (fields_autoplaced)
+    (property "Reference" "#PWR0181" (id 0) (at 34.29 184.15 0)
+      (effects (font (size 1.27 1.27)) hide)
+    )
+    (property "Value" "PD_GND" (id 1) (at 34.29 182.88 0))
+    (property "Footprint" "" (id 2) (at 34.29 177.8 0)
+      (effects (font (size 1.27 1.27)) hide)
+    )
+    (property "Datasheet" "" (id 3) (at 34.29 177.8 0)
       (effects (font (size 1.27 1.27)) hide)
     )
@@
     (pin "1")
   )
-  (symbol (lib_id "Device:C_Small") (at 41.91 177.8 0) (mirror x) (unit 1)
-    (in_bom yes) (on_board yes)
-    (property "Reference" "C99" (id 0) (at 44.2468 178.9684 0)
-      (effects (font (size 1.27 1.27)) (justify left))
-    )
-    (property "Value" "10u" (id 1) (at 44.2468 176.657 0)
-      (effects (font (size 1.27 1.27)) (justify left))
-    )
-    (property "Footprint" "Capacitor_SMD:C_0603_1608Metric" (id 2) (at 41.91 177.8 0)
-      (effects (font (size 1.27 1.27)) hide)
-    )
-    (property "Datasheet" "https://datasheet.lcsc.com/lcsc/2304140030_Samsung-Electro-Mechanics-CL10A106MA8NRNC_C96446.pdf" (id 3) (at 41.91 177.8 0)
-      (effects (font (size 1.27 1.27)) hide)
-    )
-    (property "LCSC" "C96446" (id 4) (at 41.91 177.8 0)
-      (effects (font (size 1.27 1.27)) hide)
-    )
-    (pin "1")
-    (pin "2")
-  )
   (symbol (lib_name "SolderJumper_3_Open_3") (lib_id "Jumper:SolderJumper_3_Open") (at 151.13 54.61 0) (unit 1)
     (in_bom yes) (on_board yes)
     (property "Reference" "JP3" (id 0) (at 151.13 49.53 0))
     (property "Value" "CASS B ~{MOTOR}" (id 1) (at 151.13 52.07 0))
-    (property "Footprint" "Jumper:SolderJumper-3_P1.3mm_Bridged12_RoundedPad1.0x1.5mm" (id 2) (at 151.13 54.61 0)
+    (property "Footprint" "Jumper:SolderJumper-3_P1.3mm_Open_RoundedPad1.0x1.5mm" (id 2) (at 151.13 54.61 0)
       (effects (font (size 1.27 1.27)) hide)
     )
@@
     (property "Reference" "JP5" (id 0) (at 113.03 69.85 0))
     (property "Value" "CASS B READ" (id 1) (at 113.03 72.39 0))
-    (property "Footprint" "Jumper:SolderJumper-3_P1.3mm_Bridged12_RoundedPad1.0x1.5mm" (id 2) (at 113.03 74.93 0)
-      (effects (font (size 1.27 1.27)) hide)
-    )
+    (property "Footprint" "Jumper:SolderJumper-3_P1.3mm_Open_RoundedPad1.0x1.5mm" (id 2) (at 113.03 74.93 0)
+      (effects (font (size 1.27 1.27)) hide)
+    )
