File: hw/Mainboard/MCU.kicad_sch (KiCad schematic)
At the start: 66 parts, among them J12 NOT_HDMI_A, J13 Micro_SD, J14 USB2.0_HOST_TYPE_C, J15 DEBUG, J16 MCU, J17 BOOTSEL, SW2 MCU_RESET, SW3 MENU, U14 RP2040, U16 W25Q128JVS, Y1 12 MHz

Commit message: hw: wip
Parts:
- added NT37, NT38: +5V, PET:NetTie-2_SMD_Pad_1.6_to_0.4mm, symbol PET:PowerTie_2
- added NT41: +3V3, PET:NetTie-2_SMD_Pad_0.4_to_0.2mm, symbol PET:PowerTie_2
- added NT42: +3V3, PET:NetTie-2_SMD_Pad_1.6_to_0.4mm, symbol PET:PowerTie_2
- NT18, NT19, NT20, NT21, NT3, NT4, NT5, NT6: symbol Device:NetTie_2 -> PET:PowerTie_2
Connections:
- net +3V3: now also NT38.2, NT41.1, NT42.2; no longer J16.2 (Pin_2)
- net DVI_VDD: now also R8.1, R9.1
- net MCU_IOVDD: now also NT41.2
- net PD_5V: now also NT37.1
- net at J14.A1_B12 (GND), J14.S1 (SHIELD), NT19.2: no longer J14.A12_B1 (GND), NT21.2
- net at J14.A9_B4 (VBUS), NT20.2, R36.1: no longer J14.A4_B9 (VBUS), NT18.2, R35.1
- removed net +5V: NT6.1, R8.1, R9.1
- net ~{FPGA_PROG} renamed ~{SPI_ENA}
- new net: J14.A12_B1 (GND), NT21.2
- new net: NT37.2, NT6.1
- new net: J14.A4_B9 (VBUS), NT18.2, R35.1
- new net PD_3V3: J16.2 (Pin_2), NT38.1, NT42.1
Other:
- note added: "~{SPI_ENA} is driven low during FPGA programming. We use this to hold the MCU in reset when programming to avoid contention on SPI pins. FT2232HL can source ~16ma, so 1K should be ok."
- moved on the sheet: C37, C38, C39, C40, C41, C42, C43, C44, C45, C46, C47, C48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
