File: hw/Mainboard/Audio.kicad_sch (KiCad schematic)
At the start: 9 parts, among them J1 Audio, J8 PET_SPEAKER_01x04_Male, Q2 MMBT3904

Commit message: Document schematics
Parts:
- J8: value PET_SPEAKER_01x04_Male -> SPEAKER
Changed lines of the file:
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@@
       (effects (font (size 1.27 1.27)) (justify right))
     )
-    (property "Value" "PET_SPEAKER_01x04_Male" (id 1) (at 189.23 100.3299 0)
+    (property "Value" "SPEAKER" (id 1) (at 189.23 100.3299 0)
       (effects (font (size 1.27 1.27)) (justify right))
     )

Commit message: hw: T8 (wip)
Parts:
- removed J1: Audio, PET:STX31205B, symbol Connector:AudioJack3_SwitchTR
- added J1: SJ-43504-SMT-TR, SnapEDA:CUI_SJ-43504-SMT-TR, symbol SnapEDA:SJ-43504-SMT-TR
Connections:
- net GND: now also J1.1
- net at C31.2: now also J1.2, J1.3
- net at RV1.2: now also J1.5, J1.6
- no-connect marks 0 -> 1
Changed lines of the file:
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@@
   (junction (at 166.37 116.84) (diameter 0) (color 0 0 0 0)
   )
-  (junction (at 116.84 100.33) (diameter 0) (color 0 0 0 0)
-  )
   (junction (at 154.94 86.36) (diameter 0) (color 0 0 0 0)
   )
+  (junction (at 114.3 102.87) (diameter 0) (color 0 0 0 0)
+  )
   (junction (at 166.37 95.25) (diameter 0) (color 0 0 0 0)
   )
   (junction (at 166.37 69.85) (diameter 0) (color 0 0 0 0)
   )
-  (junction (at 111.76 102.87) (diameter 0) (color 0 0 0 0)
+  (junction (at 120.65 99.06) (diameter 0) (color 0 0 0 0)
   )
   (junction (at 143.51 116.84) (diameter 0) (color 0 0 0 0)
@@
   (junction (at 180.34 102.87) (diameter 0) (color 0 0 0 0)
   )
+  (no_connect (at 120.65 105.41))
+  (wire (pts (xy 118.11 99.06) (xy 120.65 99.06))
+    (stroke (width 0) (type default) (color 0 0 0 0))
+  )
   (wire (pts (xy 166.37 116.84) (xy 166.37 119.38))
     (stroke (width 0) (type default) (color 0 0 0 0))
@@
     (stroke (width 0) (type default) (color 0 0 0 0))
   )
-  (wire (pts (xy 111.76 102.87) (xy 120.65 102.87))
-    (stroke (width 0) (type default) (color 0 0 0 0))
-  )
   (wire (pts (xy 166.37 105.41) (xy 166.37 116.84))
     (stroke (width 0) (type default) (color 0 0 0 0))
   )
-  (wire (pts (xy 120.65 110.49) (xy 120.65 116.84))
+  (wire (pts (xy 120.65 95.25) (xy 114.3 95.25))
     (stroke (width 0) (type default) (color 0 0 0 0))
   )
@@
     (stroke (width 0) (type default) (color 0 0 0 0))
   )
-  (wire (pts (xy 111.76 107.95) (xy 111.76 102.87))
-    (stroke (width 0) (type default) (color 0 0 0 0))
-  )
   (wire (pts (xy 180.34 102.87) (xy 180.34 116.84))
     (stroke (width 0) (type default) (color 0 0 0 0))
@@
     (stroke (width 0) (type default) (color 0 0 0 0))
   )
-  (wire (pts (xy 120.65 105.41) (xy 116.84 105.41))
-    (stroke (width 0) (type default) (color 0 0 0 0))
-  )
-  (wire (pts (xy 107.95 102.87) (xy 111.76 102.87))
+  (wire (pts (xy 107.95 102.87) (xy 114.3 102.87))
     (stroke (width 0) (type default) (color 0 0 0 0))
   )
@@
     (stroke (width 0) (type default) (color 0 0 0 0))
   )
-  (wire (pts (xy 116.84 100.33) (xy 120.65 100.33))
+  (wire (pts (xy 114.3 102.87) (xy 120.65 102.87))
+    (stroke (width 0) (type default) (color 0 0 0 0))
+  )
+  (wire (pts (xy 114.3 95.25) (xy 114.3 102.87))
     (stroke (width 0) (type default) (color 0 0 0 0))
   )
@@
     (stroke (width 0) (type default) (color 0 0 0 0))
   )
+  (wire (pts (xy 118.11 92.71) (xy 118.11 99.06))
+    (stroke (width 0) (type default) (color 0 0 0 0))
+  )
   (wire (pts (xy 166.37 69.85) (xy 166.37 81.28))
     (stroke (width 0) (type default) (color 0 0 0 0))
@@
     (stroke (width 0) (type default) (color 0 0 0 0))
   )
-  (wire (pts (xy 116.84 92.71) (xy 139.7 92.71))
+  (wire (pts (xy 118.11 92.71) (xy 139.7 92.71))
+    (stroke (width 0) (type default) (color 0 0 0 0))
+  )
+  (wire (pts (xy 120.65 97.79) (xy 120.65 99.06))
     (stroke (width 0) (type default) (color 0 0 0 0))
   )
@@
     (stroke (width 0) (type default) (color 0 0 0 0))
   )
-  (wire (pts (xy 111.76 107.95) (xy 120.65 107.95))
-    (stroke (width 0) (type default) (color 0 0 0 0))
-  )
-  (wire (pts (xy 116.84 105.41) (xy 116.84 100.33))
+  (wire (pts (xy 120.65 99.06) (xy 120.65 100.33))
     (stroke (width 0) (type default) (color 0 0 0 0))
   )
@@
     (stroke (width 0) (type default) (color 0 0 0 0))
   )
-  (wire (pts (xy 116.84 92.71) (xy 116.84 100.33))
+  (wire (pts (xy 120.65 107.95) (xy 120.65 116.84))
     (stroke (width 0) (type default) (color 0 0 0 0))
   )
@@
     (pin "3")
   )
-  (symbol (lib_id "Connector:AudioJack3_SwitchTR") (at 125.73 107.95 180) (unit 1)
+  (symbol (lib_id "SnapEDA:SJ-43504-SMT-TR") (at 125.73 102.87 180) (unit 1)
     (in_bom yes) (on_board yes) (fields_autoplaced)
-    (property "Reference" "J1" (id 0) (at 133.35 103.5049 0)
+    (property "Reference" "J1" (id 0) (at 135.89 101.5999 0)
       (effects (font (size 1.27 1.27)) (justify right))
     )
-    (property "Value" "Audio" (id 1) (at 133.35 106.0449 0)
-      (effects (font (size 1.27 1.27)) (justify right))
-    )
-    (property "Footprint" "PET:STX31205B" (id 2) (at 125.73 107.95 0)
-      (effects (font (size 1.27 1.27)) hide)
-    )
-    (property "Datasheet" "https://www.mouser.com/datasheet/2/222/STX3120-334667.pdf" (id 3) (at 125.73 107.95 0)
-      (effects (font (size 1.27 1.27)) hide)
-    )
-    (property "MOUSER" "806-STX-3120-5B" (id 4) (at 125.73 107.95 0)
-      (effects (font (size 1.27 1.27)) hide)
-    )
-    (property "MPN" "STX-3120-5B" (id 5) (at 125.73 107.95 0)
-      (effects (font (size 1.27 1.27)) hide)
-    )
-    (pin "R")
-    (pin "RN")
-    (pin "S")
-    (pin "T")
-    (pin "TN")
+    (property "Value" "SJ-43504-SMT-TR" (id 1) (at 135.89 101.5999 0)
+      (effects (font (size 1.27 1.27)) (justify right) hide)
+    )
+    (property "Footprint" "SnapEDA:CUI_SJ-43504-SMT-TR" (id 2) (at 125.73 102.87 0)
+      (effects (font (size 1.27 1.27)) (justify left bottom) hide)
+    )
+    (property "Datasheet" "https://www.mouser.com/datasheet/2/670/sj_43504_smt_tr-1779335.pdf" (id 3) (at 125.73 102.87 0)
+      (effects (font (size 1.27 1.27)) (justify left bottom) hide)
+    )
+    (property "PARTREV" "10/08/2019" (id 4) (at 125.73 102.87 0)
+      (effects (font (size 1.27 1.27)) (justify left bottom) hide)
+    )
+    (property "SNAPEDA_PN" "SJ-43504-SMT-TR" (id 5) (at 125.73 102.87 0)
+      (effects (font (size 1.27 1.27)) (justify left bottom) hide)
+    )
+    (property "MANUFACTURER" "CUI Devices" (id 6) (at 125.73 102.87 0)
+      (effects (font (size 1.27 1.27)) (justify left bottom) hide)
+    )
+    (property "MAXIMUM_PACKAGE_HEIGHT" "3.3 mm" (id 7) (at 125.73 102.87 0)
+      (effects (font (size 1.27 1.27)) (justify left bottom) hide)
+    )
+    (property "STANDARD" "Manufacturer Recommendations" (id 8) (at 125.73 102.87 0)
+      (effects (font (size 1.27 1.27)) (justify left bottom) hide)
+    )
+    (property "MOUSER" "490-SJ-43504-SMT-TR" (id 9) (at 135.89 102.8699 0)
+      (effects (font (size 1.27 1.27)) (justify right) hide)
+    )
+    (pin "1")
+    (pin "2")
+    (pin "3")
+    (pin "4")
+    (pin "5")
+    (pin "6")
   )
   (symbol (lib_id "power:GND") (at 24.13 182.88 0) (unit 1)

Commit message: hw: routing (excluding MCU)
Parts:
- J1: LCSC (none) -> C319101
Changed lines of the file:
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@@
+    (stroke (width 0) (type default) (color 0 0 0 0))
+  )
+  (wire (pts (xy 166.37 95.25) (xy 182.88 95.25))
     (stroke (width 0) (type default) (color 0 0 0 0))
   )
@@
   )
   (wire (pts (xy 166.37 91.44) (xy 166.37 95.25))
-    (stroke (width 0) (type default) (color 0 0 0 0))
-  )
-  (wire (pts (xy 166.37 95.25) (xy 182.88 95.25))
     (stroke (width 0) (type default) (color 0 0 0 0))
   )
@@
       (effects (font (size 1.27 1.27)) (justify right) hide)
     )
+    (property "LCSC" "C319101" (id 10) (at 125.73 102.87 0)
+      (effects (font (size 1.27 1.27)) hide)
+    )
     (pin "1")

Commit message: hw: routable (wip)
Parts:
- added NT9: +6V, PET:NetTie-2_SMD_Pad_1.6_to_0.4mm, symbol Device:NetTie_2
Connections:
- net +6V: now also NT9.2
- new net PD_6V: NT9.1
Changed lines of the file:
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@@
+    (stroke (width 0) (type default) (color 0 0 0 0))
+  )
+  (wire (pts (xy 168.91 69.85) (xy 166.37 69.85))
     (stroke (width 0) (type default) (color 0 0 0 0))
   )
@@
     (stroke (width 0) (type default) (color 0 0 0 0))
   )
+  (wire (pts (xy 176.53 69.85) (xy 173.99 69.85))
+    (stroke (width 0) (type default) (color 0 0 0 0))
+  )
   (wire (pts (xy 24.13 176.53) (xy 24.13 175.26))
     (stroke (width 0) (type default) (color 0 0 0 0))
@@
   )
   (wire (pts (xy 114.3 95.25) (xy 114.3 102.87))
+    (stroke (width 0) (type default) (color 0 0 0 0))
+  )
+  (wire (pts (xy 176.53 67.31) (xy 176.53 69.85))
     (stroke (width 0) (type default) (color 0 0 0 0))
   )
@@
     (pin "1")
   )
+  (symbol (lib_id "Device:NetTie_2") (at 171.45 69.85 0) (mirror y) (unit 1)
+    (in_bom yes) (on_board yes)
+    (property "Reference" "NT9" (id 0) (at 171.45 67.31 0)
+      (effects (font (size 1.27 1.27)) hide)
+    )
+    (property "Value" "+6V" (id 1) (at 171.45 67.31 0)
+      (effects (font (size 1.27 1.27)) hide)
+    )
+    (property "Footprint" "PET:NetTie-2_SMD_Pad_1.6_to_0.4mm" (id 2) (at 171.45 69.85 0)
+      (effects (font (size 1.27 1.27)) hide)
+    )
+    (property "Datasheet" "~" (id 3) (at 171.45 69.85 0)
+      (effects (font (size 1.27 1.27)) hide)
+    )
+    (pin "1")
+    (pin "2")
+  )
   (symbol (lib_id "Device:R_Small") (at 154.94 102.87 0) (unit 1)
     (in_bom yes) (on_board yes)
@@
       (effects (font (size 1.27 1.27)) hide)
     )
+    (pin "1")
+  )
+  (symbol (lib_id "PET:PD_6V") (at 176.53 67.31 0) (unit 1)
+    (in_bom yes) (on_board yes)
+    (property "Reference" "#PWR0197" (id 0) (at 176.53 71.12 0)
+      (effects (font (size 1.27 1.27)) hide)
+    )
+    (property "Value" "PD_6V" (id 1) (at 176.53 62.23 0))
+    (property "Footprint" "" (id 2) (at 176.53 67.31 0)
+      (effects (font (size 1.27 1.27)) hide)
+    )
+    (property "Datasheet" "" (id 3) (at 176.53 67.31 0)
+      (effects (font (size 1.27 1.27)) hide)
+    )

Commit message: hw: wip
Parts:
- removed NT9: +6V, PET:NetTie-2_SMD_Pad_1.6_to_0.4mm, symbol Device:NetTie_2
- added NT24: GND, PET:NetTie-2_SMD_Pad_1.6_to_0.4mm, symbol Device:NetTie_2
Connections:
- net GND: now also NT24.2; no longer J8.1 (Pin_1), J8.3 (Pin_3), R62.2
- new net PD_GND: J8.1 (Pin_1), J8.3 (Pin_3), NT24.1, R62.2

Commit message: hw: larger schematic pages, routed w/netties
Parts:
- added NT9: +6V, PET:NetTie-2_SMD_Pad_1.6_to_0.4mm, symbol Device:NetTie_2
Connections:
- net +6V: no longer names the net of C30.1, Q2.3 (C), R53.1
- net +6V: now also NT9.2
- new net PD_6V: NT9.1
Other:
- moved on the sheet: C30, C31, J1, J8, Q2, R53, R61, R62, RV1

Commit message: hw: wip
Parts:
- NT24, NT9: symbol Device:NetTie_2 -> PET:PowerTie_2
Connections:
- net GND: no longer J1.1, NT24.2, R61.2, RV1.1
- new net: J1.1, NT24.2, R61.2, RV1.1
Changed lines of the file:
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@@
-    (stroke (width 0) (type default) (color 0 0 0 0))
-  )
-  (wire (pts (xy 224.79 154.94) (xy 224.79 157.48))
     (stroke (width 0) (type default) (color 0 0 0 0))
   )
@@
     (pin "2")
   )
-  (symbol (lib_id "Device:NetTie_2") (at 231.14 154.94 0) (mirror y) (unit 1)
+  (symbol (lib_id "PET:PowerTie_2") (at 231.14 154.94 0) (mirror y) (unit 1)
     (in_bom yes) (on_board yes)
     (property "Reference" "NT24" (id 0) (at 231.14 152.4 0)
@@
     (pin "1")
   )
-  (symbol (lib_id "Device:NetTie_2") (at 250.19 107.95 0) (mirror y) (unit 1)
+  (symbol (lib_id "PET:PowerTie_2") (at 250.19 107.95 0) (mirror y) (unit 1)
     (in_bom yes) (on_board yes)
     (property "Reference" "NT9" (id 0) (at 250.19 105.41 0)
@@
     (pin "3")
   )
-  (symbol (lib_id "power:GND") (at 224.79 157.48 0) (mirror y) (unit 1)
-    (in_bom yes) (on_board yes)
-    (property "Reference" "#PWR0118" (id 0) (at 224.79 163.83 0)
-      (effects (font (size 1.27 1.27)) hide)
-    )
-    (property "Value" "GND" (id 1) (at 224.663 161.8742 0))
-    (property "Footprint" "" (id 2) (at 224.79 157.48 0)
-      (effects (font (size 1.27 1.27)) hide)
-    )
-    (property "Datasheet" "" (id 3) (at 224.79 157.48 0)
-      (effects (font (size 1.27 1.27)) hide)
-    )
-    (pin "1")
-  )
   (symbol (lib_id "PET:PD_6V") (at 255.27 105.41 0) (unit 1)

Commit message: jlcpcb - 1/19
Parts:
- added LS1: Speaker, SnapEDA:XDCR_AT-1224-TWT-5V-2-R, symbol Device:Speaker
- C31: value 1u -> 1u 25V
- J1: Alt-LCSC (none) -> C319101; LCSC C319101 -> (none); MANUFACTURER CUI Devices -> (none); MAXIMUM_PACKAGE_HEIGHT 3.3 mm -> (none); PARTREV 10/08/2019 -> (none); SNAPEDA_PN SJ-43504-SMT-TR -> (none); STANDARD Manufacturer Recommendations -> (none)
- R61: value 4.7k -> 4k7
Connections:
- net PD_GND: now also LS1.2
- net at J8.4 (Pin_4), Q2.2 (E), R62.1: now also LS1.1
Other:
- note added: "+"
- note added: "-"
- title: (none) -> Audio
Changed lines of the file:
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@@
 (kicad_sch (version 20211123) (generator eeschema)
   (paper "B")
+  (title_block
+    (title "Audio")
+  )
   (junction (at 236.22 133.35) (diameter 0) (color 0 0 0 0)
   )
@@
   )
   (junction (at 184.15 140.97) (diameter 0) (color 0 0 0 0)
+  )
+  (junction (at 250.19 133.35) (diameter 0) (color 0 0 0 0)
   )
   (junction (at 190.5 137.16) (diameter 0) (color 0 0 0 0)
@@
     (stroke (width 0) (type default) (color 0 0 0 0))
   )
+  (wire (pts (xy 250.19 128.27) (xy 250.19 133.35))
+    (stroke (width 0) (type default) (color 0 0 0 0))
+  )
   (wire (pts (xy 236.22 143.51) (xy 236.22 154.94))
     (stroke (width 0) (type default) (color 0 0 0 0))
@@
     (stroke (width 0) (type default) (color 0 0 0 0))
   )
+  (wire (pts (xy 273.05 154.94) (xy 250.19 154.94))
+    (stroke (width 0) (type default) (color 0 0 0 0))
+  )
   (wire (pts (xy 250.19 140.97) (xy 250.19 154.94))
     (stroke (width 0) (type default) (color 0 0 0 0))
@@
     (stroke (width 0) (type default) (color 0 0 0 0))
   )
+  (wire (pts (xy 273.05 135.89) (xy 273.05 128.27))
+    (stroke (width 0) (type default) (color 0 0 0 0))
+  )
   (wire (pts (xy 190.5 135.89) (xy 190.5 137.16))
     (stroke (width 0) (type default) (color 0 0 0 0))
@@
     (stroke (width 0) (type default) (color 0 0 0 0))
   )
+  (wire (pts (xy 273.05 138.43) (xy 273.05 154.94))
+    (stroke (width 0) (type default) (color 0 0 0 0))
+  )
   (wire (pts (xy 190.5 137.16) (xy 190.5 138.43))
     (stroke (width 0) (type default) (color 0 0 0 0))
   )
+  (wire (pts (xy 273.05 128.27) (xy 250.19 128.27))
+    (stroke (width 0) (type default) (color 0 0 0 0))
+  )
+  (wire (pts (xy 250.19 133.35) (xy 252.73 133.35))
+    (stroke (width 0) (type default) (color 0 0 0 0))
+  )
   (wire (pts (xy 190.5 146.05) (xy 190.5 154.94))
     (stroke (width 0) (type default) (color 0 0 0 0))
@@
     (stroke (width 0) (type default) (color 0 0 0 0))
   )
-  (wire (pts (xy 236.22 133.35) (xy 252.73 133.35))
-    (stroke (width 0) (type default) (color 0 0 0 0))
+  (wire (pts (xy 236.22 133.35) (xy 250.19 133.35))
+    (stroke (width 0) (type default) (color 0 0 0 0))
+  )
+  (text "+" (at 276.225 137.16 0)
+    (effects (font (size 1.27 1.27)) (justify left bottom))
+  )
+  (text "-" (at 276.225 139.065 0)
+    (effects (font (size 1.27 1.27)) (justify left bottom))
   )
   (hierarchical_label "AUDIO" (shape input) (at 166.37 140.97 180)
@@
       (effects (font (size 1.27 1.27)) hide)
     )
-    (property "Datasheet" "~" (id 3) (at 243.84 111.76 0)
+    (property "Datasheet" "https://datasheet.lcsc.com/lcsc/1810191219_Samsung-Electro-Mechanics-CL05B104KO5NNNC_C1525.pdf" (id 3) (at 243.84 111.76 0)
       (effects (font (size 1.27 1.27)) hide)
     )
@@
       (effects (font (size 1.27 1.27)) hide)
     )
-    (property "Datasheet" "~" (id 3) (at 236.22 140.97 0)
+    (property "Datasheet" "https://datasheet.lcsc.com/lcsc/2205311830_UNI-ROYAL-Uniroyal-Elec-0805W8F3300T5E_C17630.pdf" (id 3) (at 236.22 140.97 0)
       (effects (font (size 1.27 1.27)) hide)
     )
@@
       (effects (font (size 1.27 1.27) italic) (justify left) hide)
     )
-    (property "Datasheet" "https://www.onsemi.com/pub/Collateral/2N3903-D.PDF" (id 3) (at 233.68 124.46 0)
+    (property "Datasheet" "https://datasheet.lcsc.com/lcsc/2207041900_Jiangsu-Changjing-Electronics-Technology-Co---Ltd--MMBT3904_C20526.pdf" (id 3) (at 233.68 124.46 0)
       (effects (font (size 1.27 1.27)) (justify left) hide)
     )
@@
       (effects (font (size 1.27 1.27)) (justify left bottom) hide)
     )
-    (property "PARTREV" "10/08/2019" (id 4) (at 195.58 140.97 0)
-      (effects (font (size 1.27 1.27)) (justify left bottom) hide)
-    )
-    (property "SNAPEDA_PN" "SJ-43504-SMT-TR" (id 5) (at 195.58 140.97 0)
-      (effects (font (size 1.27 1.27)) (justify left bottom) hide)
-    )
-    (property "MANUFACTURER" "CUI Devices" (id 6) (at 195.58 140.97 0)
-      (effects (font (size 1.27 1.27)) (justify left bottom) hide)
-    )
-    (property "MAXIMUM_PACKAGE_HEIGHT" "3.3 mm" (id 7) (at 195.58 140.97 0)
-      (effects (font (size 1.27 1.27)) (justify left bottom) hide)
-    )
-    (property "STANDARD" "Manufacturer Recommendations" (id 8) (at 195.58 140.97 0)
-      (effects (font (size 1.27 1.27)) (justify left bottom) hide)
-    )
     (property "MOUSER" "490-SJ-43504-SMT-TR" (id 9) (at 205.74 140.9699 0)
       (effects (font (size 1.27 1.27)) (justify right) hide)
     )
-    (property "LCSC" "C319101" (id 10) (at 195.58 140.97 0)
+    (property "Alt-LCSC" "C319101" (id 10) (at 195.58 140.97 0)
       (effects (font (size 1.27 1.27)) hide)
     )
@@
       (effects (font (size 1.27 1.27)) (justify left))
     )
-    (property "Value" "4.7k" (id 1) (at 226.2886 142.113 0)
+    (property "Value" "4k7" (id 1) (at 226.2886 142.113 0)
       (effects (font (size 1.27 1.27)) (justify left))
     )
@@
       (effects (font (size 1.27 1.27)) hide)
     )
-    (property "Datasheet" "~" (id 3) (at 224.79 140.97 0)
+    (property "Datasheet" "https://datasheet.lcsc.com/lcsc/2206010045_UNI-ROYAL-Uniroyal-Elec-0402WGF4701TCE_C25900.pdf" (id 3) (at 224.79 140.97 0)
       (effects (font (size 1.27 1.27)) hide)
     )
@@
       (effects (font (size 1.27 1.27)) hide)
     )
-    (property "Datasheet" "~" (id 3) (at 224.79 115.57 0)
+    (property "Datasheet" "https://datasheet.lcsc.com/lcsc/2206010100_UNI-ROYAL-Uniroyal-Elec-0402WGF2202TCE_C25768.pdf" (id 3) (at 224.79 115.57 0)
       (effects (font (size 1.27 1.27)) hide)
     )
@@
       (effects (font (size 1.27 1.27)) (justify left))
     )
-    (property "Value" "1u" (id 1) (at 176.53 137.795 90)
+    (property "Value" "1u 25V" (id 1) (at 176.53 137.795 90)
       (effects (font (size 1.27 1.27)) (justify left))
     )
@@
       (effects (font (size 1.27 1.27)) hide)
     )
-    (property "Datasheet" "~" (id 3) (at 175.26 140.97 0)
+    (property "Datasheet" "https://datasheet.lcsc.com/lcsc/1811091611_Samsung-Electro-Mechanics-CL05A105KA5NQNC_C52923.pdf" (id 3) (at 175.26 140.97 0)
       (effects (font (size 1.27 1.27)) hide)
     )
@@
     (pin "3")
   )
+  (symbol (lib_id "Device:Speaker") (at 278.13 135.89 0) (unit 1)
+    (in_bom yes) (on_board yes) (fields_autoplaced)
+    (property "Reference" "LS1" (id 0) (at 283.21 135.8899 0)
+      (effects (font (size 1.27 1.27)) (justify left))
+    )
+    (property "Value" "Speaker" (id 1) (at 283.21 138.4299 0)
+      (effects (font (size 1.27 1.27)) (justify left))
+    )
+    (property "Footprint" "SnapEDA:XDCR_AT-1224-TWT-5V-2-R" (id 2) (at 278.13 140.97 0)
+      (effects (font (size 1.27 1.27)) hide)
+    )
+    (property "Datasheet" "https://www.mouser.com/datasheet/2/334/AT-1224-TWT-5V-2-R-532234.pdf" (id 3) (at 277.876 137.16 0)
+      (effects (font (size 1.27 1.27)) hide)
+    )
+    (property "MOUSER" "665-AT1224TWT5V2R" (id 4) (at 278.13 135.89 0)
+      (effects (font (size 1.27 1.27)) hide)
+    )
+    (property "MPN" "AT-1224-TWT-5V-2-R" (id 5) (at 278.13 135.89 0)
+      (effects (font (size 1.27 1.27)) hide)
+    )
+    (pin "1")
+    (pin "2")
+  )
   (symbol (lib_id "PET:PD_6V") (at 255.27 105.41 0) (unit 1)
