File: hw/Mainboard/FPGA.kicad_sch (KiCad schematic)
At the start: 43 parts, among them J19 PROG, J21 FPGA-P4, J23 FPGA_P2, J24 FPGA_P3, Q4 MMBT3904, SW5 CONFIG, U21 T8Q144C3

Commit message: hw: move DVI to separate hierarchical sheet, fix buses, annotate power
Parts:
- removed NT39: +3V3, PET:NetTie-2_SMD_Pad_1.6_to_0.4mm, symbol Device:NetTie_2
- removed PT3: PowerTie_2, PET:NetTie-2_SMD_Pad_1.6_to_0.4mm, symbol Device:NetTie_2
Connections:
- net PD_GND is gone; now on net GND: J19.7 (Pin_7)
- net MCU_CEC renamed CEC
Changed lines of the file:
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@@
   (junction (at 62.23 175.26) (diameter 0) (color 0 0 0 0)
   )
-  (junction (at 38.1 160.02) (diameter 0) (color 0 0 0 0)
-  )
   (junction (at 62.23 167.64) (diameter 0) (color 0 0 0 0)
   )
@@
   (junction (at 383.54 203.2) (diameter 0) (color 0 0 0 0)
   )
-  (junction (at 26.67 160.02) (diameter 0) (color 0 0 0 0)
-  )
   (junction (at 63.5 259.08) (diameter 0) (color 0 0 0 0)
   )
@@
     (stroke (width 0) (type default) (color 0 0 0 0))
   )
-  (wire (pts (xy 26.67 162.56) (xy 30.48 162.56))
-    (stroke (width 0) (type default) (color 0 0 0 0))
-  )
   (wire (pts (xy 38.1 252.73) (xy 38.1 251.46))
     (stroke (width 0) (type default) (color 0 0 0 0))
@@
     (stroke (width 0) (type default) (color 0 0 0 0))
   )
-  (wire (pts (xy 38.1 160.02) (xy 38.1 162.56))
-    (stroke (width 0) (type default) (color 0 0 0 0))
-  )
   (wire (pts (xy 63.5 259.08) (xy 76.2 259.08))
     (stroke (width 0) (type default) (color 0 0 0 0))
@@
     (stroke (width 0) (type default) (color 0 0 0 0))
   )
-  (wire (pts (xy 35.56 160.02) (xy 38.1 160.02))
-    (stroke (width 0) (type default) (color 0 0 0 0))
-  )
   (wire (pts (xy 66.04 54.61) (xy 67.31 54.61))
     (stroke (width 0) (type default) (color 0 0 0 0))
@@
     (stroke (width 0) (type default) (color 0 0 0 0))
   )
-  (wire (pts (xy 26.67 160.02) (xy 26.67 158.75))
-    (stroke (width 0) (type default) (color 0 0 0 0))
-  )
   (bus (pts (xy 414.02 81.28) (xy 414.02 101.6))
     (stroke (width 0) (type default) (color 0 0 0 0))
@@
     (stroke (width 0) (type default) (color 0 0 0 0))
   )
-  (wire (pts (xy 26.67 160.02) (xy 26.67 162.56))
-    (stroke (width 0) (type default) (color 0 0 0 0))
-  )
   (wire (pts (xy 368.3 114.3) (xy 377.19 114.3))
     (stroke (width 0) (type default) (color 0 0 0 0))
@@
     (stroke (width 0) (type default) (color 0 0 0 0))
   )
-  (wire (pts (xy 35.56 162.56) (xy 38.1 162.56))
-    (stroke (width 0) (type default) (color 0 0 0 0))
-  )
   (wire (pts (xy 175.26 57.15) (xy 153.67 57.15))
     (stroke (width 0) (type default) (color 0 0 0 0))
@@
     (stroke (width 0) (type default) (color 0 0 0 0))
   )
-  (wire (pts (xy 30.48 160.02) (xy 26.67 160.02))
-    (stroke (width 0) (type default) (color 0 0 0 0))
-  )
   (text "BD0" (at 153.67 57.15 0)
     (effects (font (size 1.27 1.27)) (justify left bottom))
@@
     (effects (font (size 1.27 1.27)) (justify right))
   )
-  (hierarchical_label "RAM_A" (shape output) (at 363.22 127 180)
+  (hierarchical_label "{RAM_A}" (shape output) (at 363.22 127 180)
     (effects (font (size 1.27 1.27)) (justify right))
   )
@@
     (effects (font (size 1.27 1.27)) (justify left))
   )
-  (hierarchical_label "MCU_CEC" (shape bidirectional) (at 67.31 67.31 180)
+  (hierarchical_label "CEC" (shape bidirectional) (at 67.31 67.31 180)
     (effects (font (size 1.27 1.27)) (justify right))
   )
@@
     (pin "2")
   )
+  (symbol (lib_id "power:GND") (at 160.02 62.23 0) (unit 1)
+    (in_bom yes) (on_board yes)
+    (property "Reference" "#PWR036" (id 0) (at 160.02 68.58 0)
+      (effects (font (size 1.27 1.27)) hide)
+    )
+    (property "Value" "GND" (id 1) (at 160.147 66.6242 0))
+    (property "Footprint" "" (id 2) (at 160.02 62.23 0)
+      (effects (font (size 1.27 1.27)) hide)
+    )
+    (property "Datasheet" "" (id 3) (at 160.02 62.23 0)
+      (effects (font (size 1.27 1.27)) hide)
+    )
+    (pin "1")
+  )
   (symbol (lib_id "power:+3V3") (at 163.83 30.48 0) (unit 1)
     (in_bom yes) (on_board yes)
@@
     (pin "2")
   )
-  (symbol (lib_id "Device:NetTie_2") (at 33.02 162.56 0) (unit 1)
-    (in_bom yes) (on_board yes) (fields_autoplaced)
-    (property "Reference" "PT3" (id 0) (at 33.02 160.655 0)
-      (effects (font (size 1.27 1.27)) hide)
-    )
-    (property "Value" "PowerTie_2" (id 1) (at 33.02 164.465 0)
-      (effects (font (size 1.27 1.27)) hide)
-    )
-    (property "Footprint" "PET:NetTie-2_SMD_Pad_1.6_to_0.4mm" (id 2) (at 33.02 162.56 0)
-      (effects (font (size 1.27 1.27)) hide)
-    )
-    (property "Datasheet" "~" (id 3) (at 33.02 162.56 0)
-      (effects (font (size 1.27 1.27)) hide)
-    )
-    (pin "1")
-    (pin "2")
-  )
   (symbol (lib_id "power:GND") (at 300.99 242.57 0) (unit 1)
     (in_bom yes) (on_board yes)
@@
     (pin "1")
   )
-  (symbol (lib_id "PET:PD_GND") (at 160.02 62.23 0) (unit 1)
-    (in_bom yes) (on_board yes) (fields_autoplaced)
-    (property "Reference" "#PWR036" (id 0) (at 160.02 68.58 0)
-      (effects (font (size 1.27 1.27)) hide)
-    )
-    (property "Value" "PD_GND" (id 1) (at 160.02 67.31 0))
-    (property "Footprint" "" (id 2) (at 160.02 62.23 0)
-      (effects (font (size 1.27 1.27)) hide)
-    )
-    (property "Datasheet" "" (id 3) (at 160.02 62.23 0)
-      (effects (font (size 1.27 1.27)) hide)
-    )
-    (pin "1")
-  )
   (symbol (lib_id "Device:C_Small") (at 95.25 237.49 0) (unit 1)
     (in_bom yes) (on_board yes)
@@
     (pin "1")
   )
-  (symbol (lib_id "Device:NetTie_2") (at 33.02 160.02 0) (unit 1)
-    (in_bom yes) (on_board yes)
-    (property "Reference" "NT39" (id 0) (at 33.02 157.48 0)
-      (effects (font (size 1.27 1.27)) hide)
-    )
-    (property "Value" "+3V3" (id 1) (at 33.02 157.48 0)
-      (effects (font (size 1.27 1.27)) hide)
-    )
-    (property "Footprint" "PET:NetTie-2_SMD_Pad_1.6_to_0.4mm" (id 2) (at 33.02 160.02 0)
-      (effects (font (size 1.27 1.27)) hide)
-    )
-    (property "Datasheet" "~" (id 3) (at 33.02 160.02 0)
-      (effects (font (size 1.27 1.27)) hide)
-    )
-    (pin "1")
-    (pin "2")
-  )
   (symbol (lib_id "power:GND") (at 45.72 66.04 0) (mirror y) (unit 1)
     (in_bom yes) (on_board yes) (fields_autoplaced)
@@
     (pin "2")
   )
-  (symbol (lib_id "PET:PD_3V3") (at 26.67 158.75 0) (unit 1)
-    (in_bom yes) (on_board yes) (fields_autoplaced)
-    (property "Reference" "#PWR045" (id 0) (at 26.67 162.56 0)
-      (effects (font (size 1.27 1.27)) hide)
-    )
-    (property "Value" "PD_3V3" (id 1) (at 26.67 153.67 0))
-    (property "Footprint" "" (id 2) (at 26.67 158.75 0)
-      (effects (font (size 1.27 1.27)) hide)
-    )
-    (property "Datasheet" "" (id 3) (at 26.67 158.75 0)
-      (effects (font (size 1.27 1.27)) hide)
-    )
-    (pin "1")
-  )
   (symbol (lib_id "power:+3V3") (at 38.1 158.75 0) (unit 1)

Commit message: hw: wip
Parts:
- removed C70: 1u 25V, Capacitor_SMD:C_0402_1005Metric, symbol Device:C_Small
- removed C74, C82: 100n, Capacitor_SMD:C_0402_1005Metric, symbol Device:C_Small
- removed J24: FPGA_P3, Connector_PinHeader_2.54mm:PinHeader_2x14_P2.54mm_Vertical, symbol Connector_Generic:Conn_02x14_Odd_Even
- removed NT44, NT8: +3V3, PET:NetTie-2_SMD_Pad_0.4_to_0.28mm, symbol PET:PowerTie_2
- added J24: Conn_02x15_Odd_Even, Connector_PinHeader_2.54mm:PinHeader_2x15_P2.54mm_Vertical, symbol Connector_Generic:Conn_02x15_Odd_Even
- C60, C69: value 1u 25V -> 1u
- C65, C66, C67, C68, C78, C79: value 10n 50V -> 10n
- C77, C80: value 10n 50V -> 100n; LCSC C15195 -> C1525
Connections:
- net A16 is gone; now on net A15: U21.77 (GPIOR_154)
- net FPGA_GND is gone; now on net GND: U21.1 (GND), U21.104 (GND), U21.108 (GND), U21.120 (GND), U21.121 (GND), U21.126 (GND), U21.127 (GND), U21.129 (GND), U21.133 (GND), U21.37 (GND), U21.44 (GND), U21.5 (GND), U21.50 (GND), U21.64 (GND), U21.9 (GND), U21.94 (GND)
- net FPGA_VCC is gone; now on net +1V2: C60.1, C61.1, C62.1, C63.1, C64.1, C65.1, C66.1, C67.1, C68.1, U21.125 (VCC), U21.128 (VCC), U21.13 (VCC), U21.130 (VCC), U21.22 (VCC), U21.49 (VCC), U21.57 (VCC), U21.85 (VCC), U21.96 (VCC)
- net +3V3: no longer J19.3 (Pin_3)
- net A0: now also U21.70 (GPIOB_RXP12_EXTFB0), J24.1 (Pin_1); no longer U21.65 (GPIOB_RXN07)
- net A1: now also U21.72 (GPIOB_CLKN0), J24.3 (Pin_3); no longer U21.67 (GPIOB_RXP10)
- net A10: now also J24.21 (Pin_21)
- net A11: now also J24.25 (Pin_25)
- net A12: now also U21.69 (GPIOB_RXN12_EXTFB0), J24.2 (Pin_2); no longer U21.66 (GPIOB_RXP07)
- net A13: now also U21.71 (GPIOB_CLKP0), J24.4 (Pin_4); no longer U21.68 (GPIOB_RXN10)
- net A14: now also U21.76 (GPIOR_155), J24.6 (Pin_6); no longer U21.70 (GPIOB_RXP12_EXTFB0)
- net A15: now also J24.8 (Pin_8); no longer U21.72 (GPIOB_CLKN0)
- net A2: now also U21.75 (GPIOR_157_PLLIN), J24.5 (Pin_5); no longer U21.69 (GPIOB_RXN12_EXTFB0)
- net A3: now also U21.81 (GPIOR_139), J24.7 (Pin_7); no longer U21.71 (GPIOB_CLKP0)
- net A4: now also U21.83 (GPIOR_136_CDI16), J24.9 (Pin_9); no longer U21.76 (GPIOR_155)
- net A5: now also U21.86 (GPIOR_133_CDI18), J24.11 (Pin_11); no longer U21.81 (GPIOR_139)
- net A6: now also U21.89 (GPIOR_129_CTRL10), J24.13 (Pin_13); no longer U21.83 (GPIOR_136_CDI16)
- net A7: now also U21.92 (GPIOR_125_CLK10), J24.15 (Pin_15); no longer U21.86 (GPIOR_133_CDI18)
- net A8: now also J24.17 (Pin_17)
- net A9: now also J24.19 (Pin_19)
- net BE: now also U21.66 (GPIOB_RXP07); no longer U21.59 (GPIOB_RXN02)
- net CBUS0: now also RN15.3 (R3.1); no longer RN15.1 (R1.1)
- net CBUS2: now also RN15.1 (R1.1); no longer RN15.3 (R3.1)
- net CDONE: now also J19.16 (Pin_16); no longer J19.10 (Pin_10)
- net CSI: now also R27.1; no longer RN15.4 (R4.1)
- net D0: now also U21.87 (GPIOR_132_CDI19), J24.14 (Pin_14); no longer U21.82 (GPIOR_138)
- net D1: now also U21.90 (GPIOR_128_CTRL11), J24.16 (Pin_16); no longer U21.84 (GPIOR_135_CDI17)
- net D2: now also U21.93 (GPIOR_123_CLK12_CDI20), J24.18 (Pin_18); no longer U21.87 (GPIOR_132_CDI19)
- net D3: now also J24.20 (Pin_20)
- net D4: now also J24.22 (Pin_22)
- net D5: now also J24.24 (Pin_24)
- net D6: now also J24.26 (Pin_26)
- net D7: now also J24.28 (Pin_28)
- net DIAG: now also J23.13 (Pin_13), U21.48 (GPIOB_TXN09); no longer J23.12 (Pin_12), U21.42 (GPIOB_TXP04)
- net GND: now also J19.1 (Pin_1); no longer J19.7 (Pin_7)
- net GRAPHICS: now also J23.15 (Pin_15), U21.54 (GPIOB_TXN11); no longer J23.14 (Pin_14), U21.45 (GPIOB_TXP06)
- net HOLD: now also J19.15 (Pin_15); no longer J19.14 (Pin_14)
- net NSTATUS: now also J19.11 (Pin_11); no longer J19.5 (Pin_5)
- net RAM_A10: now also J24.23 (Pin_23)
- net RAM_A11: now also J24.27 (Pin_27)
- net RAM_A15: now also U21.82 (GPIOR_138), J24.10 (Pin_10); no longer J23.16 (Pin_16), U21.47 (GPIOB_TXP09)
- net RAM_A16: now also U21.84 (GPIOR_135_CDI17), J24.12 (Pin_12)
- net RDY: now also U21.59 (GPIOB_RXN02); no longer U21.54 (GPIOB_TXN11)
- net R~{W}: now also J24.30 (Pin_30)
- net SPI0_RX: no longer J19.2 (Pin_2)
- net SPI0_SCK: no longer J19.6 (Pin_6)
- net SPI0_TX: no longer J19.4 (Pin_4)
- net SPI0_~{CS}: now also J19.12 (Pin_12); no longer J19.8 (Pin_8)
- net SYNC: now also U21.68 (GPIOB_RXN10); no longer U21.61 (GPIOB_RXP03)
- net TCK: now also J19.2 (Pin_2), RN14.1 (R1.1); no longer J19.13 (Pin_13), RN14.2 (R2.1)
- net TDI: now also J19.4 (Pin_4), RN14.2 (R2.1); no longer J19.15 (Pin_15), RN14.3 (R3.1)
- net TDO: now also J19.6 (Pin_6); no longer J19.9 (Pin_9)
- net TMS: now also J19.8 (Pin_8), RN14.3 (R3.1); no longer J19.11 (Pin_11), RN14.1 (R1.1)
- net VIA_CB2: now also J23.14 (Pin_14), U21.53 (GPIOB_TXP11); no longer J23.13 (Pin_13), U21.43 (GPIOB_TXN04)
- net ~{CRESET}: now also J19.14 (Pin_14); no longer J19.12 (Pin_12)
- net ~{IRQ}: now also U21.61 (GPIOB_RXP03); no longer U21.56 (GPIOB_RXN00)
- net ~{ML}: now also U21.65 (GPIOB_RXN07); no longer U21.58 (GPIOB_RXP02)
- net ~{NMI}: now also U21.67 (GPIOB_RXP10); no longer U21.60 (GPIOB_RXN03)
- net ~{RAM_OE}: now also J23.16 (Pin_16), U21.55 (GPIOB_RXP00); no longer J23.15 (Pin_15), U21.46 (GPIOB_TXN06)
- net ~{RAM_WE}: now also U21.56 (GPIOB_RXN00); no longer U21.48 (GPIOB_TXN09)
- net ~{SO}: now also U21.60 (GPIOB_RXN03); no longer U21.55 (GPIOB_RXP00)
- net ~{SPI_ENA}: now also J19.13 (Pin_13); no longer J19.16 (Pin_16)
- net ~{TEST}: now also RN15.4 (R4.1); no longer R27.1
- net ~{VP}: now also U21.58 (GPIOB_RXP02); no longer U21.53 (GPIOB_TXP11)
- net MCU_CLK renamed FPGA_CLK
- new net SWCLK: J19.3 (Pin_3)
- new net SWD: J19.5 (Pin_5)
- new net UART_RX: J19.7 (Pin_7)
- new net UART_TX: J19.9 (Pin_9)
- no-connect marks 19 -> 14
Other:
- note added: "CDONE is open drain and requires pullup to enter user mode. TDO is terminated by the programmer at the receiving end."
- note added: "During configuration, all GPIO pins excluding LVDS as GPIO are configured in weak pull-up mode. The LVDS as GPIO pins are tri-stated without a pull-up or pull-down resistor."
- note added: "Minimum decoupling caps is one 100nF and one 10nF"
- note added: "Pull ~{CRESET} low to reset FPGA until MCU is ready. Note that MCU drives ~{CRESET} through 10k resistor so it can be overridden by programmer when connected. Pull CSI high to enable FPGA configuration Pull TEST_N high to deactivate test mode Pull CBUS[2:0] high for SPI x1 Leave CBSEL[1:0] floating (not using multi-image) MCU config: MCU drives SS_N low to select passive SPI MCU transitions CRESE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"
- note removed: "AD0"
- note removed: "AD1"
- note removed: "AD2"
- note removed: "CDONE is open drain and requires pullup. Otherwise, FPGA will not enter user mode. TDO is terminated by the programmer at the receiving end."
- note removed: "Pull ~{CRESET} low to reset FPGA until MCU is ready. Note that MCU drives ~{CRESET} through 10k resistor so it can be overridden by programmer when connected. Pull CSI high to enable FPGA configuration Pull TEST_N high to deactivate test mode Pull CBUS[2:0] high for 1x SPI width Leave CBSEL[1:0] floating (not using multi-image) MCU config: MCU drives SS_N low to select passive SPI MCU transitions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"
- moved on the sheet: C69, C71, C72, C73, J19, R27, RN14, RN15

Commit message: wip: support 8x16 keyboard matrix
Parts:
- added J16: MCU, Connector_PinHeader_2.54mm:PinHeader_2x12_P2.54mm_Vertical, symbol Connector_Generic:Conn_02x12_Odd_Even
- added R68, R70, R71: 33, Resistor_SMD:R_0402_1005Metric, symbol Device:R_Small
Connections:
- net +3V3: now also J16.24 (Pin_24)
- net AUDIO: now also J23.5 (Pin_5); no longer J23.4 (Pin_4)
- net BE: now also J23.25 (Pin_25), U21.67 (GPIOB_RXP10); no longer J23.24 (Pin_24), U21.66 (GPIOB_RXP07)
- net CEC: now also U21.4 (GPIOL_54_CDI11), J16.21 (Pin_21); no longer U21.33 (GPIOL_05_CSO)
- net DIAG: now also J23.15 (Pin_15), U21.53 (GPIOB_TXP11); no longer J23.13 (Pin_13), U21.48 (GPIOB_TXN09)
- net FPGA_CLK: now also J21.16 (Pin_16); no longer J21.15 (Pin_15)
- net GND: now also J16.1 (Pin_1), J16.23 (Pin_23); no longer J21.12 (Pin_12), J23.27 (Pin_27), J23.3 (Pin_3)
- net GRAPHICS: now also J23.17 (Pin_17), U21.55 (GPIOB_RXP00); no longer J23.15 (Pin_15), U21.54 (GPIOB_TXN11)
- net I2C1_SCL: now also U21.15 (GPIOL_24_CLK0), J16.6 (Pin_6); no longer U21.14 (GPIOL_25_CLK1)
- net I2C1_SDA: now also U21.16 (GPIOL_22_CTRL2), J16.4 (Pin_4); no longer U21.15 (GPIOL_24_CLK0)
- net L64: now also J21.26 (Pin_26); no longer J21.25 (Pin_25)
- net L65: now also J21.24 (Pin_24); no longer J21.23 (Pin_23)
- net L66: now also J21.23 (Pin_23); no longer J21.26 (Pin_26)
- net L67: now also J21.21 (Pin_21); no longer J21.24 (Pin_24)
- net N02: now also J23.8 (Pin_8); no longer J23.10 (Pin_10)
- net NSTATUS: now also J21.17 (Pin_17); no longer J21.20 (Pin_20)
- net P02: now also J23.7 (Pin_7); no longer J23.8 (Pin_8)
- net R76: now also J21.12 (Pin_12); no longer J21.11 (Pin_11)
- net RDY: now also J23.21 (Pin_21), U21.60 (GPIOB_RXN03); no longer J23.19 (Pin_19), U21.59 (GPIOB_RXN02)
- net S1: now also J21.15 (Pin_15); no longer J21.18 (Pin_18)
- net S2: now also J21.18 (Pin_18); no longer J21.17 (Pin_17)
- net S3: now also J21.20 (Pin_20); no longer J21.19 (Pin_19)
- net S4: now also J21.19 (Pin_19); no longer J21.22 (Pin_22)
- net SPI0_RX: now also J16.9 (Pin_9), R70.1; no longer U21.28 (GPIOL_09_CDI1)
- net SPI0_SCK: now also J16.5 (Pin_5)
- net SPI0_TX: now also J16.7 (Pin_7)
- net SPI0_~{CS}: now also J16.3 (Pin_3)
- net SPI1_RX: now also J16.22 (Pin_22), R68.1; no longer U21.8 (GPIOL_40_CDI8)
- net SPI1_SCK: now also J16.18 (Pin_18)
- net SPI1_TX: now also U21.8 (GPIOL_40_CDI8), J16.20 (Pin_20); no longer U21.7 (GPIOL_41_CDI9)
- net SPI1_~{CS}: now also J16.16 (Pin_16)
- net SPI1_~{READY}: now also J16.14 (Pin_14), R71.1; no longer U21.18 (GPIOL_20_CTRL0_CDI4)
- net VIA_CB2: now also J23.16 (Pin_16), U21.54 (GPIOB_TXN11); no longer J23.14 (Pin_14), U21.53 (GPIOB_TXP11)
- net ~{IO_OE}: now also U21.119 (GPIOR_78_EXTFB0_CDI31); no longer U21.123 (GPIOR_77_PLLIN1)
- net ~{IRQ}: now also J23.23 (Pin_23), U21.65 (GPIOB_RXN07); no longer J23.22 (Pin_22), U21.61 (GPIOB_RXP03)
- net ~{ML}: now also J23.24 (Pin_24), U21.66 (GPIOB_RXP07); no longer J23.23 (Pin_23), U21.65 (GPIOB_RXN07)
- net ~{NMI}: now also J21.22 (Pin_22), U21.139 (GPIOL_68); no longer J23.25 (Pin_25), U21.67 (GPIOB_RXP10)
- net ~{PIA2_CS}: now also U21.123 (GPIOR_77_PLLIN1); no longer U21.119 (GPIOR_78_EXTFB0_CDI31)
- net ~{RAM_OE}: now also J23.18 (Pin_18), U21.56 (GPIOB_RXN00); no longer J23.16 (Pin_16), U21.55 (GPIOB_RXP00)
- net ~{RAM_WE}: now also J23.19 (Pin_19), U21.58 (GPIOB_RXP02); no longer J23.17 (Pin_17), U21.56 (GPIOB_RXN00)
- net ~{RES}: now also J23.27 (Pin_27); no longer J23.20 (Pin_20)
- net ~{SO}: now also J23.22 (Pin_22), U21.61 (GPIOB_RXP03); no longer J23.21 (Pin_21), U21.60 (GPIOB_RXN03)
- net ~{VP}: now also J23.20 (Pin_20), U21.59 (GPIOB_RXN02); no longer J23.18 (Pin_18), U21.58 (GPIOB_RXP02)
- net P06: now reaches J23.11 (Pin_11)
- net P06: now also U21.45 (GPIOB_TXP06)
- net N06: now reaches J23.12 (Pin_12)
- net N06: now also U21.46 (GPIOB_TXN06)
- net P04: now reaches J23.9 (Pin_9)
- net P04: now also U21.42 (GPIOB_TXP04)
- net N04: now reaches U21.43 (GPIOB_TXN04)
- net N04: now also J23.10 (Pin_10)
- net P09: now reaches U21.47 (GPIOB_TXP09)
- net P09: now also J23.13 (Pin_13)
- net L75: now reaches U21.131 (GPIOL_75_PLLIN1)
- net L75: now also J21.11 (Pin_11)
- net YY4: now reaches U21.17 (GPIOL_21_CTRL1_CDI5)
- net YY4: now also J16.13 (Pin_13)
- net YY2: now reaches U21.19 (GPIOL_13_CDI3)
- net YY2: now also J16.11 (Pin_11)
- net YY1: now reaches U21.20 (GPIOL_12_CDI2)
- net YY1: now also J16.10 (Pin_10)
- net L53: now reaches U21.3 (GPIOL_53_CDI10)
- net L53: now also J21.25 (Pin_25)
- net YY5: now reaches U21.6 (GPIOL_46)
- net YY5: now also J16.15 (Pin_15)
- removed net L68: J21.21 (Pin_21), U21.139 (GPIOL_68)
- new net +1V1: J16.2 (Pin_2)
- new net FPGA_SPI0_TX: R70.2, U21.28 (GPIOL_09_CDI1)
- new net FPGA_SPI1_TX: R68.2, U21.7 (GPIOL_41_CDI9)
- new net FPGA_SPI1_~{READY}: R71.2, U21.14 (GPIOL_25_CLK1)
- new net I2C0_SCL: J16.19 (Pin_19)
- new net I2C0_SDA: J16.17 (Pin_17)
- new net N09: J23.14 (Pin_14), U21.48 (GPIOB_TXN09)
- new net YY3: J16.12 (Pin_12), U21.18 (GPIOL_20_CTRL0_CDI4)
- new net YY6: J16.8 (Pin_8), U21.33 (GPIOL_05_CSO)
- no-connect marks 14 -> 0
Other:
- note added: "Do not connect I2C0 to FPGA as it can be pulled up to +5V. (See MCU/DVI)"
- moved on the sheet: R33
