File: hw/Mainboard/MicroSD.kicad_sch (KiCad schematic)
At the start: 5 parts, among them J13 MicroSD

Commit message: wip: support 8x16 keyboard matrix
Parts:
- added R69: 33, Resistor_SMD:R_0402_1005Metric, symbol Device:R_Small
Connections:
- net DAT0: now also R69.2; no longer J13.7 (DAT0)
- net GND: no longer J13.14 (SHIELD)
- new net: J13.7 (DAT0), R69.1
Other:
- note added: "DAT[0] : (POCI) is open-drain output that requires pullup. DAT[2:1] : Unused inputs in SPI mode. Pullups recommended to avoid current draw due to metastablitiy. DAT[3] : (~{CS}) has built-in 22-50k pullup to ensure card is deselected by default. CMD : (PICO) input in SPI mode. CLK : (SCK) always an input. Never gets pullup. CM1624 uses: 25k pullup for DAT[0:3] and CMD 40 Ohm termination for DAT[0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"
- note removed: "DAT0 (RX) is open collector and requires pullup. DAT[3:1] are inputs on powerup and get weak pullups to avoid excessive current draw due to metastablitiy. CMD gets pullup in some designs. Usused DAT[2:1] could possible share a pullup? CLK should not get pull up. CM1624: 25k pullup for DAT[0:3] and CMD 40 Ohm termination for DAT[0:3], CMD, and CLK"
Changed lines of the file:
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@@
+    (stroke (width 0) (type default) (color 0 0 0 0))
+  )
+  (wire (pts (xy 149.86 96.52) (xy 147.32 96.52))
+    (stroke (width 0) (type default) (color 0 0 0 0))
+  )
+  (wire (pts (xy 120.65 106.68) (xy 149.86 106.68))
+    (stroke (width 0) (type default) (color 0 0 0 0))
+  )
+  (wire (pts (xy 120.65 74.93) (xy 130.81 74.93))
+    (stroke (width 0) (type default) (color 0 0 0 0))
+  )
+  (wire (pts (xy 133.35 74.93) (xy 135.89 74.93))
+    (stroke (width 0) (type default) (color 0 0 0 0))
+  )
+  (wire (pts (xy 130.81 74.93) (xy 133.35 74.93))
+    (stroke (width 0) (type default) (color 0 0 0 0))
+  )
+  (wire (pts (xy 154.94 73.66) (xy 154.94 72.39))
+    (stroke (width 0) (type default) (color 0 0 0 0))
+  )
+  (wire (pts (xy 149.86 88.9) (xy 138.43 88.9))
+    (stroke (width 0) (type default) (color 0 0 0 0))
+  )
+  (wire (pts (xy 130.81 76.2) (xy 130.81 74.93))
+    (stroke (width 0) (type default) (color 0 0 0 0))
+  )
+  (wire (pts (xy 154.94 67.31) (xy 154.94 66.04))
+    (stroke (width 0) (type default) (color 0 0 0 0))
+  )
+  (wire (pts (xy 154.94 74.93) (xy 154.94 73.66))
+    (stroke (width 0) (type default) (color 0 0 0 0))
+  )
+  (wire (pts (xy 147.32 101.6) (xy 147.32 118.11))
+    (stroke (width 0) (type default) (color 0 0 0 0))
+  )
+  (wire (pts (xy 102.87 91.44) (xy 135.89 91.44))
+    (stroke (width 0) (type default) (color 0 0 0 0))
+  )
+  (wire (pts (xy 142.24 104.14) (xy 149.86 104.14))
+    (stroke (width 0) (type default) (color 0 0 0 0))
+  )
+  (wire (pts (xy 147.32 64.77) (xy 147.32 66.04))
+    (stroke (width 0) (type default) (color 0 0 0 0))
+  )
+  (wire (pts (xy 165.1 66.04) (xy 165.1 67.31))
+    (stroke (width 0) (type default) (color 0 0 0 0))
+  )
+  (wire (pts (xy 120.65 78.74) (xy 120.65 74.93))
     (stroke (width 0) (type default) (color 0 0 0 0))
   )
@@
     (stroke (width 0) (type default) (color 0 0 0 0))
   )
-  (wire (pts (xy 149.86 96.52) (xy 147.32 96.52))
-    (stroke (width 0) (type default) (color 0 0 0 0))
-  )
-  (wire (pts (xy 120.65 106.68) (xy 149.86 106.68))
-    (stroke (width 0) (type default) (color 0 0 0 0))
-  )
-  (wire (pts (xy 120.65 74.93) (xy 130.81 74.93))
-    (stroke (width 0) (type default) (color 0 0 0 0))
-  )
-  (wire (pts (xy 133.35 74.93) (xy 135.89 74.93))
-    (stroke (width 0) (type default) (color 0 0 0 0))
-  )
-  (wire (pts (xy 130.81 74.93) (xy 133.35 74.93))
-    (stroke (width 0) (type default) (color 0 0 0 0))
-  )
-  (wire (pts (xy 154.94 73.66) (xy 154.94 72.39))
-    (stroke (width 0) (type default) (color 0 0 0 0))
-  )
-  (wire (pts (xy 149.86 88.9) (xy 138.43 88.9))
-    (stroke (width 0) (type default) (color 0 0 0 0))
-  )
-  (wire (pts (xy 130.81 76.2) (xy 130.81 74.93))
-    (stroke (width 0) (type default) (color 0 0 0 0))
-  )
-  (wire (pts (xy 154.94 67.31) (xy 154.94 66.04))
-    (stroke (width 0) (type default) (color 0 0 0 0))
-  )
-  (wire (pts (xy 154.94 74.93) (xy 154.94 73.66))
-    (stroke (width 0) (type default) (color 0 0 0 0))
-  )
-  (wire (pts (xy 147.32 101.6) (xy 147.32 118.11))
-    (stroke (width 0) (type default) (color 0 0 0 0))
-  )
-  (wire (pts (xy 102.87 91.44) (xy 135.89 91.44))
-    (stroke (width 0) (type default) (color 0 0 0 0))
-  )
-  (wire (pts (xy 147.32 64.77) (xy 147.32 66.04))
-    (stroke (width 0) (type default) (color 0 0 0 0))
-  )
-  (wire (pts (xy 165.1 66.04) (xy 165.1 67.31))
-    (stroke (width 0) (type default) (color 0 0 0 0))
-  )
-  (wire (pts (xy 130.81 104.14) (xy 149.86 104.14))
-    (stroke (width 0) (type default) (color 0 0 0 0))
-  )
-  (wire (pts (xy 120.65 78.74) (xy 120.65 74.93))
+  (wire (pts (xy 130.81 104.14) (xy 137.16 104.14))
     (stroke (width 0) (type default) (color 0 0 0 0))
   )
@@
     (stroke (width 0) (type default) (color 0 0 0 0))
   )
-  (text "DAT0 (RX) is open collector and requires pullup.\n\nDAT[3:1] are inputs on powerup and get weak pullups\nto avoid excessive current draw due to metastablitiy.\n\nCMD gets pullup in some designs.\nUsused DAT[2:1] could possible share a pullup?\nCLK should not get pull up.\n\nCM1624:\n25k pullup for DAT[0:3] and CMD\n40 Ohm termination for DAT[0:3], CMD, and CLK"
-    (at 157.48 149.86 0)
+  (text "DAT[0]   : (POCI) is open-drain output that requires pullup.\nDAT[2:1] : Unused inputs in SPI mode.  Pullups recommended\n           to avoid current draw due to metastablitiy.\nDAT[3]   : (~{CS}) has built-in 22-50k pullup to ensure card\n           is deselected by default.\nCMD      : (PICO) input in SPI mode.\nCLK      : (SCK) always an input.  Never gets pullup.\n\nCM1624 uses:\n25k pullup for DAT[0:3] and CMD\n40 Ohm termination for DAT[0:3], CMD, and CLK\n\n10k pullups common (e.g., ExpressIf documentation)."
+    (at 153.67 149.86 0)
     (effects (font (size 1.27 1.27)) (justify left bottom))
   )
@@
     (pin "12")
     (pin "13")
-    (pin "14")
     (pin "1")
     (pin "10")
@@
     (pin "1")
   )
+  (symbol (lib_id "Device:R_Small") (at 139.7 104.14 270) (unit 1)
+    (in_bom yes) (on_board yes)
+    (property "Reference" "R69" (id 0) (at 133.35 102.87 90)
+      (effects (font (size 1.27 1.27)) (justify left))
+    )
+    (property "Value" "33" (id 1) (at 138.43 104.14 90)
+      (effects (font (size 1.27 1.27)) (justify left))
+    )
+    (property "Footprint" "Resistor_SMD:R_0402_1005Metric" (id 2) (at 139.7 104.14 0)
+      (effects (font (size 1.27 1.27)) hide)
+    )
+    (property "Datasheet" "" (id 3) (at 139.7 104.14 0)
+      (effects (font (size 1.27 1.27)) hide)
+    )
+    (property "LCSC" "C25105" (id 4) (at 139.7 104.14 0)
+      (effects (font (size 1.27 1.27)) hide)
+    )
+    (pin "1")
+    (pin "2")
+  )
   (symbol (lib_id "Device:C_Small") (at 154.94 69.85 0) (unit 1)

Commit message: hw: update 10u caps
Other:
- title: (none) -> CBM PET Mainboard Replacement
Changed lines of the file:
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@@
 (kicad_sch (version 20211123) (generator eeschema)
-  (paper "A4")
+  (paper "A")
+  (title_block
+    (title "CBM PET Mainboard Replacement")
+  )
   (junction (at 130.81 74.93) (diameter 0) (color 0 0 0 0)
   )
