File: hw/Mainboard/MicroSD.kicad_sch (KiCad schematic)
At the start: 6 parts, among them J13 MicroSD

Commit message: hw: wip
Parts:
- C49: LCSC C1525 -> C307331
Changed lines of the file:
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@@
       (effects (font (size 1.27 1.27)) hide)
     )
-    (property "Datasheet" "https://datasheet.lcsc.com/lcsc/1810191219_Samsung-Electro-Mechanics-CL05B104KO5NNNC_C1525.pdf" (id 3) (at 154.94 69.85 0)
+    (property "Datasheet" "" (id 3) (at 154.94 69.85 0)
       (effects (font (size 1.27 1.27)) hide)
     )
-    (property "LCSC" "C1525" (id 4) (at 154.94 69.85 0)
+    (property "LCSC" "C307331" (id 4) (at 154.94 69.85 0)
       (effects (font (size 1.27 1.27)) hide)
     )

Commit message: wip
Connections:
- net DAT0: no longer RN16.4 (R4.1)
- net at J13.7 (DAT0), R69.1: now also RN16.4 (R4.1)
Other:
- moved on the sheet: R69
Changed lines of the file:
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@@
     (title "CBM PET Mainboard Replacement")
   )
+  (junction (at 130.81 104.14) (diameter 0) (color 0 0 0 0)
+  )
   (junction (at 130.81 74.93) (diameter 0) (color 0 0 0 0)
   )
   (junction (at 154.94 73.66) (diameter 0) (color 0 0 0 0)
   )
-  (junction (at 130.81 104.14) (diameter 0) (color 0 0 0 0)
-  )
   (junction (at 154.94 66.04) (diameter 0) (color 0 0 0 0)
   )
@@
     (stroke (width 0) (type default) (color 0 0 0 0))
   )
+  (wire (pts (xy 102.87 104.14) (xy 123.19 104.14))
+    (stroke (width 0) (type default) (color 0 0 0 0))
+  )
   (wire (pts (xy 149.86 88.9) (xy 138.43 88.9))
     (stroke (width 0) (type default) (color 0 0 0 0))
@@
     (stroke (width 0) (type default) (color 0 0 0 0))
   )
-  (wire (pts (xy 142.24 104.14) (xy 149.86 104.14))
-    (stroke (width 0) (type default) (color 0 0 0 0))
-  )
   (wire (pts (xy 147.32 64.77) (xy 147.32 66.04))
     (stroke (width 0) (type default) (color 0 0 0 0))
@@
     (stroke (width 0) (type default) (color 0 0 0 0))
   )
-  (wire (pts (xy 102.87 104.14) (xy 130.81 104.14))
-    (stroke (width 0) (type default) (color 0 0 0 0))
-  )
-  (wire (pts (xy 130.81 104.14) (xy 137.16 104.14))
+  (wire (pts (xy 130.81 104.14) (xy 149.86 104.14))
     (stroke (width 0) (type default) (color 0 0 0 0))
   )
@@
   )
   (wire (pts (xy 133.35 93.98) (xy 149.86 93.98))
+    (stroke (width 0) (type default) (color 0 0 0 0))
+  )
+  (wire (pts (xy 128.27 104.14) (xy 130.81 104.14))
     (stroke (width 0) (type default) (color 0 0 0 0))
   )
@@
     (pin "1")
   )
-  (symbol (lib_id "Device:R_Small") (at 139.7 104.14 270) (unit 1)
-    (in_bom yes) (on_board yes)
-    (property "Reference" "R69" (id 0) (at 133.35 102.87 90)
-      (effects (font (size 1.27 1.27)) (justify left))
-    )
-    (property "Value" "33" (id 1) (at 138.43 104.14 90)
-      (effects (font (size 1.27 1.27)) (justify left))
-    )
-    (property "Footprint" "Resistor_SMD:R_0402_1005Metric" (id 2) (at 139.7 104.14 0)
-      (effects (font (size 1.27 1.27)) hide)
-    )
-    (property "Datasheet" "" (id 3) (at 139.7 104.14 0)
-      (effects (font (size 1.27 1.27)) hide)
-    )
-    (property "LCSC" "C25105" (id 4) (at 139.7 104.14 0)
-      (effects (font (size 1.27 1.27)) hide)
-    )
+  (symbol (lib_id "Device:R_Small") (at 125.73 104.14 270) (unit 1)
+    (in_bom yes) (on_board yes)
+    (property "Reference" "R69" (id 0) (at 123.825 101.6 90)
+      (effects (font (size 1.27 1.27)) (justify left))
+    )
+    (property "Value" "33" (id 1) (at 124.46 104.14 90)
+      (effects (font (size 1.27 1.27)) (justify left))
+    )
+    (property "Footprint" "Resistor_SMD:R_0402_1005Metric" (id 2) (at 125.73 104.14 0)
+      (effects (font (size 1.27 1.27)) hide)
+    )
+    (property "Datasheet" "" (id 3) (at 125.73 104.14 0)
+      (effects (font (size 1.27 1.27)) hide)
+    )
+    (property "LCSC" "C25105" (id 4) (at 125.73 104.14 0)
+      (effects (font (size 1.27 1.27)) hide)
+    )

Commit message: hw: 9V DC plug on left edge, change default track size
Parts:
- renumbered C49 to C82, C50 to C83, J13 to J24, R20 to R68
Changed lines of the file:
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@@
   (symbol (lib_id "power:+3V3") (at 138.43 74.93 0) (mirror y) (unit 1)
     (in_bom yes) (on_board yes)
-    (property "Reference" "#PWR0148" (id 0) (at 138.43 78.74 0)
+    (property "Reference" "#PWR0145" (id 0) (at 138.43 78.74 0)
       (effects (font (size 1.27 1.27)) hide)
     )
@@
   (symbol (lib_id "power:+3V3") (at 147.32 64.77 0) (unit 1)
     (in_bom yes) (on_board yes)
-    (property "Reference" "#PWR0147" (id 0) (at 147.32 68.58 0)
+    (property "Reference" "#PWR0144" (id 0) (at 147.32 68.58 0)
       (effects (font (size 1.27 1.27)) hide)
     )
@@
   (symbol (lib_id "Connector:Micro_SD_Card_Det") (at 172.72 99.06 0) (unit 1)
     (in_bom yes) (on_board yes) (fields_autoplaced)
-    (property "Reference" "J13" (id 0) (at 173.355 77.47 0))
+    (property "Reference" "J24" (id 0) (at 173.355 77.47 0))
     (property "Value" "MicroSD" (id 1) (at 173.355 80.01 0))
     (property "Footprint" "JLCPCB:TF-SMD_TF-PUSH" (id 2) (at 224.79 81.28 0)
@@
   (symbol (lib_id "power:GND") (at 194.31 113.03 0) (unit 1)
     (in_bom yes) (on_board yes) (fields_autoplaced)
-    (property "Reference" "#PWR0150" (id 0) (at 194.31 119.38 0)
+    (property "Reference" "#PWR0147" (id 0) (at 194.31 119.38 0)
       (effects (font (size 1.27 1.27)) hide)
     )
@@
   (symbol (lib_id "power:GND") (at 147.32 118.11 0) (unit 1)
     (in_bom yes) (on_board yes) (fields_autoplaced)
-    (property "Reference" "#PWR0149" (id 0) (at 147.32 124.46 0)
+    (property "Reference" "#PWR0148" (id 0) (at 147.32 124.46 0)
       (effects (font (size 1.27 1.27)) hide)
     )
@@
   (symbol (lib_id "Device:C_Small") (at 165.1 69.85 0) (unit 1)
     (in_bom yes) (on_board yes)
-    (property "Reference" "C50" (id 0) (at 167.4368 68.6816 0)
+    (property "Reference" "C83" (id 0) (at 167.4368 68.6816 0)
       (effects (font (size 1.27 1.27)) (justify left))
     )
@@
   (symbol (lib_id "Device:R_Small") (at 120.65 81.28 0) (unit 1)
     (in_bom yes) (on_board yes)
-    (property "Reference" "R20" (id 0) (at 118.745 83.185 90)
+    (property "Reference" "R68" (id 0) (at 118.745 83.185 90)
       (effects (font (size 1.27 1.27)) (justify left))
     )
@@
   (symbol (lib_id "power:GND") (at 154.94 74.93 0) (unit 1)
     (in_bom yes) (on_board yes) (fields_autoplaced)
-    (property "Reference" "#PWR0151" (id 0) (at 154.94 81.28 0)
+    (property "Reference" "#PWR0146" (id 0) (at 154.94 81.28 0)
       (effects (font (size 1.27 1.27)) hide)
     )
@@
   (symbol (lib_id "Device:C_Small") (at 154.94 69.85 0) (unit 1)
     (in_bom yes) (on_board yes)
-    (property "Reference" "C49" (id 0) (at 157.2768 68.6816 0)
+    (property "Reference" "C82" (id 0) (at 157.2768 68.6816 0)
       (effects (font (size 1.27 1.27)) (justify left))
     )

Commit message: hw: 25x2 header (wip)
Parts:
- renumbered J24 to J25
Changed lines of the file:
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@@
   (symbol (lib_id "power:+3V3") (at 138.43 74.93 0) (mirror y) (unit 1)
     (in_bom yes) (on_board yes)
-    (property "Reference" "#PWR0145" (id 0) (at 138.43 78.74 0)
+    (property "Reference" "#PWR0147" (id 0) (at 138.43 78.74 0)
       (effects (font (size 1.27 1.27)) hide)
     )
@@
   (symbol (lib_id "power:+3V3") (at 147.32 64.77 0) (unit 1)
     (in_bom yes) (on_board yes)
-    (property "Reference" "#PWR0144" (id 0) (at 147.32 68.58 0)
+    (property "Reference" "#PWR0146" (id 0) (at 147.32 68.58 0)
       (effects (font (size 1.27 1.27)) hide)
     )
@@
   (symbol (lib_id "Connector:Micro_SD_Card_Det") (at 172.72 99.06 0) (unit 1)
     (in_bom yes) (on_board yes) (fields_autoplaced)
-    (property "Reference" "J24" (id 0) (at 173.355 77.47 0))
+    (property "Reference" "J25" (id 0) (at 173.355 77.47 0))
     (property "Value" "MicroSD" (id 1) (at 173.355 80.01 0))
     (property "Footprint" "JLCPCB:TF-SMD_TF-PUSH" (id 2) (at 224.79 81.28 0)
@@
   (symbol (lib_id "power:GND") (at 194.31 113.03 0) (unit 1)
     (in_bom yes) (on_board yes) (fields_autoplaced)
-    (property "Reference" "#PWR0147" (id 0) (at 194.31 119.38 0)
+    (property "Reference" "#PWR0149" (id 0) (at 194.31 119.38 0)
       (effects (font (size 1.27 1.27)) hide)
     )
@@
   (symbol (lib_id "power:GND") (at 147.32 118.11 0) (unit 1)
     (in_bom yes) (on_board yes) (fields_autoplaced)
-    (property "Reference" "#PWR0148" (id 0) (at 147.32 124.46 0)
+    (property "Reference" "#PWR0150" (id 0) (at 147.32 124.46 0)
       (effects (font (size 1.27 1.27)) hide)
     )
@@
   (symbol (lib_id "power:GND") (at 154.94 74.93 0) (unit 1)
     (in_bom yes) (on_board yes) (fields_autoplaced)
-    (property "Reference" "#PWR0146" (id 0) (at 154.94 81.28 0)
+    (property "Reference" "#PWR0148" (id 0) (at 154.94 81.28 0)
       (effects (font (size 1.27 1.27)) hide)
     )

Commit message: hw: 2x config switch (wip)
Parts:
- renumbered J25 to J24
Changed lines of the file:
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@@
   (symbol (lib_id "power:+3V3") (at 138.43 74.93 0) (mirror y) (unit 1)
     (in_bom yes) (on_board yes)
-    (property "Reference" "#PWR0147" (id 0) (at 138.43 78.74 0)
+    (property "Reference" "#PWR0153" (id 0) (at 138.43 78.74 0)
       (effects (font (size 1.27 1.27)) hide)
     )
@@
   (symbol (lib_id "power:+3V3") (at 147.32 64.77 0) (unit 1)
     (in_bom yes) (on_board yes)
-    (property "Reference" "#PWR0146" (id 0) (at 147.32 68.58 0)
+    (property "Reference" "#PWR0152" (id 0) (at 147.32 68.58 0)
       (effects (font (size 1.27 1.27)) hide)
     )
@@
   (symbol (lib_id "Connector:Micro_SD_Card_Det") (at 172.72 99.06 0) (unit 1)
     (in_bom yes) (on_board yes) (fields_autoplaced)
-    (property "Reference" "J25" (id 0) (at 173.355 77.47 0))
+    (property "Reference" "J24" (id 0) (at 173.355 77.47 0))
     (property "Value" "MicroSD" (id 1) (at 173.355 80.01 0))
     (property "Footprint" "JLCPCB:TF-SMD_TF-PUSH" (id 2) (at 224.79 81.28 0)
@@
   (symbol (lib_id "power:GND") (at 194.31 113.03 0) (unit 1)
     (in_bom yes) (on_board yes) (fields_autoplaced)
-    (property "Reference" "#PWR0149" (id 0) (at 194.31 119.38 0)
+    (property "Reference" "#PWR0155" (id 0) (at 194.31 119.38 0)
       (effects (font (size 1.27 1.27)) hide)
     )
@@
   (symbol (lib_id "power:GND") (at 147.32 118.11 0) (unit 1)
     (in_bom yes) (on_board yes) (fields_autoplaced)
-    (property "Reference" "#PWR0150" (id 0) (at 147.32 124.46 0)
+    (property "Reference" "#PWR0156" (id 0) (at 147.32 124.46 0)
       (effects (font (size 1.27 1.27)) hide)
     )
@@
   (symbol (lib_id "power:GND") (at 154.94 74.93 0) (unit 1)
     (in_bom yes) (on_board yes) (fields_autoplaced)
-    (property "Reference" "#PWR0148" (id 0) (at 154.94 81.28 0)
+    (property "Reference" "#PWR0154" (id 0) (at 154.94 81.28 0)
       (effects (font (size 1.27 1.27)) hide)
     )
