File: hw/Mainboard/DVI.kicad_sch (KiCad schematic)
At the start: 16 parts, among them J12 NOT_HDMI_A

Commit message: hw: wip
Parts:
- added PT18: PowerTie_2, PET:NetTie-2_SMD_Pad_1.6_to_0.4mm, symbol PET:PowerTie_2
Connections:
- net +5V: now also PT18.1; no longer J12.18 (+5V), R8.1, R9.1
- new net: J12.18 (+5V), PT18.2, R8.1, R9.1
Other:
- moved on the sheet: J12, JP7, JP8, JP9, R1, R10, R11, R16, R2, R3, R4, R5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

Commit message: hw: update 10u caps
Other:
- title: (none) -> CBM PET Mainboard Replacement
Changed lines of the file:
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@@
 (kicad_sch (version 20211123) (generator eeschema)
-  (paper "A4")
+  (paper "A")
+  (title_block
+    (title "CBM PET Mainboard Replacement")
+  )
   (bus_alias "DVI" (members "DVI_D2+" "DVI_D2-" "DVI_D1+" "DVI_D1-" "DVI_D0+" "DVI_D0-" "DVI_CK+" "DVI_CK-"))
   (junction (at 134.62 111.76) (diameter 0) (color 0 0 0 0)

Commit message: wip
Parts:
- added PT37: PowerTie_2, PET:NetTie-2_SMD_Pad_1.6_to_0.4mm, symbol PET:PowerTie_2
Connections:
- net VCC: now reaches J12.18 (+5V), PT18.2, R8.1, R9.1
- net GND renamed VSS
- net VSS: now also PT37.2; no longer J12.SH
- new net PD_GND: J12.SH, PT37.1
Changed lines of the file:
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@@
   (junction (at 134.62 111.76) (diameter 0) (color 0 0 0 0)
   )
-  (junction (at 198.12 118.11) (diameter 0) (color 0 0 0 0)
-  )
   (junction (at 193.04 118.11) (diameter 0) (color 0 0 0 0)
   )
   (junction (at 190.5 59.69) (diameter 0) (color 0 0 0 0)
   )
-  (junction (at 195.58 118.11) (diameter 0) (color 0 0 0 0)
-  )
   (junction (at 134.62 59.69) (diameter 0) (color 0 0 0 0)
+  )
+  (junction (at 198.12 120.65) (diameter 0) (color 0 0 0 0)
   )
   (junction (at 190.5 118.11) (diameter 0) (color 0 0 0 0)
@@
     (stroke (width 0) (type default) (color 0 0 0 0))
   )
+  (wire (pts (xy 190.5 118.11) (xy 190.5 120.65))
+    (stroke (width 0) (type default) (color 0 0 0 0))
+  )
   (wire (pts (xy 111.76 101.6) (xy 129.54 101.6))
     (stroke (width 0) (type default) (color 0 0 0 0))
@@
     (stroke (width 0) (type default) (color 0 0 0 0))
   )
-  (wire (pts (xy 198.12 118.11) (xy 198.12 119.38))
+  (wire (pts (xy 198.12 116.84) (xy 198.12 120.65))
     (stroke (width 0) (type default) (color 0 0 0 0))
   )
@@
     (stroke (width 0) (type default) (color 0 0 0 0))
   )
+  (wire (pts (xy 190.5 120.65) (xy 193.04 120.65))
+    (stroke (width 0) (type default) (color 0 0 0 0))
+  )
   (wire (pts (xy 187.96 118.11) (xy 190.5 118.11))
     (stroke (width 0) (type default) (color 0 0 0 0))
@@
     (stroke (width 0) (type default) (color 0 0 0 0))
   )
-  (wire (pts (xy 195.58 118.11) (xy 198.12 118.11))
-    (stroke (width 0) (type default) (color 0 0 0 0))
-  )
   (wire (pts (xy 97.79 91.44) (xy 104.14 91.44))
     (stroke (width 0) (type default) (color 0 0 0 0))
@@
     (stroke (width 0) (type default) (color 0 0 0 0))
   )
+  (wire (pts (xy 198.12 120.65) (xy 198.12 121.92))
+    (stroke (width 0) (type default) (color 0 0 0 0))
+  )
   (wire (pts (xy 193.04 118.11) (xy 195.58 118.11))
     (stroke (width 0) (type default) (color 0 0 0 0))
@@
   )
   (wire (pts (xy 167.64 91.44) (xy 180.34 91.44))
-    (stroke (width 0) (type default) (color 0 0 0 0))
-  )
-  (wire (pts (xy 198.12 116.84) (xy 198.12 118.11))
     (stroke (width 0) (type default) (color 0 0 0 0))
   )
@@
     (effects (font (size 1.27 1.27)) (justify right bottom))
   )
+  (label "VSS" (at 190.5 120.65 0)
+    (effects (font (size 1.27 1.27)) (justify left bottom))
+  )
   (label "HDMI_CK+" (at 180.34 83.82 180)
     (effects (font (size 1.27 1.27)) (justify right bottom))
@@
   )
   (label "HDMI_D1-" (at 180.34 76.2 180)
+    (effects (font (size 1.27 1.27)) (justify right bottom))
+  )
+  (label "VCC" (at 189.23 59.69 180)
     (effects (font (size 1.27 1.27)) (justify right bottom))
   )
@@
     )
     (property "LCSC" "C25879" (id 4) (at 134.62 83.82 0)
+      (effects (font (size 1.27 1.27)) hide)
+    )
+    (pin "1")
+    (pin "2")
+  )
+  (symbol (lib_id "PET:PowerTie_2") (at 195.58 120.65 180) (unit 1)
+    (in_bom yes) (on_board yes) (fields_autoplaced)
+    (property "Reference" "PT37" (id 0) (at 195.58 122.555 0)
+      (effects (font (size 1.27 1.27)) hide)
+    )
+    (property "Value" "PowerTie_2" (id 1) (at 195.58 118.745 0)
+      (effects (font (size 1.27 1.27)) hide)
+    )
+    (property "Footprint" "PET:NetTie-2_SMD_Pad_1.6_to_0.4mm" (id 2) (at 195.58 120.65 0)
+      (effects (font (size 1.27 1.27)) hide)
+    )
+    (property "Datasheet" "" (id 3) (at 195.58 120.65 0)
       (effects (font (size 1.27 1.27)) hide)
     )
@@
     (pin "2")
   )
-  (symbol (lib_id "power:GND") (at 198.12 119.38 0) (unit 1)
-    (in_bom yes) (on_board yes)
-    (property "Reference" "#PWR0146" (id 0) (at 198.12 125.73 0)
-      (effects (font (size 1.27 1.27)) hide)
-    )
-    (property "Value" "GND" (id 1) (at 198.2343 123.7044 0))
-    (property "Footprint" "" (id 2) (at 198.12 119.38 0))
-    (property "Datasheet" "" (id 3) (at 198.12 119.38 0))
-    (pin "1")
-  )
   (symbol (lib_id "Device:R_Small") (at 165.1 78.74 90) (unit 1)
     (in_bom yes) (on_board yes)
@@
     (pin "2")
   )
+  (symbol (lib_id "PET:PD_GND") (at 198.12 121.92 0) (unit 1)
+    (in_bom yes) (on_board yes) (fields_autoplaced)
+    (property "Reference" "#PWR0146" (id 0) (at 198.12 128.27 0)
+      (effects (font (size 1.27 1.27)) hide)
+    )
+    (property "Value" "PD_GND" (id 1) (at 198.12 127 0))
+    (property "Footprint" "" (id 2) (at 198.12 121.92 0)
+      (effects (font (size 1.27 1.27)) hide)
+    )
+    (property "Datasheet" "" (id 3) (at 198.12 121.92 0)
+      (effects (font (size 1.27 1.27)) hide)
+    )
+    (pin "1")
+  )
   (symbol (lib_id "Device:R_Small") (at 165.1 71.12 90) (unit 1)
