File: hw/Mainboard/MAGIC.kicad_sch (KiCad schematic)
At the start: 17 parts, among them U18 SN74LVC4245APWR, U19 SN74LVC4245APWR, U20 SN74LVC4245APWR

Commit message: hw: wip
Parts:
- C18, C19, C20, C23, C27, C28: LCSC C1525 -> C307331
Changed lines of the file:
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@@
       (effects (font (size 1.27 1.27)) hide)
     )
-    (property "Datasheet" "https://datasheet.lcsc.com/lcsc/1810191219_Samsung-Electro-Mechanics-CL05B104KO5NNNC_C1525.pdf" (id 3) (at 207.01 22.86 0)
+    (property "Datasheet" "" (id 3) (at 207.01 22.86 0)
       (effects (font (size 1.27 1.27)) hide)
     )
-    (property "LCSC" "C1525" (id 4) (at 207.01 22.86 0)
+    (property "LCSC" "C307331" (id 4) (at 207.01 22.86 0)
       (effects (font (size 1.27 1.27)) hide)
     )
@@
       (effects (font (size 1.27 1.27)) hide)
     )
-    (property "Datasheet" "https://datasheet.lcsc.com/lcsc/1810191219_Samsung-Electro-Mechanics-CL05B104KO5NNNC_C1525.pdf" (id 3) (at 207.01 125.73 0)
+    (property "Datasheet" "" (id 3) (at 207.01 125.73 0)
       (effects (font (size 1.27 1.27)) hide)
     )
-    (property "LCSC" "C1525" (id 4) (at 207.01 125.73 0)
+    (property "LCSC" "C307331" (id 4) (at 207.01 125.73 0)
       (effects (font (size 1.27 1.27)) hide)
     )
@@
       (effects (font (size 1.27 1.27)) hide)
     )
-    (property "Datasheet" "https://datasheet.lcsc.com/lcsc/1810191219_Samsung-Electro-Mechanics-CL05B104KO5NNNC_C1525.pdf" (id 3) (at 236.22 22.86 0)
+    (property "Datasheet" "" (id 3) (at 236.22 22.86 0)
       (effects (font (size 1.27 1.27)) hide)
     )
-    (property "LCSC" "C1525" (id 4) (at 236.22 22.86 0)
+    (property "LCSC" "C307331" (id 4) (at 236.22 22.86 0)
       (effects (font (size 1.27 1.27)) hide)
     )
@@
       (effects (font (size 1.27 1.27)) hide)
     )
-    (property "Datasheet" "https://datasheet.lcsc.com/lcsc/1810191219_Samsung-Electro-Mechanics-CL05B104KO5NNNC_C1525.pdf" (id 3) (at 240.03 125.73 0)
+    (property "Datasheet" "" (id 3) (at 240.03 125.73 0)
       (effects (font (size 1.27 1.27)) hide)
     )
-    (property "LCSC" "C1525" (id 4) (at 240.03 125.73 0)
+    (property "LCSC" "C307331" (id 4) (at 240.03 125.73 0)
       (effects (font (size 1.27 1.27)) hide)
     )
@@
       (effects (font (size 1.27 1.27)) hide)
     )
-    (property "Datasheet" "https://datasheet.lcsc.com/lcsc/1810191219_Samsung-Electro-Mechanics-CL05B104KO5NNNC_C1525.pdf" (id 3) (at 236.22 73.66 0)
+    (property "Datasheet" "" (id 3) (at 236.22 73.66 0)
       (effects (font (size 1.27 1.27)) hide)
     )
-    (property "LCSC" "C1525" (id 4) (at 236.22 73.66 0)
+    (property "LCSC" "C307331" (id 4) (at 236.22 73.66 0)
       (effects (font (size 1.27 1.27)) hide)
     )
@@
       (effects (font (size 1.27 1.27)) hide)
     )
-    (property "Datasheet" "https://datasheet.lcsc.com/lcsc/1810191219_Samsung-Electro-Mechanics-CL05B104KO5NNNC_C1525.pdf" (id 3) (at 207.01 73.66 0)
+    (property "Datasheet" "" (id 3) (at 207.01 73.66 0)
       (effects (font (size 1.27 1.27)) hide)
     )
-    (property "LCSC" "C1525" (id 4) (at 207.01 73.66 0)
+    (property "LCSC" "C307331" (id 4) (at 207.01 73.66 0)
       (effects (font (size 1.27 1.27)) hide)
     )

Commit message: wip
Connections:
- net A3: now also U19.18 (B4); no longer U19.17 (B5)
- net BA3: now also U19.6 (A4); no longer U19.7 (A5)
- net B~{RES}: now also U19.7 (A5); no longer U19.6 (A4)
- net ~{RES}: now also U19.17 (B5); no longer U19.18 (B4)
- net Bϕ2 renamed BPHI2
- net ϕ2 renamed PHI2
Other:
- sheet FPGA ports: added PHI2; removed ϕ2
