File: hw/Mainboard/Mainboard.kicad_sch (KiCad schematic)
At the start: 0 parts

Commit message: wip
Other:
- sheet CPU \ RAM ports: added PHI2; removed ϕ2
- sheet IO ports: added BPHI2; removed Bϕ2
- sheet MAGIC ports: added BPHI2, PHI2; removed Bϕ2, ϕ2
Changed lines of the file:
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@@
       (effects (font (size 1.27 1.27)) (justify right))
     )
-    (pin "ϕ2" input (at 66.04 34.29 0)
+    (pin "PHI2" input (at 66.04 34.29 0)
       (effects (font (size 1.27 1.27)) (justify right))
     )
@@
       (effects (font (size 1.27 1.27)) (justify left))
     )
-    (pin "ϕ2" output (at 78.74 34.29 180)
+    (pin "PHI2" output (at 78.74 34.29 180)
       (effects (font (size 1.27 1.27)) (justify left))
     )
@@
       (effects (font (size 1.27 1.27)) (justify right))
     )
-    (pin "Bϕ2" output (at 104.14 34.29 0)
+    (pin "BPHI2" output (at 104.14 34.29 0)
       (effects (font (size 1.27 1.27)) (justify right))
     )
@@
       (effects (font (size 1.27 1.27)) (justify left))
     )
-    (pin "Bϕ2" input (at 116.84 34.29 180)
+    (pin "BPHI2" input (at 116.84 34.29 180)
       (effects (font (size 1.27 1.27)) (justify left))
     )
@@
       (reference "#PWR0120") (unit 1) (value "CHASSIS_GND") (footprint "")
     )
-    (path "/00000000-0000-0000-0000-000061b3f8ab/6e96bf9a-1a30-45a4-b544-533d518185ae"
-      (reference "#PWR0121") (unit 1) (value "PD_GND") (footprint "")
+    (path "/00000000-0000-0000-0000-000061b3f8ab/d50248b6-83ef-4da3-809d-d049b5613651"
+      (reference "#PWR0121") (unit 1) (value "+5V") (footprint "")
     )
     (path "/00000000-0000-0000-0000-000061bef9ce/bb660bb3-33ad-4033-ab93-6e9f17203d8c"
@@
       (reference "#PWR0187") (unit 1) (value "PD_GND") (footprint "")
     )
-    (path "/00000000-0000-0000-0000-000061b3f8ab/b9dc6cb0-9a01-48b4-8dc8-9af546e03724"
-      (reference "#PWR0188") (unit 1) (value "+5V") (footprint "")
-    )
     (path "/00000000-0000-0000-0000-000061bef9ce/72112a3f-57d1-478d-920d-031564fd3919"
       (reference "#PWR0189") (unit 1) (value "+5V") (footprint "")
@@
       (reference "#PWR0198") (unit 1) (value "+3V3") (footprint "")
     )
+    (path "/00000000-0000-0000-0000-0000617d6918/00000000-0000-0000-0000-000062edbe39/cd5f77c3-7436-4c27-9ecf-2ce63c5e5e19"
+      (reference "#PWR0199") (unit 1) (value "+1V2") (footprint "")
+    )
     (path "/00000000-0000-0000-0000-0000617d6918/b70241ab-8a5c-42d5-a1ab-8f4bc50a1197/cc6f1ce2-2835-4ca3-b032-2c76c20963f9"
       (reference "#PWR0200") (unit 1) (value "GND") (footprint "")
@@
       (reference "#PWR0204") (unit 1) (value "GND") (footprint "")
     )
+    (path "/00000000-0000-0000-0000-0000617d6918/00000000-0000-0000-0000-000062edbe39/62d1ff3c-42de-44b2-b130-b7f2c9c1001c"
+      (reference "#PWR0205") (unit 1) (value "+3V3") (footprint "")
+    )
     (path "/00000000-0000-0000-0000-0000614e685e/4169575a-365e-4e73-8a5b-3e025bc6ef61"
       (reference "#PWR0221") (unit 1) (value "GND") (footprint "")
@@
       (reference "C51") (unit 1) (value "100n") (footprint "Capacitor_SMD:C_0402_1005Metric")
     )
-    (path "/00000000-0000-0000-0000-0000617d6918/b70241ab-8a5c-42d5-a1ab-8f4bc50a1197/4bbfc88f-5e22-453e-ac3d-d10fbc3241d7"
-      (reference "C52") (unit 1) (value "10u") (footprint "Capacitor_SMD:C_0603_1608Metric")
+    (path "/00000000-0000-0000-0000-0000617d6918/b70241ab-8a5c-42d5-a1ab-8f4bc50a1197/de13ea05-947c-4492-a583-365a4a17d5bf"
+      (reference "C52") (unit 1) (value "2.2u 6.3V") (footprint "Capacitor_SMD:C_0402_1005Metric")
     )
     (path "/00000000-0000-0000-0000-0000617d6918/00000000-0000-0000-0000-000062edbe39/49410563-a4a5-43e3-8211-c6bc8d86586e"
@@
       (reference "JP9") (unit 1) (value "DVI_SDA") (footprint "Jumper:SolderJumper-2_P1.3mm_Open_RoundedPad1.0x1.5mm")
     )
+    (path "/00000000-0000-0000-0000-000061b3f8ab/9f5d630c-e8c2-4aa8-92b1-30205b28ed54"
+      (reference "JP10") (unit 1) (value "VIDEO_OR_5V") (footprint "Jumper:SolderJumper-3_P1.3mm_Open_RoundedPad1.0x1.5mm")
+    )
     (path "/5178399f-3ceb-4969-8efa-17e54018f3f1/5a88016c-3777-4d9c-b2cd-526d05ee5dce"
       (reference "LS1") (unit 1) (value "Speaker") (footprint "SamacSys_Parts:AT1220TT9R")
@@
     )
     (path "/00000000-0000-0000-0000-0000617d6918/00000000-0000-0000-0000-000062edbe39/c0149dcc-7328-4bf7-b520-fec6ae8b045d"
-      (reference "PT40") (unit 1) (value "PowerTie_2") (footprint "PET:NetTie-2_SMD_Pad_1.6_to_0.4mm")
+      (reference "PT40") (unit 1) (value "PowerTie_2") (footprint "PET:NetTie-2_SMD_Pad_0.28")
     )
     (path "/00000000-0000-0000-0000-0000617d6918/00000000-0000-0000-0000-000062edbe39/c0d916aa-6e62-440f-a4ea-a9a0d59a0e0c"
-      (reference "PT41") (unit 1) (value "PowerTie_2") (footprint "PET:NetTie-2_SMD_Pad_1.6_to_0.4mm")
+      (reference "PT41") (unit 1) (value "PowerTie_2") (footprint "PET:NetTie-2_SMD_Pad_0.28")
+    )
+    (path "/00000000-0000-0000-0000-0000617d6918/00000000-0000-0000-0000-000062edbe39/072ae20c-d6e3-4e5a-a8be-ca8fc98a33e0"
+      (reference "PT42") (unit 1) (value "PowerTie_2") (footprint "PET:NetTie-2_SMD_Pad_0.28")
+    )
+    (path "/00000000-0000-0000-0000-0000617d6918/00000000-0000-0000-0000-000062edbe39/f644d0c6-60c4-4dc5-8e66-4d8bca6db5b5"
+      (reference "PT43") (unit 1) (value "PowerTie_2") (footprint "PET:NetTie-2_SMD_Pad_0.28")
+    )
+    (path "/00000000-0000-0000-0000-0000617d6918/00000000-0000-0000-0000-000062edbe39/ecd1293c-e0b8-4710-abfb-8e3b49384eed"
+      (reference "PT44") (unit 1) (value "PowerTie_2") (footprint "PET:NetTie-2_SMD_Pad_0.28")
+    )
+    (path "/00000000-0000-0000-0000-0000617d6918/00000000-0000-0000-0000-000062edbe39/cbeb6a8c-5e02-499e-8659-bd2b817e6b75"
+      (reference "PT45") (unit 1) (value "PowerTie_2") (footprint "PET:NetTie-2_SMD_Pad_0.28")
+    )
+    (path "/00000000-0000-0000-0000-0000617d6918/00000000-0000-0000-0000-000062edbe39/3737fd9e-7433-4025-bf4d-e3ec0992daa1"
+      (reference "PT46") (unit 1) (value "PowerTie_2") (footprint "PET:NetTie-2_SMD_Pad_0.28")
+    )
+    (path "/00000000-0000-0000-0000-0000617d6918/00000000-0000-0000-0000-000062edbe39/77e3b5aa-5ae1-4149-a1bd-ebf52e6baa0a"
+      (reference "PT47") (unit 1) (value "PowerTie_2") (footprint "PET:NetTie-2_SMD_Pad_0.28")
+    )
+    (path "/00000000-0000-0000-0000-0000617d6918/00000000-0000-0000-0000-000062edbe39/56a8011c-5036-4fae-9142-33adce49520b"
+      (reference "PT48") (unit 1) (value "PowerTie_2") (footprint "PET:NetTie-2_SMD_Pad_0.28")
+    )
+    (path "/00000000-0000-0000-0000-0000617d6918/00000000-0000-0000-0000-000062edbe39/8d79f325-9827-4665-b6ea-377f47fd7b11"
+      (reference "PT49") (unit 1) (value "PowerTie_2") (footprint "PET:NetTie-2_SMD_Pad_0.28")
+    )
+    (path "/00000000-0000-0000-0000-0000617d6918/00000000-0000-0000-0000-000062edbe39/694af70e-4a56-4ba8-92b8-04ac6f9b1a04"
+      (reference "PT50") (unit 1) (value "PowerTie_2") (footprint "PET:NetTie-2_SMD_Pad_0.28")
+    )
+    (path "/00000000-0000-0000-0000-0000617d6918/00000000-0000-0000-0000-000062edbe39/1fe12ae2-3b0d-4ccb-890b-944a6ae68fdf"
+      (reference "PT51") (unit 1) (value "PowerTie_2") (footprint "PET:NetTie-2_SMD_Pad_0.28")
+    )
+    (path "/00000000-0000-0000-0000-0000617d6918/00000000-0000-0000-0000-000062edbe39/2e5a9dbb-685d-4682-a65e-21f208913358"
+      (reference "PT52") (unit 1) (value "PowerTie_2") (footprint "PET:NetTie-2_SMD_Pad_0.28")
+    )
+    (path "/00000000-0000-0000-0000-0000617d6918/00000000-0000-0000-0000-000062edbe39/1d9c7528-f905-4794-8ab8-35e92fb22d45"
+      (reference "PT53") (unit 1) (value "PowerTie_2") (footprint "PET:NetTie-2_SMD_Pad_0.28")
+    )
+    (path "/00000000-0000-0000-0000-0000617d6918/00000000-0000-0000-0000-000062edbe39/1e9d9dc0-3281-4706-a981-e2b737272d3b"
+      (reference "PT54") (unit 1) (value "PowerTie_2") (footprint "PET:NetTie-2_SMD_Pad_0.28")
+    )
+    (path "/00000000-0000-0000-0000-000061b9c2eb/111375f9-032b-4541-b4f8-f58be30b9c15"
+      (reference "PT55") (unit 1) (value "PowerTie_2") (footprint "PET:NetTie-2_SMD_Pad_1.6_to_0.4mm")
     )
     (path "/00000000-0000-0000-0000-000061bef9ce/04ae58fc-a1df-4733-997e-a64d33434240"
@@
     )
     (path "/00000000-0000-0000-0000-000061ed99de/1cb7efbd-cb21-4c0a-bb06-295ded2b2bb4"
-      (reference "U15") (unit 1) (value "LM317AG-TN3-R") (footprint "Package_TO_SOT_SMD:TO-252-2")
+      (reference "U15") (unit 1) (value "LM317AG-TN3-R") (footprint "PET:TO-252-2_ThermalVias")
     )
     (path "/00000000-0000-0000-0000-0000617d6918/b70241ab-8a5c-42d5-a1ab-8f4bc50a1197/3b6d0c70-6282-4619-97c5-f97c852cfe84/946cbf38-e765-47d9-a77d-709a42611048"
