File: hw/Mainboard/FLASH.kicad_sch (KiCad schematic)
At the start: 5 parts, among them J17 BOOTSEL, U16 W25Q128JVS

Commit message: hw: update 10u caps
Other:
- title: (none) -> CBM PET Mainboard Replacement
Changed lines of the file:
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@@
 (kicad_sch (version 20211123) (generator eeschema)
-  (paper "A4")
+  (paper "A")
+  (title_block
+    (title "CBM PET Mainboard Replacement")
+  )
   (junction (at 149.86 76.2) (diameter 0) (color 0 0 0 0)
   )

Commit message: hw: wip
Parts:
- removed J17: BOOTSEL, Connector_PinHeader_2.54mm:PinHeader_1x02_P2.54mm_Vertical, symbol Connector:Conn_01x02_Male
Other:
- moved on the sheet: R26
Changed lines of the file:
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@@
     (stroke (width 0) (type default) (color 0 0 0 0))
   )
-  (wire (pts (xy 139.7 76.2) (xy 139.7 78.74))
+  (wire (pts (xy 139.7 76.2) (xy 139.7 81.28))
     (stroke (width 0) (type default) (color 0 0 0 0))
   )
   (wire (pts (xy 149.86 76.2) (xy 152.4 76.2))
-    (stroke (width 0) (type default) (color 0 0 0 0))
-  )
-  (wire (pts (xy 139.7 105.41) (xy 139.7 106.68))
     (stroke (width 0) (type default) (color 0 0 0 0))
   )
@@
     (stroke (width 0) (type default) (color 0 0 0 0))
   )
-  (wire (pts (xy 139.7 83.82) (xy 139.7 102.87))
+  (wire (pts (xy 134.62 91.44) (xy 139.7 91.44))
     (stroke (width 0) (type default) (color 0 0 0 0))
   )
@@
     (stroke (width 0) (type default) (color 0 0 0 0))
   )
+  (wire (pts (xy 139.7 91.44) (xy 139.7 86.36))
+    (stroke (width 0) (type default) (color 0 0 0 0))
+  )
   (text "Flash" (at 113.03 53.34 0)
     (effects (font (size 4 4)) (justify left bottom))
-  )
-  (label "BOOTSEL" (at 139.7 100.33 90)
-    (effects (font (size 1.27 1.27)) (justify left bottom))
   )
   (hierarchical_label "SD3" (shape bidirectional) (at 179.07 83.82 0)
@@
     (effects (font (size 1.27 1.27)) (justify left))
   )
+  (hierarchical_label "BOOTSEL" (shape input) (at 134.62 91.44 180)
+    (effects (font (size 1.27 1.27)) (justify right))
+  )
   (hierarchical_label "SD0" (shape bidirectional) (at 179.07 73.66 0)
     (effects (font (size 1.27 1.27)) (justify left))
@@
   (hierarchical_label "~{CS}" (shape input) (at 135.89 76.2 180)
     (effects (font (size 1.27 1.27)) (justify right))
-  )
-  (symbol (lib_id "power:GND") (at 139.7 106.68 0) (mirror y) (unit 1)
-    (in_bom yes) (on_board yes)
-    (property "Reference" "#PWR082" (id 0) (at 139.7 113.03 0)
-      (effects (font (size 1.27 1.27)) hide)
-    )
-    (property "Value" "GND" (id 1) (at 139.573 111.0742 0))
-    (property "Footprint" "Connector_PinHeader_2.54mm:PinHeader_1x02_P2.54mm_Vertical" (id 2) (at 139.7 106.68 0)
-      (effects (font (size 1.27 1.27)) hide)
-    )
-    (property "Datasheet" "" (id 3) (at 139.7 106.68 0)
-      (effects (font (size 1.27 1.27)) hide)
-    )
-    (pin "1")
   )
   (symbol (lib_id "power:GND") (at 165.1 90.17 0) (unit 1)
@@
     (pin "1")
   )
-  (symbol (lib_id "Connector:Conn_01x02_Male") (at 134.62 105.41 0) (mirror x) (unit 1)
+  (symbol (lib_id "Device:R_Small") (at 139.7 83.82 180) (unit 1)
     (in_bom yes) (on_board yes)
-    (property "Reference" "J17" (id 0) (at 146.05 105.41 0))
-    (property "Value" "BOOTSEL" (id 1) (at 146.05 102.87 0))
-    (property "Footprint" "Connector_PinHeader_2.54mm:PinHeader_1x02_P2.54mm_Vertical" (id 2) (at 134.62 105.41 0)
+    (property "Reference" "R26" (id 0) (at 138.43 86.36 90)
+      (effects (font (size 1.27 1.27)) (justify left))
+    )
+    (property "Value" "1k" (id 1) (at 139.7 82.55 90)
+      (effects (font (size 1.27 1.27)) (justify left))
+    )
+    (property "Footprint" "Resistor_SMD:R_0402_1005Metric" (id 2) (at 139.7 83.82 0)
       (effects (font (size 1.27 1.27)) hide)
     )
-    (property "Datasheet" "~" (id 3) (at 134.62 105.41 0)
+    (property "Datasheet" "https://datasheet.lcsc.com/lcsc/2206010216_UNI-ROYAL-Uniroyal-Elec-0402WGF1001TCE_C11702.pdf" (id 3) (at 139.7 83.82 0)
       (effects (font (size 1.27 1.27)) hide)
     )
-    (pin "1")
-    (pin "2")
-  )
-  (symbol (lib_id "Device:R_Small") (at 139.7 81.28 180) (unit 1)
-    (in_bom yes) (on_board yes)
-    (property "Reference" "R26" (id 0) (at 138.43 83.82 90)
-      (effects (font (size 1.27 1.27)) (justify left))
-    )
-    (property "Value" "1k" (id 1) (at 139.7 80.01 90)
-      (effects (font (size 1.27 1.27)) (justify left))
-    )
-    (property "Footprint" "Resistor_SMD:R_0402_1005Metric" (id 2) (at 139.7 81.28 0)
+    (property "LCSC" "C11702" (id 4) (at 139.7 83.82 0)
       (effects (font (size 1.27 1.27)) hide)
     )
-    (property "Datasheet" "https://datasheet.lcsc.com/lcsc/2206010216_UNI-ROYAL-Uniroyal-Elec-0402WGF1001TCE_C11702.pdf" (id 3) (at 139.7 81.28 0)
-      (effects (font (size 1.27 1.27)) hide)
-    )
-    (property "LCSC" "C11702" (id 4) (at 139.7 81.28 0)
-      (effects (font (size 1.27 1.27)) hide)
-    )

Commit message: hw: wip
Parts:
- C51: LCSC C1525 -> C307331
Changed lines of the file:
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@@
       (effects (font (size 1.27 1.27)) hide)
     )
-    (property "Datasheet" "https://datasheet.lcsc.com/lcsc/1810191219_Samsung-Electro-Mechanics-CL05B104KO5NNNC_C1525.pdf" (id 3) (at 168.91 60.96 0)
+    (property "Datasheet" "" (id 3) (at 168.91 60.96 0)
       (effects (font (size 1.27 1.27)) hide)
     )
-    (property "LCSC" "C1525" (id 4) (at 168.91 60.96 0)
+    (property "LCSC" "C307331" (id 4) (at 168.91 60.96 0)
       (effects (font (size 1.27 1.27)) hide)
     )

Commit message: wip
Parts:
- added J8: FLASH, Connector_PinHeader_2.54mm:PinHeader_1x02_P2.54mm_Vertical, symbol Connector:Conn_01x02_Male
Connections:
- net GND: now also J8.1 (Pin_1)
- net BOOTSEL: no longer names the net of R26.1
- net BOOTSEL: now also J8.2 (Pin_2)
Other:
- moved on the sheet: C51, R25, R26, U16
