File: hw/Mainboard/CPU.kicad_sch (KiCad schematic)
At the start: 12 parts, among them SW1 RESET, SW4 NMI, U11 W65C02S, U12 AS6C1008

Commit message: hw: wip
Connections:
- net GND: no longer SW1.1, SW4.1, U11.21 (VSS), U12.16 (VSS), U12.22 (CE#)
- new net PD_GND: SW1.1, SW4.1, U11.21 (VSS), U12.16 (VSS), U12.22 (CE#)
Changed lines of the file:
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@@
   (junction (at 41.91 187.96) (diameter 0) (color 0 0 0 0)
-  )
-  (junction (at 132.08 189.23) (diameter 0) (color 0 0 0 0)
-  )
-  (junction (at 101.6 189.23) (diameter 0) (color 0 0 0 0)
   )
   (junction (at 125.73 179.07) (diameter 0) (color 0 0 0 0)
@@
     (stroke (width 0) (type default) (color 0 0 0 0))
   )
-  (wire (pts (xy 101.6 189.23) (xy 95.25 189.23))
-    (stroke (width 0) (type default) (color 0 0 0 0))
-  )
   (wire (pts (xy 60.96 107.95) (xy 60.96 66.04))
     (stroke (width 0) (type default) (color 0 0 0 0))
@@
     (stroke (width 0) (type default) (color 0 0 0 0))
   )
-  (wire (pts (xy 132.08 189.23) (xy 138.43 189.23))
-    (stroke (width 0) (type default) (color 0 0 0 0))
-  )
   (wire (pts (xy 95.25 179.07) (xy 107.95 179.07))
     (stroke (width 0) (type default) (color 0 0 0 0))
   )
-  (wire (pts (xy 101.6 190.5) (xy 101.6 189.23))
-    (stroke (width 0) (type default) (color 0 0 0 0))
-  )
   (wire (pts (xy 139.7 87.63) (xy 175.26 87.63))
     (stroke (width 0) (type default) (color 0 0 0 0))
@@
     (stroke (width 0) (type default) (color 0 0 0 0))
   )
-  (wire (pts (xy 132.08 190.5) (xy 132.08 189.23))
-    (stroke (width 0) (type default) (color 0 0 0 0))
-  )
   (bus (pts (xy 114.3 86.36) (xy 114.3 88.9))
     (stroke (width 0) (type default) (color 0 0 0 0))
@@
     (stroke (width 0) (type default) (color 0 0 0 0))
   )
-  (wire (pts (xy 101.6 189.23) (xy 107.95 189.23))
-    (stroke (width 0) (type default) (color 0 0 0 0))
-  )
   (bus (pts (xy 137.16 119.38) (xy 137.16 118.11))
     (stroke (width 0) (type default) (color 0 0 0 0))
@@
   )
   (wire (pts (xy 53.34 124.46) (xy 77.47 124.46))
-    (stroke (width 0) (type default) (color 0 0 0 0))
-  )
-  (wire (pts (xy 132.08 189.23) (xy 125.73 189.23))
     (stroke (width 0) (type default) (color 0 0 0 0))
   )
@@
     (pin "2")
   )
+  (symbol (lib_id "power:GND") (at 138.43 189.23 0) (unit 1)
+    (in_bom yes) (on_board yes)
+    (property "Reference" "#PWR0176" (id 0) (at 138.43 195.58 0)
+      (effects (font (size 1.27 1.27)) hide)
+    )
+    (property "Value" "GND" (id 1) (at 138.557 193.6242 0))
+    (property "Footprint" "" (id 2) (at 138.43 189.23 0)
+      (effects (font (size 1.27 1.27)) hide)
+    )
+    (property "Datasheet" "" (id 3) (at 138.43 189.23 0)
+      (effects (font (size 1.27 1.27)) hide)
+    )
+    (pin "1")
+  )
   (symbol (lib_id "Device:R_Small") (at 76.2 71.12 0) (unit 1)
     (in_bom yes) (on_board yes)
@@
     (pin "1")
     (pin "2")
+  )
+  (symbol (lib_id "PET:PD_GND") (at 125.73 189.23 0) (unit 1)
+    (in_bom yes) (on_board yes) (fields_autoplaced)
+    (property "Reference" "#PWR0140" (id 0) (at 125.73 195.58 0)
+      (effects (font (size 1.27 1.27)) hide)
+    )
+    (property "Value" "PD_GND" (id 1) (at 125.73 194.31 0))
+    (property "Footprint" "" (id 2) (at 125.73 189.23 0)
+      (effects (font (size 1.27 1.27)) hide)
+    )
+    (property "Datasheet" "" (id 3) (at 125.73 189.23 0)
+      (effects (font (size 1.27 1.27)) hide)
+    )
+    (pin "1")
   )
   (symbol (lib_id "power:GND") (at 41.91 189.23 0) (unit 1)
@@
     (pin "1")
   )
-  (symbol (lib_id "power:GND") (at 101.6 190.5 0) (unit 1)
-    (in_bom yes) (on_board yes)
-    (property "Reference" "#PWR078" (id 0) (at 101.6 196.85 0)
-      (effects (font (size 1.27 1.27)) hide)
-    )
-    (property "Value" "GND" (id 1) (at 101.727 194.8942 0))
-    (property "Footprint" "" (id 2) (at 101.6 190.5 0)
-      (effects (font (size 1.27 1.27)) hide)
-    )
-    (property "Datasheet" "" (id 3) (at 101.6 190.5 0)
+  (symbol (lib_id "PET:PD_GND") (at 95.25 189.23 0) (unit 1)
+    (in_bom yes) (on_board yes) (fields_autoplaced)
+    (property "Reference" "#PWR0171" (id 0) (at 95.25 195.58 0)
+      (effects (font (size 1.27 1.27)) hide)
+    )
+    (property "Value" "PD_GND" (id 1) (at 95.25 194.31 0))
+    (property "Footprint" "" (id 2) (at 95.25 189.23 0)
+      (effects (font (size 1.27 1.27)) hide)
+    )
+    (property "Datasheet" "" (id 3) (at 95.25 189.23 0)
       (effects (font (size 1.27 1.27)) hide)
     )
@@
     (pin "1")
     (pin "2")
+  )
+  (symbol (lib_id "power:GND") (at 107.95 189.23 0) (unit 1)
+    (in_bom yes) (on_board yes)
+    (property "Reference" "#PWR0174" (id 0) (at 107.95 195.58 0)
+      (effects (font (size 1.27 1.27)) hide)
+    )
+    (property "Value" "GND" (id 1) (at 108.077 193.6242 0))
+    (property "Footprint" "" (id 2) (at 107.95 189.23 0)
+      (effects (font (size 1.27 1.27)) hide)
+    )
+    (property "Datasheet" "" (id 3) (at 107.95 189.23 0)
+      (effects (font (size 1.27 1.27)) hide)
+    )
+    (pin "1")
   )
   (symbol (lib_id "Switch:SW_Push") (at 125.73 184.15 90) (unit 1)
@@
     (pin "1")
   )
-  (symbol (lib_id "power:GND") (at 187.96 127 0) (unit 1)
-    (in_bom yes) (on_board yes)
-    (property "Reference" "#PWR075" (id 0) (at 187.96 133.35 0)
-      (effects (font (size 1.27 1.27)) hide)
-    )
-    (property "Value" "GND" (id 1) (at 188.087 131.3942 0))
-    (property "Footprint" "" (id 2) (at 187.96 127 0)
-      (effects (font (size 1.27 1.27)) hide)
-    )
-    (property "Datasheet" "" (id 3) (at 187.96 127 0)
-      (effects (font (size 1.27 1.27)) hide)
-    )
-    (pin "1")
-  )
-  (symbol (lib_id "power:GND") (at 92.71 143.51 0) (unit 1)
-    (in_bom yes) (on_board yes)
-    (property "Reference" "#PWR076" (id 0) (at 92.71 149.86 0)
-      (effects (font (size 1.27 1.27)) hide)
-    )
-    (property "Value" "GND" (id 1) (at 92.837 147.9042 0))
+  (symbol (lib_id "PET:PD_GND") (at 92.71 143.51 0) (unit 1)
+    (in_bom yes) (on_board yes) (fields_autoplaced)
+    (property "Reference" "#PWR0104" (id 0) (at 92.71 149.86 0)
+      (effects (font (size 1.27 1.27)) hide)
+    )
+    (property "Value" "PD_GND" (id 1) (at 92.71 148.59 0))
     (property "Footprint" "" (id 2) (at 92.71 143.51 0)
       (effects (font (size 1.27 1.27)) hide)
     )
     (property "Datasheet" "" (id 3) (at 92.71 143.51 0)
-      (effects (font (size 1.27 1.27)) hide)
-    )
-    (pin "1")
-  )
-  (symbol (lib_id "power:GND") (at 132.08 190.5 0) (unit 1)
-    (in_bom yes) (on_board yes)
-    (property "Reference" "#PWR085" (id 0) (at 132.08 196.85 0)
-      (effects (font (size 1.27 1.27)) hide)
-    )
-    (property "Value" "GND" (id 1) (at 132.207 194.8942 0))
-    (property "Footprint" "" (id 2) (at 132.08 190.5 0)
-      (effects (font (size 1.27 1.27)) hide)
-    )
-    (property "Datasheet" "" (id 3) (at 132.08 190.5 0)
       (effects (font (size 1.27 1.27)) hide)
     )
@@
     (pin "2")
   )
+  (symbol (lib_id "PET:PD_GND") (at 187.96 127 0) (unit 1)
+    (in_bom yes) (on_board yes) (fields_autoplaced)
+    (property "Reference" "#PWR0101" (id 0) (at 187.96 133.35 0)
+      (effects (font (size 1.27 1.27)) hide)
+    )
+    (property "Value" "PD_GND" (id 1) (at 187.96 132.08 0))
+    (property "Footprint" "" (id 2) (at 187.96 127 0)
+      (effects (font (size 1.27 1.27)) hide)
+    )
+    (property "Datasheet" "" (id 3) (at 187.96 127 0)
+      (effects (font (size 1.27 1.27)) hide)
+    )
+    (pin "1")
+  )
   (symbol (lib_id "power:+3V3") (at 41.91 179.07 0) (unit 1)

Commit message: hw: wip
Parts:
- C10, C11: LCSC C1525 -> C307331
Changed lines of the file:
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@@
       (effects (font (size 1.27 1.27)) hide)
     )
-    (property "Datasheet" "https://datasheet.lcsc.com/lcsc/1810191219_Samsung-Electro-Mechanics-CL05B104KO5NNNC_C1525.pdf" (id 3) (at 35.56 184.15 0)
+    (property "Datasheet" "" (id 3) (at 35.56 184.15 0)
       (effects (font (size 1.27 1.27)) hide)
     )
-    (property "LCSC" "C1525" (id 4) (at 35.56 184.15 0)
+    (property "LCSC" "C307331" (id 4) (at 35.56 184.15 0)
       (effects (font (size 1.27 1.27)) hide)
     )
@@
       (effects (font (size 1.27 1.27)) hide)
     )
-    (property "Datasheet" "https://datasheet.lcsc.com/lcsc/1810191219_Samsung-Electro-Mechanics-CL05B104KO5NNNC_C1525.pdf" (id 3) (at 48.26 184.15 0)
+    (property "Datasheet" "" (id 3) (at 48.26 184.15 0)
       (effects (font (size 1.27 1.27)) hide)
     )
-    (property "LCSC" "C1525" (id 4) (at 48.26 184.15 0)
+    (property "LCSC" "C307331" (id 4) (at 48.26 184.15 0)
       (effects (font (size 1.27 1.27)) hide)
     )

Commit message: wip
Connections:
- net ϕ2 renamed PHI2
Changed lines of the file:
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@@
     (effects (font (size 1.27 1.27)) (justify right))
   )
-  (hierarchical_label "ϕ2" (shape input) (at 53.34 83.82 180)
+  (hierarchical_label "PHI2" (shape input) (at 53.34 83.82 180)
     (effects (font (size 1.27 1.27)) (justify right))
   )
@@
       (effects (font (size 1.27 1.27)) hide)
     )
-    (property "Datasheet" "" (id 3) (at 92.71 58.42 0)
+    (property "Datasheet" "https://www.mouser.com/datasheet/2/436/w65c02s-2572.pdf" (id 3) (at 92.71 58.42 0)
       (effects (font (size 1.27 1.27)) hide)
     )
@@
       (effects (font (size 1.27 1.27)) hide)
     )
-    (property "Datasheet" "" (id 3) (at 187.96 95.25 0)
+    (property "Datasheet" "https://www.mouser.com/datasheet/2/12/AS6C1008feb2007-1511508.pdf" (id 3) (at 187.96 95.25 0)
       (effects (font (size 1.27 1.27)) hide)
     )
@@
       (effects (font (size 1.27 1.27)) hide)
     )
-    (property "Datasheet" "" (id 3) (at 66.04 90.17 0)
+    (property "Datasheet" "https://datasheet.lcsc.com/lcsc/2206010045_UNI-ROYAL-Uniroyal-Elec-0402WGF4701TCE_C25900.pdf" (id 3) (at 66.04 90.17 0)
       (effects (font (size 1.27 1.27)) hide)
     )
@@
       (effects (font (size 1.27 1.27)) hide)
     )
-    (property "Datasheet" "" (id 3) (at 60.96 110.49 0)
+    (property "Datasheet" "https://datasheet.lcsc.com/lcsc/2206010045_UNI-ROYAL-Uniroyal-Elec-0402WGF4701TCE_C25900.pdf" (id 3) (at 60.96 110.49 0)
       (effects (font (size 1.27 1.27)) hide)
     )
@@
       (effects (font (size 1.27 1.27)) hide)
     )
-    (property "Datasheet" "" (id 3) (at 71.12 90.17 0)
+    (property "Datasheet" "https://datasheet.lcsc.com/lcsc/2206010045_UNI-ROYAL-Uniroyal-Elec-0402WGF4701TCE_C25900.pdf" (id 3) (at 71.12 90.17 0)
       (effects (font (size 1.27 1.27)) hide)
     )
@@
       (effects (font (size 1.27 1.27)) hide)
     )
-    (property "Datasheet" "" (id 3) (at 76.2 71.12 0)
-      (effects (font (size 1.27 1.27)) hide)
-    )
+    (property "Datasheet" "https://datasheet.lcsc.com/lcsc/2206010045_UNI-ROYAL-Uniroyal-Elec-0402WGF4701TCE_C25900.pdf" (id 3) (at 76.2 71.12 0)
+      (effects (font (size 1.27 1.27)) hide)
+    )

Commit message: hw: add more Mouse part numbers
Parts:
- SW1, SW4: MOUSER (none) -> 611-PTS636SK43LFS
Changed lines of the file:
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@@
+      (effects (font (size 1.27 1.27)) hide)
+    )
+    (property "MOUSER" "611-PTS636SK43LFS" (id 6) (at 95.25 184.15 0)
       (effects (font (size 1.27 1.27)) hide)
     )
@@
       (effects (font (size 1.27 1.27)) hide)
     )
+    (property "MOUSER" "611-PTS636SK43LFS" (id 6) (at 125.73 184.15 0)
+      (effects (font (size 1.27 1.27)) hide)
+    )

Commit message: hw: PN for IC, remove dup PNs, remove redundant headroom text on PWR
Parts:
- U11: DIGI-KEY AE10008-ND -> (none); MOUSER 955-W65C02S6TPG-14 -> 955-W65C02S6TPG-14,571-1-2199299-5
- U12: DIGI-KEY 2057-ICS-632-T-ND -> (none); MOUSER 913-AS6C1008-55PCN -> 913-AS6C1008-55PCN,649-DILB32P223TLF
Changed lines of the file:
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@@
       (effects (font (size 1.27 1.27)) hide)
     )
-    (property "MOUSER" "955-W65C02S6TPG-14" (id 4) (at 92.71 106.68 0)
-      (effects (font (size 1.27 1.27)) hide)
-    )
-    (property "DIGI-KEY" "AE10008-ND" (id 5) (at 92.71 106.68 0)
+    (property "MOUSER" "955-W65C02S6TPG-14,571-1-2199299-5" (id 4) (at 92.71 106.68 0)
       (effects (font (size 1.27 1.27)) hide)
     )
@@
       (effects (font (size 1.27 1.27)) hide)
     )
-    (property "MOUSER" "913-AS6C1008-55PCN" (id 4) (at 187.96 97.79 0)
+    (property "MOUSER" "913-AS6C1008-55PCN,649-DILB32P223TLF" (id 4) (at 187.96 97.79 0)
       (effects (font (size 1.27 1.27)) hide)
     )
-    (property "DIGI-KEY" "2057-ICS-632-T-ND" (id 5) (at 187.96 97.79 0)
-      (effects (font (size 1.27 1.27)) hide)
-    )

Commit message: hw: 9V DC plug on left edge, change default track size
Parts:
- renumbered C10 to C1, C11 to C2, C24 to C3, C25 to C4, R59 to R1, R38 to R2, R39 to R3, R40 to R4, SW4 to SW2, U12 to U1, U11 to U2
Changed lines of the file:
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@@
   (symbol (lib_id "Mainboard-rescue:W65C02SxP-PET") (at 92.71 106.68 0) (unit 1)
     (in_bom yes) (on_board yes)
-    (property "Reference" "U11" (id 0) (at 100.33 71.12 0))
+    (property "Reference" "U2" (id 0) (at 100.33 71.12 0))
     (property "Value" "W65C02S" (id 1) (at 92.71 102.87 0)
       (effects (font (size 1.27 1.27) bold italic))
@@
   (symbol (lib_id "Mainboard-rescue:AS6C1008-PET") (at 187.96 97.79 0) (unit 1)
     (in_bom yes) (on_board yes)
-    (property "Reference" "U12" (id 0) (at 195.58 71.12 0))
+    (property "Reference" "U1" (id 0) (at 195.58 71.12 0))
     (property "Value" "AS6C1008" (id 1) (at 187.96 96.52 0)
       (effects (font (size 1.27 1.27) bold italic))
@@
   (symbol (lib_id "Device:R_Small") (at 66.04 90.17 0) (unit 1)
     (in_bom yes) (on_board yes)
-    (property "Reference" "R38" (id 0) (at 64.135 92.075 90)
+    (property "Reference" "R2" (id 0) (at 64.135 92.075 90)
       (effects (font (size 1.27 1.27)) (justify left))
     )
@@
   (symbol (lib_id "Device:R_Small") (at 60.96 110.49 180) (unit 1)
     (in_bom yes) (on_board yes)
-    (property "Reference" "R40" (id 0) (at 59.055 108.585 90)
+    (property "Reference" "R4" (id 0) (at 59.055 108.585 90)
       (effects (font (size 1.27 1.27)) (justify left))
     )
@@
   (symbol (lib_id "Device:R_Small") (at 71.12 90.17 0) (unit 1)
     (in_bom yes) (on_board yes)
-    (property "Reference" "R39" (id 0) (at 69.215 92.075 90)
+    (property "Reference" "R3" (id 0) (at 69.215 92.075 90)
       (effects (font (size 1.27 1.27)) (justify left))
     )
@@
   (symbol (lib_id "Device:C_Small") (at 35.56 184.15 0) (unit 1)
     (in_bom yes) (on_board yes)
-    (property "Reference" "C10" (id 0) (at 37.8968 182.9816 0)
+    (property "Reference" "C1" (id 0) (at 37.8968 182.9816 0)
       (effects (font (size 1.27 1.27)) (justify left))
     )
@@
   (symbol (lib_id "Device:C_Small") (at 48.26 184.15 0) (unit 1)
     (in_bom yes) (on_board yes)
-    (property "Reference" "C11" (id 0) (at 50.5968 182.9816 0)
+    (property "Reference" "C2" (id 0) (at 50.5968 182.9816 0)
       (effects (font (size 1.27 1.27)) (justify left))
     )
@@
   (symbol (lib_id "power:GND") (at 138.43 189.23 0) (unit 1)
     (in_bom yes) (on_board yes)
-    (property "Reference" "#PWR0176" (id 0) (at 138.43 195.58 0)
+    (property "Reference" "#PWR010" (id 0) (at 138.43 195.58 0)
       (effects (font (size 1.27 1.27)) hide)
     )
@@
   (symbol (lib_id "Device:R_Small") (at 76.2 71.12 0) (unit 1)
     (in_bom yes) (on_board yes)
-    (property "Reference" "R59" (id 0) (at 74.295 73.025 90)
+    (property "Reference" "R1" (id 0) (at 74.295 73.025 90)
       (effects (font (size 1.27 1.27)) (justify left))
     )
@@
   (symbol (lib_id "PET:PD_GND") (at 125.73 189.23 0) (unit 1)
     (in_bom yes) (on_board yes) (fields_autoplaced)
-    (property "Reference" "#PWR0140" (id 0) (at 125.73 195.58 0)
+    (property "Reference" "#PWR09" (id 0) (at 125.73 195.58 0)
       (effects (font (size 1.27 1.27)) hide)
     )
@@
   (symbol (lib_id "power:GND") (at 41.91 189.23 0) (unit 1)
     (in_bom yes) (on_board yes)
-    (property "Reference" "#PWR0221" (id 0) (at 41.91 195.58 0)
+    (property "Reference" "#PWR06" (id 0) (at 41.91 195.58 0)
       (effects (font (size 1.27 1.27)) hide)
     )
@@
   (symbol (lib_id "PET:PD_GND") (at 95.25 189.23 0) (unit 1)
     (in_bom yes) (on_board yes) (fields_autoplaced)
-    (property "Reference" "#PWR0171" (id 0) (at 95.25 195.58 0)
+    (property "Reference" "#PWR07" (id 0) (at 95.25 195.58 0)
       (effects (font (size 1.27 1.27)) hide)
     )
@@
   (symbol (lib_id "Device:C_Small") (at 107.95 184.15 0) (unit 1)
     (in_bom yes) (on_board yes)
-    (property "Reference" "C24" (id 0) (at 110.2868 182.9816 0)
+    (property "Reference" "C3" (id 0) (at 110.2868 182.9816 0)
       (effects (font (size 1.27 1.27)) (justify left))
     )
@@
   (symbol (lib_id "power:GND") (at 107.95 189.23 0) (unit 1)
     (in_bom yes) (on_board yes)
-    (property "Reference" "#PWR0174" (id 0) (at 107.95 195.58 0)
+    (property "Reference" "#PWR08" (id 0) (at 107.95 195.58 0)
       (effects (font (size 1.27 1.27)) hide)
     )
@@
   (symbol (lib_id "Switch:SW_Push") (at 125.73 184.15 90) (unit 1)
     (in_bom yes) (on_board yes)
-    (property "Reference" "SW4" (id 0) (at 126.9492 182.9816 90)
+    (property "Reference" "SW2" (id 0) (at 126.9492 182.9816 90)
       (effects (font (size 1.27 1.27)) (justify right))
     )
@@
   (symbol (lib_id "power:+3V3") (at 187.96 67.31 0) (unit 1)
     (in_bom yes) (on_board yes) (fields_autoplaced)
-    (property "Reference" "#PWR074" (id 0) (at 187.96 71.12 0)
+    (property "Reference" "#PWR02" (id 0) (at 187.96 71.12 0)
       (effects (font (size 1.27 1.27)) hide)
     )
@@
   (symbol (lib_id "PET:PD_GND") (at 92.71 143.51 0) (unit 1)
     (in_bom yes) (on_board yes) (fields_autoplaced)
-    (property "Reference" "#PWR0104" (id 0) (at 92.71 149.86 0)
+    (property "Reference" "#PWR04" (id 0) (at 92.71 149.86 0)
       (effects (font (size 1.27 1.27)) hide)
     )
@@
   (symbol (lib_id "power:+3V3") (at 92.71 64.77 0) (unit 1)
     (in_bom yes) (on_board yes) (fields_autoplaced)
-    (property "Reference" "#PWR070" (id 0) (at 92.71 68.58 0)
+    (property "Reference" "#PWR01" (id 0) (at 92.71 68.58 0)
       (effects (font (size 1.27 1.27)) hide)
     )
@@
   (symbol (lib_id "Device:C_Small") (at 138.43 184.15 0) (unit 1)
     (in_bom yes) (on_board yes)
-    (property "Reference" "C25" (id 0) (at 140.7668 182.9816 0)
+    (property "Reference" "C4" (id 0) (at 140.7668 182.9816 0)
       (effects (font (size 1.27 1.27)) (justify left))
     )
@@
   (symbol (lib_id "PET:PD_GND") (at 187.96 127 0) (unit 1)
     (in_bom yes) (on_board yes) (fields_autoplaced)
-    (property "Reference" "#PWR0101" (id 0) (at 187.96 133.35 0)
+    (property "Reference" "#PWR03" (id 0) (at 187.96 133.35 0)
       (effects (font (size 1.27 1.27)) hide)
     )
@@
   (symbol (lib_id "power:+3V3") (at 41.91 179.07 0) (unit 1)
     (in_bom yes) (on_board yes) (fields_autoplaced)
-    (property "Reference" "#PWR07" (id 0) (at 41.91 182.88 0)
-      (effects (font (size 1.27 1.27)) hide)
-    )
+    (property "Reference" "#PWR05" (id 0) (at 41.91 182.88 0)
+      (effects (font (size 1.27 1.27)) hide)
+    )
