File: hw/Mainboard/USB.kicad_sch (KiCad schematic)
At the start: 6 parts, among them J25 USB2.0_HOST_TYPE_C

Commit message: hw: renumber J* refs to match PET connectors
Parts:
- renumbered C101 to C100, C84 to C101, D3 to D12, J25 to J24, R70 to R56, R71 to R57
Changed lines of the file:
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@@
   (symbol (lib_id "Device:C_Small") (at 97.79 82.55 0) (unit 1)
     (in_bom yes) (on_board yes)
-    (property "Reference" "C84" (id 0) (at 100.1268 81.3816 0)
+    (property "Reference" "C101" (id 0) (at 100.1268 81.3816 0)
       (effects (font (size 1.27 1.27)) (justify left))
     )
@@
   (symbol (lib_id "PET:PD_GND") (at 83.82 87.63 0) (unit 1)
     (in_bom yes) (on_board yes) (fields_autoplaced)
-    (property "Reference" "#PWR0158" (id 0) (at 83.82 93.98 0)
+    (property "Reference" "#PWR0171" (id 0) (at 83.82 93.98 0)
       (effects (font (size 1.27 1.27)) hide)
     )
@@
   (symbol (lib_id "JLCPCB:USB_C_Receptacle_USB2.0") (at 152.4 92.71 0) (mirror y) (unit 1)
     (in_bom yes) (on_board yes) (fields_autoplaced)
-    (property "Reference" "J25" (id 0) (at 163.83 90.8049 0)
+    (property "Reference" "J24" (id 0) (at 163.83 90.8049 0)
       (effects (font (size 1.27 1.27)) (justify right))
     )
@@
   (symbol (lib_id "Device:D_Schottky_Small") (at 83.82 66.04 90) (unit 1)
     (in_bom yes) (on_board yes)
-    (property "Reference" "D3" (id 0) (at 88.9 66.04 0))
+    (property "Reference" "D12" (id 0) (at 88.9 66.04 0))
     (property "Value" "SS54" (id 1) (at 86.614 67.183 0))
     (property "Footprint" "Diode_SMD:D_SMA" (id 2) (at 83.82 66.04 90)
@@
   (symbol (lib_id "Device:R_Small") (at 128.27 85.09 90) (mirror x) (unit 1)
     (in_bom yes) (on_board yes)
-    (property "Reference" "R71" (id 0) (at 130.175 86.995 90)
+    (property "Reference" "R57" (id 0) (at 130.175 86.995 90)
       (effects (font (size 1.27 1.27)) (justify left))
     )
@@
   (symbol (lib_id "Device:C_Small") (at 83.82 82.55 0) (unit 1)
     (in_bom yes) (on_board yes)
-    (property "Reference" "C101" (id 0) (at 86.1568 81.3816 0)
+    (property "Reference" "C100" (id 0) (at 86.1568 81.3816 0)
       (effects (font (size 1.27 1.27)) (justify left))
     )
@@
   (symbol (lib_id "power:+5V") (at 83.82 62.23 0) (mirror y) (unit 1)
     (in_bom yes) (on_board yes) (fields_autoplaced)
-    (property "Reference" "#PWR0157" (id 0) (at 83.82 66.04 0)
+    (property "Reference" "#PWR0170" (id 0) (at 83.82 66.04 0)
       (effects (font (size 1.27 1.27)) hide)
     )
@@
   (symbol (lib_id "Device:R_Small") (at 128.27 82.55 90) (mirror x) (unit 1)
     (in_bom yes) (on_board yes)
-    (property "Reference" "R70" (id 0) (at 130.175 80.645 90)
+    (property "Reference" "R56" (id 0) (at 130.175 80.645 90)
       (effects (font (size 1.27 1.27)) (justify left))
     )
@@
   (symbol (lib_id "PET:PD_GND") (at 153.67 123.19 0) (unit 1)
     (in_bom yes) (on_board yes) (fields_autoplaced)
-    (property "Reference" "#PWR0159" (id 0) (at 153.67 129.54 0)
+    (property "Reference" "#PWR0172" (id 0) (at 153.67 129.54 0)
       (effects (font (size 1.27 1.27)) hide)
     )
@@
   (symbol (lib_id "power:GND") (at 160.02 123.19 0) (unit 1)
     (in_bom yes) (on_board yes) (fields_autoplaced)
-    (property "Reference" "#PWR0160" (id 0) (at 160.02 129.54 0)
+    (property "Reference" "#PWR0173" (id 0) (at 160.02 129.54 0)
       (effects (font (size 1.27 1.27)) hide)
     )
